File: GEM.sch (KiCad schematic (older format))
At the start: 0 parts

Commit message: Added datasheets. Schematic design for STN1110 complete TODO: create subsystems for STN1110
Parts:
- added C1, C2: 30p, symbol C
- added C3, C4: 1u, symbol C
- added C5: CP1, symbol CP1
- added JP1: JUMPER, symbol JUMPER
- added R1, R4, R6: 100K, symbol R
- added R2: 10K, symbol R
- added R3, R7: 1K, symbol R
- added R5: 10, symbol R
- added U1: STN1110, symbol STN1110
- added X1: 16Mhz, symbol CRYSTAL
Connections:
- net labels added: +3.3V, +5V, ANALOG_IN, CAN_RX, CAN_TX, GND, J1850_BUS+_TX, PWM/~VPW, PWM_RX, UART_RX, UART_TX, ~ISO_K_TX, ~ISO_L_TX, ~ISO_RX, ~J1850_BUS-_TX, ~OBD_RX_LED/INT, ~OBD_TX_LED/RST_NVM, ~PWR_SAVE, ~RESET, ~SLEEP, ~UART_RX_LED, ~UART_TX_LED, ~VPW_RX
- wire segments 0 -> 69
Other:
- note added: "0.1"
- note added: "1"
- note added: "11/9/14"
- note added: "Jumper reset non-volatile memory"
- note added: "OBD-II INTERPRETER INTERFACE"
- note added: "TODO: CREATE 5V_SW POWER"

Commit message: Created hierarchical scheme for schematics TODO: Change power ports to hierarchical pins
Parts:
- removed C1, C2: 30p, symbol C
- removed C3, C4: 1u, symbol C
- removed C5: CP1, symbol CP1
- removed JP1: JUMPER, symbol JUMPER
- removed R1, R4, R6: 100K, symbol R
- removed R2: 10K, symbol R
- removed R3, R7: 1K, symbol R
- removed R5: 10, symbol R
- removed U1: STN1110, symbol STN1110
- removed X1: 16Mhz, symbol CRYSTAL
Connections:
- net labels removed: +3.3V, +5V, ANALOG_IN, CAN_RX, CAN_TX, GND, J1850_BUS+_TX, PWM/~VPW, PWM_RX, UART_RX, UART_TX, ~ISO_K_TX, ~ISO_L_TX, ~ISO_RX, ~J1850_BUS-_TX, ~OBD_RX_LED/INT, ~OBD_TX_LED/RST_NVM, ~PWR_SAVE, ~RESET, ~SLEEP, ~UART_RX_LED, ~UART_TX_LED, ~VPW_RX
- wire segments 69 -> 0
Other:
- note removed: "Jumper reset non-volatile memory"
- note removed: "TODO: CREATE 5V_SW POWER"

Commit message: Added power ports to STN1110
Changed lines of the file:
@@
 F20 "~ISO_K_TX" O R 3300 2050 60
 F21 "~ISO_L_TX" O R 3300 1950 60
+F22 "3.3V" B L 1300 3000 60
+F23 "5V_SW" B R 3300 3000 60
+F24 "GND" B L 1300 1800 60
 $EndSheet
 $EndSCHEMATC

Commit message: Added MCP2551 and it's connections to STN1110
Changed lines of the file:
@@
 $Descr A4 11693 8268
 encoding utf-8
-Sheet 1 2
+Sheet 1 3
 Title ""
 Date ""
@@
 F24 "GND" B L 1300 1800 60
 $EndSheet
+$Sheet
+S 1350 3700 1700 2000
+U 5462582D
+F0 "MCP2551" 60
+F1 "MCP2551.sch" 60
+F2 "CAN_TX" I R 3050 4950 60
+F3 "CAN_RX" O L 1350 5100 60
+F4 "GND" I L 1350 5550 60
+F5 "5V_SW" I R 3050 5550 60
+F6 "CAN_HI" B R 3050 5350 60
+F7 "CAN_LOW" B R 3050 5100 60
+$EndSheet
+Wire Wire Line
+	1350 5100 1150 5100
+Wire Wire Line
+	1150 5100 1150 2850
+Wire Wire Line
+	1150 2850 1300 2850
+Wire Wire Line
+	3050 4950 3400 4950
+Wire Wire Line
+	3400 4950 3400 2850
+Wire Wire Line
+	3400 2850 3300 2850
 $EndSCHEMATC

Commit message: Added status lights sheet
Changed lines of the file:
@@
 $Descr A4 11693 8268
 encoding utf-8
-Sheet 1 3
+Sheet 1 4
 Title ""
 Date ""
@@
 $EndSheet
 $Sheet
-S 1350 3700 1700 2000
+S 1350 3700 1950 1000
 U 5462582D
 F0 "MCP2551" 60
 F1 "MCP2551.sch" 60
-F2 "CAN_TX" I R 3050 4950 60
-F3 "CAN_RX" O L 1350 5100 60
-F4 "GND" I L 1350 5550 60
-F5 "5V_SW" I R 3050 5550 60
-F6 "CAN_HI" B R 3050 5350 60
-F7 "CAN_LOW" B R 3050 5100 60
+F2 "CAN_TX" I R 3300 3900 60
+F3 "CAN_RX" O L 1350 3900 60
+F4 "GND" I R 3300 4500 60
+F5 "5V_SW" I R 3300 4350 60
+F6 "CAN_HI" B R 3300 4200 60
+F7 "CAN_LOW" B R 3300 4050 60
 $EndSheet
-Wire Wire Line
-	1350 5100 1150 5100
-Wire Wire Line
-	1150 5100 1150 2850
 Wire Wire Line
 	1150 2850 1300 2850
 Wire Wire Line
-	3050 4950 3400 4950
+	3300 2850 3500 2850
 Wire Wire Line
-	3400 4950 3400 2850
+	1150 2850 1150 3900
 Wire Wire Line
-	3400 2850 3300 2850
+	1150 3900 1350 3900
+Wire Wire Line
+	3300 3900 3500 3900
+Wire Wire Line
+	3500 3900 3500 2850
+$Sheet
+S 3950 1800 1150 1100
+U 5462AB81
+F0 "STATUS_LIGHTS" 60
+F1 "STATUS_LIGHTS.sch" 60
+F2 "3.3V" I L 3950 1950 60
+F3 "~OBD_TX_LED/RST_NVM" I L 3950 2450 60
+F4 "~OBD_RX_LED/INT" I L 3950 2350 60
+F5 "~UART_TX_LED" I L 3950 2250 60
+F6 "~UART_RX_LED" I L 3950 2150 60
+$EndSheet
+Wire Wire Line
+	3300 2150 3950 2150
+Wire Wire Line
+	3300 2250 3950 2250
+Wire Wire Line
+	3300 2350 3950 2350
+Wire Wire Line
+	3300 2450 3950 2450
 $EndSCHEMATC

Commit message: Added transceivers for J1850 and ISO
Other:
- note removed: "0.1"
- note removed: "1"
- note removed: "11/9/14"
- note removed: "OBD-II INTERPRETER INTERFACE"
Changed lines of the file:
@@
 $Descr A4 11693 8268
 encoding utf-8
-Sheet 1 4
-Title ""
-Date ""
-Rev ""
-Comp ""
+Sheet 1 5
+Title "GEM"
+Date "Saturday, November 15, 2014"
+Rev "1"
+Comp "UCF Senior Design Group 8"
 Comment1 ""
 Comment2 ""
@@
 Comment4 ""
 $EndDescr
-Text Notes 10700 7650 2    60   ~ 0
-0.1
-Text Notes 8800 7500 2    60   ~ 0
-OBD-II INTERPRETER INTERFACE
-Text Notes 7350 7250 2    60   ~ 0
-1
-Text Notes 8550 7650 2    60   ~ 0
-11/9/14
 $Sheet
 S 1300 1700 2000 1400
@@
 Wire Wire Line
 	3300 2450 3950 2450
+$Sheet
+S 1200 5500 1700 1950
+U 5467BC13
+F0 "TRANSCEIVERS" 60
+F1 "transceivers.sch" 60
+F2 "BAT" B L 1200 7250 60
+F3 "GND" I R 2900 7250 60
+F4 "~ISO_K_TX" I R 2900 7100 60
+F5 "K-LINE" O R 2900 6950 60
+F6 "L-LINE" I R 2900 6800 60
+F7 "~ISO_L_TX" I R 2900 6650 60
+F8 "BAT_SW" I R 2900 6500 60
+F9 "~ISO_RX" I R 2900 6350 60
+F10 "3.3V" I R 2900 6200 60
+F11 "PWM/~VPW" I R 2900 6050 60
+F12 "J1850_BUS+_TX" I R 2900 5850 60
+F13 "J1850_BUS+" O R 2900 5700 60
+F14 "J1850_BUS-" I L 1200 7100 60
+F15 "PWM_RX" O L 1200 6900 60
+F16 "5V_SW" I L 1200 6750 60
+F17 "~VPW_RX" O L 1200 6550 60
+F18 "~J1850_BUS-_TX" I L 1200 6400 60
+$EndSheet
 $EndSCHEMATC

Commit message: Added transceivers, power and voltage sense. Updated connections between complete sub groups with busses.
Parts:
- added CON1: OBD_PORT, symbol OBD_PORT
Connections:
- new net BAT_RAW: CON1.~ (BAT_RAW)
- new net CAN_HIGH: CON1.6 (CAN_HIGH)
- new net CAN_LOW: CON1.14 (CAN_LOW)
- new net GND: CON1.5 (SIG_GND)
- new net J1850_BUS+: CON1.2 (J1850_BUS+)
- new net J1850_BUS-: CON1.10 (J1850_BUS-)
- new net K_LINE: CON1.7 (K_LINE)
- new net L_LINE: CON1.15 (L_LINE)
- no-connect marks 0 -> 8
