File: GEM.sch (KiCad schematic (older format))
At the start: 1 part, among them CON1 OBD_PORT

Commit message: Added Bluetooth module and SD card
Added RN4020 and a microSD card to libraries, connected most pins. Also
added datasheets.
Changed lines of the file:
@@
 $Descr A4 11693 8268
 encoding utf-8
-Sheet 1 8
+Sheet 1 10
 Title "GEM"
 Date "Saturday, November 15, 2014"
@@
 ANALOG_IN
 $Sheet
-S 6300 900  1800 1100
+S 5650 1150 1650 950
 U 546F8CA0
 F0 "MSP430F247" 60
 F1 "MSP430F247.sch" 60
-F2 "3.3V" I L 6300 1050 60
-F3 "GND" I L 6300 1150 60
-F4 "UART_RX" I L 6300 1250 60
-F5 "UART_TX" O L 6300 1350 60
+F2 "3.3V" I L 5650 1300 60
+F3 "GND" I L 5650 1400 60
+F4 "UART_RX" I L 5650 1500 60
+F5 "UART_TX" O L 5650 1600 60
+F6 "UART_TX_BT" B L 5650 1700 60
+F7 "UART_RX_BT" B L 5650 1800 60
+F8 "WAKE_SW" O L 5650 1900 60
+F9 "CMD" O R 7300 1300 60
+F10 "WAKE_HW" O R 7300 1400 60
+F11 "SPI/PIO" O R 7300 1500 60
+F12 "SPI_SIMO" B R 7300 1600 60
+F13 "SPI_SOMI" B R 7300 1700 60
+F14 "SPI_CLK" T R 7300 1800 60
 $EndSheet
+$Sheet
+S 9650 950  1050 1350
+U 5478DA1E
+F0 "RN4020" 60
+F1 "RN4020.sch" 60
+F2 "3.3V" I L 9650 1100 60
+F3 "GND" I L 9650 1200 60
+F4 "UART_RX_BT" I L 9650 1300 60
+F5 "UART_TX_BT" O L 9650 1400 60
+F6 "WAKE_SW" I L 9650 1500 60
+F7 "CMD" I L 9650 1600 60
+F8 "WAKE_HW" I L 9650 1700 60
+F9 "SPI/PIO" I L 9650 1800 60
+F10 "BT_CNT_LED" O L 9650 1900 60
+F11 "BT_ACT_LED" O L 9650 2000 60
+$EndSheet
+$Sheet
+S 9650 4200 950  1100
+U 547A739C
+F0 "MicroSD" 60
+F1 "MicroSD.sch" 60
+F2 "~CS" I L 9650 4300 60
+F3 "3.3V" I L 9650 4400 60
+F4 "GND" I L 9650 4500 60
+F5 "SPI_SIMO" B L 9650 4600 60
+F6 "SPI_SOMI" B L 9650 4700 60
+F7 "SPI_CLK" T L 9650 4800 60
+$EndSheet
+Entry Wire Line
+	8700 1000 8800 1100
+Entry Wire Line
+	8700 1100 8800 1200
+Entry Wire Line
+	8700 1200 8800 1300
+Entry Wire Line
+	8700 1300 8800 1400
+Entry Wire Line
+	8700 1400 8800 1500
+Entry Wire Line
+	8700 1500 8800 1600
+Entry Wire Line
+	8700 1600 8800 1700
+Entry Wire Line
+	8700 1700 8800 1800
+Entry Wire Line
+	8700 1800 8800 1900
+Entry Wire Line
+	8700 1900 8800 2000
+Text Label 8900 1400 0    60   ~ 0
+UART_TX_BT
+Text Label 8900 1100 0    60   ~ 0
+3.3V
+Text Label 8900 1200 0    60   ~ 0
+GND
+Text Label 8900 1300 0    60   ~ 0
+UART_RX_BT
+Text Label 8900 1500 0    60   ~ 0
+WAKE_SW
+Text Label 8900 1600 0    60   ~ 0
+CMD
+Text Label 8900 1700 0    60   ~ 0
+WAKE_HW
+Text Label 8900 1800 0    60   ~ 0
+SPI/PIO
+Text Label 8900 1900 0    60   ~ 0
+BT_CNT_LED
+Text Label 8900 2000 0    60   ~ 0
+BT_ACT_LED
+Entry Wire Line
+	8700 4200 8800 4300
+Entry Wire Line
+	8700 4300 8800 4400
+Entry Wire Line
+	8700 4400 8800 4500
+Entry Wire Line
+	8700 4500 8800 4600
+Entry Wire Line
+	8700 4600 8800 4700
+Entry Wire Line
+	8700 4700 8800 4800
 Wire Wire Line
 	2150 1950 2450 1950
@@
 	2450 2850 2450 3100
 Wire Bus Line
-	4950 950  4950 5900
+	4950 900  4950 5900
 Wire Wire Line
 	3950 4700 4850 4700
@@
 	5900 3000 5050 3000
 Wire Bus Line
-	8700 2700 8700 4500
+	8700 900  8700 5400
 Wire Wire Line
 	7900 3000 8600 3000
@@
 Wire Wire Line
 	5050 5750 5650 5750
+Wire Wire Line
+	8800 1100 9650 1100
+Wire Wire Line
+	8800 1200 9650 1200
+Wire Wire Line
+	8800 1300 9650 1300
+Wire Wire Line
+	8800 1400 9650 1400
+Wire Wire Line
+	8800 1500 9650 1500
+Wire Wire Line
+	8800 1600 9650 1600
+Wire Wire Line
+	8800 1700 9650 1700
+Wire Wire Line
+	8800 1800 9650 1800
+Wire Wire Line
+	8800 1900 9650 1900
+Wire Wire Line
+	8800 2000 9650 2000
+Wire Wire Line
+	9650 4300 8800 4300
+Wire Wire Line
+	9650 4400 8800 4400
+Wire Wire Line
+	9650 4500 8800 4500
+Wire Wire Line
+	9650 4600 8800 4600
+Wire Wire Line
+	9650 4700 8800 4700
+Wire Wire Line
+	9650 4800 8800 4800
+Text Label 8950 4300 0    60   ~ 0
+~CS
+Text Label 8950 4400 0    60   ~ 0
+3.3V
+Text Label 8950 4500 0    60   ~ 0
+GND
+Text Label 8950 4600 0    60   ~ 0
+SPI_SIMO
+Text Label 8950 4700 0    60   ~ 0
+SPI_SOMI
+Text Label 8950 4800 0    60   ~ 0
+SPI_CLK
+Entry Wire Line
+	4950 1200 5050 1300
+Entry Wire Line
+	4950 1300 5050 1400
+Entry Wire Line
+	4950 1400 5050 1500
+Entry Wire Line
+	4950 1500 5050 1600
+Entry Wire Line
+	4950 1600 5050 1700
+Entry Wire Line
+	4950 1700 5050 1800
+Entry Wire Line
+	4950 1800 5050 1900
+Wire Wire Line
+	5050 1300 5650 1300
+Wire Wire Line
+	5050 1400 5650 1400
+Wire Wire Line
+	5050 1500 5650 1500
+Wire Wire Line
+	5050 1600 5650 1600
+Wire Wire Line
+	5050 1700 5650 1700
+Wire Wire Line
+	5050 1800 5650 1800
+Wire Wire Line
+	5050 1900 5650 1900
+Text Label 5050 1300 0    60   ~ 0
+3.3V
+Text Label 5050 1400 0    60   ~ 0
+GND
+Text Label 5050 1500 0    60   ~ 0
+UART_RX
+Text Label 5050 1600 0    60   ~ 0
+UART_TX
+Text Label 5050 1700 0    60   ~ 0
+UART_TX_BT
+Text Label 5050 1800 0    60   ~ 0
+UART_RX_BT
+Text Label 5050 1900 0    60   ~ 0
+WAKE_SW
+Entry Wire Line
+	7900 1300 8000 1400
+Entry Wire Line
+	7900 1400 8000 1500
+Entry Wire Line
+	7900 1500 8000 1600
+Entry Wire Line
+	7900 1600 8000 1700
+Entry Wire Line
+	7900 1700 8000 1800
+Entry Wire Line
+	7900 1800 8000 1900
+Wire Wire Line
+	7900 1300 7300 1300
+Wire Wire Line
+	7900 1400 7300 1400
+Wire Wire Line
+	7900 1500 7300 1500
+Wire Wire Line
+	7900 1600 7300 1600
+Wire Wire Line
+	7900 1700 7300 1700
+Wire Wire Line
+	7900 1800 7300 1800
+Text Label 7900 1300 2    60   ~ 0
+CMD
+Text Label 7900 1400 2    60   ~ 0
+WAKE_HW
+Text Label 7900 1500 2    60   ~ 0
+SPI/PIO
+Text Label 7900 1600 2    60   ~ 0
+SPI_SIMO
+Text Label 7900 1700 2    60   ~ 0
+SPI_SOMI
+Text Label 7900 1800 2    60   ~ 0
+SPI_CLK
+Wire Bus Line
+	4950 900  8000 900
+Wire Bus Line
+	8000 900  8000 2100
 $EndSCHEMATC

Commit message: Linked components to footprints, may have to switch to smaller components. Started board layout.
Changed lines of the file:
@@
 F 0 "CON1" H 1400 1000 60  0000 C CNN
 F 1 "OBD_PORT" H 650 1850 60  0000 C CNN
-F 2 "" H 1450 2300 60  0000 C CNN
+F 2 "" H 1450 2300 60  0001 C CNN
 F 3 "" H 1450 2300 60  0000 C CNN
 	1    1450 1800
@@
 F4 "UART_RX" I L 5650 1500 60
 F5 "UART_TX" O L 5650 1600 60
-F6 "UART_TX_BT" B L 5650 1700 60
-F7 "UART_RX_BT" B L 5650 1800 60
+F6 "UART_TX_BT" O L 5650 1700 60
+F7 "UART_RX_BT" I L 5650 1800 60
 F8 "WAKE_SW" O L 5650 1900 60
 F9 "CMD" O R 7300 1300 60
@@
 Entry Wire Line
 	1700 7300 1800 7200
+Text Label 1800 7100 0    60   ~ 0
+BT_CNT_LED
+Text Label 1800 7200 0    60   ~ 0
+BT_ACT_LED
 $EndSCHEMATC

Commit message: General fine tuning of schematics. Need to review JTAG and update. Added resistors to power stage. Getting prepped for BOM, need to go through item by item. Added current incomplete BOM
Changed lines of the file:
@@
 ANALOG_IN
 $Sheet
-S 5650 1150 1650 950
+S 5650 1150 1650 1350
 U 546F8CA0
 F0 "MSP430F247" 60
@@
 SPI_CLK
 $Sheet
-S 3600 800  800  400
+S 3600 800  850  800
 U 5473254D
 F0 "JTAG" 60
@@
 F3 "TCK" O L 3600 1000 60
 F4 "FUSE" O L 3600 1100 60
-F5 "TDO/TDI" B R 4400 900 60
-F6 "GND" I R 4400 1000 60
+F5 "TDO/TDI" B R 4450 900 60
+F6 "GND" I R 4450 1000 60
+F7 "TDI/VPP" I R 4450 1100 60
+F8 "TMS" I R 4450 1200 60
+F9 "TEST/VPP" I R 4450 1300 60
 $EndSheet
 Entry Wire Line
@@
 	3600 900  3250 900
 Wire Wire Line
-	4850 1000 4400 1000
-Wire Wire Line
-	4850 900  4400 900
-Wire Wire Line
 	5650 2000 5050 2000
 Wire Wire Line
@@
 Text Label 1800 7200 0    60   ~ 0
 BT_ACT_LED
+Wire Wire Line
+	4850 900  4450 900
+Wire Wire Line
+	4450 1000 4850 1000
+Wire Wire Line
+	4850 1100 4450 1100
+Entry Wire Line
+	4850 1100 4950 1200
+Entry Wire Line
+	4850 1200 4950 1300
+Entry Wire Line
+	4850 1300 4950 1400
+Wire Wire Line
+	4850 1200 4450 1200
+Wire Wire Line
+	4850 1300 4450 1300
+Text Label 4500 1100 0    60   ~ 0
+TDI/VPP
+Text Label 4500 1200 0    60   ~ 0
+TMS
+Text Label 4450 1300 0    60   ~ 0
+TEST/VPP
 $EndSCHEMATC

Commit message: Updated parts and data sheets
Changed lines of the file:
@@
 F17 "FUSE" I L 5650 2000 60
 F18 "TDO/TDI" B R 7300 1200 60
+F19 "TMS" I L 5650 2100 60
+F20 "TDI/VPP" I R 7300 2100 60
+F21 "~RST" I L 5650 2200 60
 $EndSheet
 $Sheet
@@
 F8 "TMS" I R 4450 1200 60
 F9 "TEST/VPP" I R 4450 1300 60
+F10 "~RST" I R 4450 1400 60
 $EndSheet
 Entry Wire Line
@@
 Text Label 4450 1300 0    60   ~ 0
 TEST/VPP
+Entry Wire Line
+	4950 2000 5050 2100
+Wire Wire Line
+	5050 2100 5650 2100
+Text Label 5050 2100 0    60   ~ 0
+TMS
+Entry Wire Line
+	7900 2100 8000 2200
+Wire Wire Line
+	7300 2100 7900 2100
+Text Label 7500 2100 0    60   ~ 0
+TDI/VPP
+Wire Wire Line
+	4450 1400 4850 1400
+Entry Wire Line
+	4850 1400 4950 1500
+Text Label 4550 1400 0    60   ~ 0
+~RST
+Entry Wire Line
+	4950 2100 5050 2200
+Wire Wire Line
+	5650 2200 5050 2200
 $EndSCHEMATC
