File: MCP2551.sch (KiCad schematic (older format))
At the start: 7 parts, among them U2 MCP2551

Commit message: Added transceivers, power and voltage sense. Updated connections between complete sub groups with busses.
Connections:
- no-connect marks 0 -> 1
Changed lines of the file:
@@
 $Descr A4 11693 8268
 encoding utf-8
-Sheet 3 5
+Sheet 3 7
 Title "GEM"
 Date "Saturday, November 15, 2014"
@@
 	1    0    0    -1
 $EndComp
-Text HLabel 3650 3100 0    60   Input ~ 0
+Text HLabel 3500 3100 0    60   Input ~ 0
 CAN_TX
-Text HLabel 3650 3200 0    60   Output ~ 0
+Text HLabel 3500 3200 0    60   Output ~ 0
 CAN_RX
 $Comp
@@
 	5550 3500 5550 3200
 Connection ~ 5550 3200
+NoConn ~ 4600 3350
+Wire Wire Line
+	3650 3100 3500 3100
+Wire Wire Line
+	3500 3200 3650 3200
 $EndSCHEMATC
