File: MCP2551.sch (KiCad schematic (older format))
At the start: 7 parts, among them U2 MCP2551

Commit message: Linked components to footprints, may have to switch to smaller components. Started board layout.
Parts:
- C5, C6, C7: footprint (none) -> SMD_Packages:SMD-1206
- R10, R8, R9: footprint (none) -> Resistors_SMD:R_1206_HandSoldering
- U3: renamed from U2; footprint (none) -> SMD_Packages:SOIC-8-N
Changed lines of the file:
@@
 $EndDescr
 $Comp
-L MCP2551 U2
+L MCP2551 U3
 U 1 1 546258C2
 P 4100 3200
-F 0 "U2" H 4200 2850 60  0000 C CNN
+F 0 "U3" H 4200 2850 60  0000 C CNN
 F 1 "MCP2551" H 4350 3500 60  0000 C CNN
-F 2 "" H 4100 3200 60  0000 C CNN
+F 2 "SMD_Packages:SOIC-8-N" H 4100 3200 60  0001 C CNN
 F 3 "" H 4100 3200 60  0000 C CNN
 	1    4100 3200
@@
 F 0 "R8" V 3630 3800 40  0000 C CNN
 F 1 "4.7K" V 3557 3801 40  0000 C CNN
-F 2 "" V 3480 3800 30  0000 C CNN
+F 2 "Resistors_SMD:R_1206_HandSoldering" V 3480 3800 30  0001 C CNN
 F 3 "" H 3550 3800 30  0000 C CNN
 	1    3550 3800
@@
 F 0 "C5" H 4500 2600 40  0000 L CNN
 F 1 "1U" H 4506 2415 40  0000 L CNN
-F 2 "" H 4538 2350 30  0000 C CNN
+F 2 "SMD_Packages:SMD-1206" H 4538 2350 30  0001 C CNN
 F 3 "" H 4500 2500 60  0000 C CNN
 	1    4500 2500
@@
 F 0 "R9" V 5180 3750 40  0000 C CNN
 F 1 "100" V 5107 3751 40  0000 C CNN
-F 2 "" V 5030 3750 30  0000 C CNN
+F 2 "Resistors_SMD:R_1206_HandSoldering" V 5030 3750 30  0001 C CNN
 F 3 "" H 5100 3750 30  0000 C CNN
 	1    5100 3750
@@
 F 0 "R10" V 5630 3750 40  0000 C CNN
 F 1 "100" V 5557 3751 40  0000 C CNN
-F 2 "" V 5480 3750 30  0000 C CNN
+F 2 "Resistors_SMD:R_1206_HandSoldering" V 5480 3750 30  0001 C CNN
 F 3 "" H 5550 3750 30  0000 C CNN
 	1    5550 3750
@@
 F 0 "C6" H 5100 4450 40  0000 L CNN
 F 1 "560P" H 5106 4265 40  0000 L CNN
-F 2 "" H 5138 4200 30  0000 C CNN
+F 2 "SMD_Packages:SMD-1206" H 5138 4200 30  0001 C CNN
 F 3 "" H 5100 4350 60  0000 C CNN
 	1    5100 4350
@@
 F 0 "C7" H 5550 4450 40  0000 L CNN
 F 1 "560P" H 5556 4265 40  0000 L CNN
-F 2 "" H 5588 4200 30  0000 C CNN
+F 2 "SMD_Packages:SMD-1206" H 5588 4200 30  0001 C CNN
 F 3 "" H 5550 4350 60  0000 C CNN
 	1    5550 4350

Commit message: General fine tuning of schematics. Need to review JTAG and update. Added resistors to power stage. Getting prepped for BOM, need to go through item by item. Added current incomplete BOM
Parts:
- C5, C6, C7: footprint SMD_Packages:SMD-1206 -> SMD_Packages:SMD-0805
Changed lines of the file:
@@
 F 0 "C5" H 4500 2600 40  0000 L CNN
 F 1 "1U" H 4506 2415 40  0000 L CNN
-F 2 "SMD_Packages:SMD-1206" H 4538 2350 30  0001 C CNN
+F 2 "SMD_Packages:SMD-0805" H 4538 2350 30  0001 C CNN
 F 3 "" H 4500 2500 60  0000 C CNN
 	1    4500 2500
@@
 F 0 "C6" H 5100 4450 40  0000 L CNN
 F 1 "560P" H 5106 4265 40  0000 L CNN
-F 2 "SMD_Packages:SMD-1206" H 5138 4200 30  0001 C CNN
+F 2 "SMD_Packages:SMD-0805" H 5138 4200 30  0001 C CNN
 F 3 "" H 5100 4350 60  0000 C CNN
 	1    5100 4350
@@
 F 0 "C7" H 5550 4450 40  0000 L CNN
 F 1 "560P" H 5556 4265 40  0000 L CNN
-F 2 "SMD_Packages:SMD-1206" H 5588 4200 30  0001 C CNN
+F 2 "SMD_Packages:SMD-0805" H 5588 4200 30  0001 C CNN
 F 3 "" H 5550 4350 60  0000 C CNN
 	1    5550 4350

Commit message: Updated parts and data sheets
Parts:
- C5, C6, C7: footprint SMD_Packages:SMD-0805 -> Capacitors_SMD:C_0805_HandSoldering
- R10, R8, R9: footprint Resistors_SMD:R_1206_HandSoldering -> Resistors_SMD:R_0805_HandSoldering
Changed lines of the file:
@@
 F 0 "R8" V 3630 3800 40  0000 C CNN
 F 1 "4.7K" V 3557 3801 40  0000 C CNN
-F 2 "Resistors_SMD:R_1206_HandSoldering" V 3480 3800 30  0001 C CNN
+F 2 "Resistors_SMD:R_0805_HandSoldering" V 3480 3800 30  0001 C CNN
 F 3 "" H 3550 3800 30  0000 C CNN
 	1    3550 3800
@@
 F 0 "C5" H 4500 2600 40  0000 L CNN
 F 1 "1U" H 4506 2415 40  0000 L CNN
-F 2 "SMD_Packages:SMD-0805" H 4538 2350 30  0001 C CNN
+F 2 "Capacitors_SMD:C_0805_HandSoldering" H 4538 2350 30  0001 C CNN
 F 3 "" H 4500 2500 60  0000 C CNN
 	1    4500 2500
@@
 F 0 "R9" V 5180 3750 40  0000 C CNN
 F 1 "100" V 5107 3751 40  0000 C CNN
-F 2 "Resistors_SMD:R_1206_HandSoldering" V 5030 3750 30  0001 C CNN
+F 2 "Resistors_SMD:R_0805_HandSoldering" V 5030 3750 30  0001 C CNN
 F 3 "" H 5100 3750 30  0000 C CNN
 	1    5100 3750
@@
 F 0 "R10" V 5630 3750 40  0000 C CNN
 F 1 "100" V 5557 3751 40  0000 C CNN
-F 2 "Resistors_SMD:R_1206_HandSoldering" V 5480 3750 30  0001 C CNN
+F 2 "Resistors_SMD:R_0805_HandSoldering" V 5480 3750 30  0001 C CNN
 F 3 "" H 5550 3750 30  0000 C CNN
 	1    5550 3750
@@
 F 0 "C6" H 5100 4450 40  0000 L CNN
 F 1 "560P" H 5106 4265 40  0000 L CNN
-F 2 "SMD_Packages:SMD-0805" H 5138 4200 30  0001 C CNN
+F 2 "Capacitors_SMD:C_0805_HandSoldering" H 5138 4200 30  0001 C CNN
 F 3 "" H 5100 4350 60  0000 C CNN
 	1    5100 4350
@@
 F 0 "C7" H 5550 4450 40  0000 L CNN
 F 1 "560P" H 5556 4265 40  0000 L CNN
-F 2 "SMD_Packages:SMD-0805" H 5588 4200 30  0001 C CNN
+F 2 "Capacitors_SMD:C_0805_HandSoldering" H 5588 4200 30  0001 C CNN
 F 3 "" H 5550 4350 60  0000 C CNN
 	1    5550 4350
