File: STN1110.sch (KiCad schematic (older format))
At the start: 15 parts

Commit message: Added power ports to STN1110
Parts:
- gave numbers to parts that had none: 15
Connections:
- net labels added: 3.3V, 5V_SW
- net labels removed: +3.3V, +5V
Changed lines of the file:
@@
 $EndDescr
 $Comp
-L R R?
+L R R2
 U 1 1 545FDE79
 P 4000 1900
-F 0 "R?" V 4080 1900 40  0000 C CNN
+F 0 "R2" V 4080 1900 40  0000 C CNN
 F 1 "10K" V 4007 1901 40  0000 C CNN
 F 2 "" V 3930 1900 30  0000 C CNN
@@
 $EndComp
 $Comp
-L +3.3V #PWR?
-U 1 1 545FDE7A
-P 4000 1550
-F 0 "#PWR?" H 4000 1510 30  0001 C CNN
-F 1 "+3.3V" H 4000 1660 30  0000 C CNN
-F 2 "" H 4000 1550 60  0000 C CNN
-F 3 "" H 4000 1550 60  0000 C CNN
-	1    4000 1550
-	1    0    0    -1
-$EndComp
-$Comp
-L STN1110 U?
+L STN1110 U1
 U 1 1 545FDE7B
 P 5100 3550
-F 0 "U?" H 5100 2100 60  0000 C CNN
+F 0 "U1" H 5100 2100 60  0000 C CNN
 F 1 "STN1110" H 5100 5150 60  0000 C CNN
 F 2 "" H 4900 3600 60  0000 C CNN
@@
 $EndComp
 $Comp
-L C C?
+L C C1
 U 1 1 545FDE7C
 P 2700 3550
-F 0 "C?" H 2700 3650 40  0000 L CNN
+F 0 "C1" H 2700 3650 40  0000 L CNN
 F 1 "30p" H 2706 3465 40  0000 L CNN
 F 2 "" H 2738 3400 30  0000 C CNN
@@
 $EndComp
 $Comp
-L C C?
+L C C2
 U 1 1 545FDE7D
 P 2700 4150
-F 0 "C?" H 2700 4250 40  0000 L CNN
+F 0 "C2" H 2700 4250 40  0000 L CNN
 F 1 "30p" H 2706 4065 40  0000 L CNN
 F 2 "" H 2738 4000 30  0000 C CNN
@@
 $EndComp
 $Comp
-L CRYSTAL X?
+L CRYSTAL X1
 U 1 1 545FDE7E
 P 3000 3850
-F 0 "X?" H 3000 4000 60  0000 C CNN
+F 0 "X1" H 3000 4000 60  0000 C CNN
 F 1 "16Mhz" H 3000 3700 60  0000 C CNN
 F 2 "" H 3000 3850 60  0000 C CNN
@@
 $EndComp
 $Comp
-L GND #PWR?
-U 1 1 545FDE7F
-P 2450 4250
-F 0 "#PWR?" H 2450 4250 30  0001 C CNN
-F 1 "GND" H 2450 4180 30  0001 C CNN
-F 2 "" H 2450 4250 60  0000 C CNN
-F 3 "" H 2450 4250 60  0000 C CNN
-	1    2450 4250
-	1    0    0    -1
-$EndComp
-$Comp
-L R R?
+L R R1
 U 1 1 545FDE80
 P 2250 3950
-F 0 "R?" V 2330 3950 40  0000 C CNN
+F 0 "R1" V 2330 3950 40  0000 C CNN
 F 1 "100K" V 2257 3951 40  0000 C CNN
 F 2 "" V 2180 3950 30  0000 C CNN
@@
 $EndComp
 $Comp
-L +3.3V #PWR?
-U 1 1 545FDE81
-P 2250 3600
-F 0 "#PWR?" H 2250 3560 30  0001 C CNN
-F 1 "+3.3V" H 2250 3710 30  0000 C CNN
-F 2 "" H 2250 3600 60  0000 C CNN
-F 3 "" H 2250 3600 60  0000 C CNN
-	1    2250 3600
-	1    0    0    -1
-$EndComp
-$Comp
-L C C?
+L C C3
 U 1 1 545FDE82
 P 2900 5050
-F 0 "C?" H 2900 5150 40  0000 L CNN
+F 0 "C3" H 2900 5150 40  0000 L CNN
 F 1 "1u" H 2906 4965 40  0000 L CNN
 F 2 "" H 2938 4900 30  0000 C CNN
@@
 $EndComp
 $Comp
-L GND #PWR?
-U 1 1 545FDE83
-P 2900 5350
-F 0 "#PWR?" H 2900 5350 30  0001 C CNN
-F 1 "GND" H 2900 5280 30  0001 C CNN
-F 2 "" H 2900 5350 60  0000 C CNN
-F 3 "" H 2900 5350 60  0000 C CNN
-	1    2900 5350
-	1    0    0    -1
-$EndComp
-$Comp
-L +3.3V #PWR?
-U 1 1 545FDE84
-P 2900 4750
-F 0 "#PWR?" H 2900 4710 30  0001 C CNN
-F 1 "+3.3V" H 2900 4860 30  0000 C CNN
-F 2 "" H 2900 4750 60  0000 C CNN
-F 3 "" H 2900 4750 60  0000 C CNN
-	1    2900 4750
-	1    0    0    -1
-$EndComp
-$Comp
-L C C?
+L C C4
 U 1 1 545FDE85
 P 6950 2200
-F 0 "C?" H 6950 2300 40  0000 L CNN
+F 0 "C4" H 6950 2300 40  0000 L CNN
 F 1 "1u" H 6956 2115 40  0000 L CNN
 F 2 "" H 6988 2050 30  0000 C CNN
@@
 $EndComp
 $Comp
-L R R?
+L R R5
 U 1 1 545FDE86
 P 6950 1650
-F 0 "R?" V 7030 1650 40  0000 C CNN
+F 0 "R5" V 7030 1650 40  0000 C CNN
 F 1 "10" V 6957 1651 40  0000 C CNN
 F 2 "" V 6880 1650 30  0000 C CNN
@@
 $EndComp
 $Comp
-L GND #PWR?
+L GND #PWR7
 U 1 1 545FDE87
 P 6950 2500
-F 0 "#PWR?" H 6950 2500 30  0001 C CNN
+F 0 "#PWR7" H 6950 2500 30  0001 C CNN
 F 1 "GND" H 6950 2430 30  0001 C CNN
 F 2 "" H 6950 2500 60  0000 C CNN
@@
 $EndComp
 $Comp
-L +3.3V #PWR?
-U 1 1 545FDE88
-P 6950 1300
-F 0 "#PWR?" H 6950 1260 30  0001 C CNN
-F 1 "+3.3V" H 6950 1410 30  0000 C CNN
-F 2 "" H 6950 1300 60  0000 C CNN
-F 3 "" H 6950 1300 60  0000 C CNN
-	1    6950 1300
-	1    0    0    -1
-$EndComp
-$Comp
-L R R?
+L R R6
 U 1 1 545FDE89
 P 7850 3200
-F 0 "R?" V 7930 3200 40  0000 C CNN
+F 0 "R6" V 7930 3200 40  0000 C CNN
 F 1 "100K" V 7857 3201 40  0000 C CNN
 F 2 "" V 7780 3200 30  0000 C CNN
@@
 $EndComp
 $Comp
-L JUMPER JP?
+L JUMPER JP1
 U 1 1 545FDE8A
 P 8400 3450
-F 0 "JP?" H 8400 3600 60  0000 C CNN
+F 0 "JP1" H 8400 3600 60  0000 C CNN
 F 1 "JUMPER" H 8400 3370 40  0000 C CNN
 F 2 "" H 8400 3450 60  0000 C CNN
@@
 	1    0    0    -1
 $EndComp
-$Comp
-L GND #PWR?
-U 1 1 545FDE8B
-P 8700 3600
-F 0 "#PWR?" H 8700 3600 30  0001 C CNN
-F 1 "GND" H 8700 3530 30  0001 C CNN
-F 2 "" H 8700 3600 60  0000 C CNN
-F 3 "" H 8700 3600 60  0000 C CNN
-	1    8700 3600
-	1    0    0    -1
-$EndComp
-$Comp
-L +3.3V #PWR?
-U 1 1 545FDE8C
-P 7850 2850
-F 0 "#PWR?" H 7850 2810 30  0001 C CNN
-F 1 "+3.3V" H 7850 2960 30  0000 C CNN
-F 2 "" H 7850 2850 60  0000 C CNN
-F 3 "" H 7850 2850 60  0000 C CNN
-	1    7850 2850
-	1    0    0    -1
-$EndComp
 Wire Wire Line
 	4000 1550 4000 1650
@@
 Jumper reset non-volatile memory
 $Comp
-L CP1 C?
+L CP1 10u/ESR<5
 U 1 1 545FDE8D
 P 7500 3950
-F 0 "C?" H 7550 4050 50  0000 L CNN
+F 0 "10u/ESR<5" H 7550 4050 50  0000 L CNN
 F 1 "CP1" H 7550 3850 50  0000 L CNN
 F 2 "" H 7500 3950 60  0000 C CNN
@@
 $EndComp
 $Comp
-L GND #PWR?
+L GND #PWR10
 U 1 1 545FDE8E
 P 7500 4250
-F 0 "#PWR?" H 7500 4250 30  0001 C CNN
+F 0 "#PWR10" H 7500 4250 30  0001 C CNN
 F 1 "GND" H 7500 4180 30  0001 C CNN
 F 2 "" H 7500 4250 60  0000 C CNN
@@
 11/9/14
 $Comp
-L R R?
+L R R7
 U 1 1 545FDE8F
 P 8000 4050
-F 0 "R?" V 8080 4050 40  0000 C CNN
+F 0 "R7" V 8080 4050 40  0000 C CNN
 F 1 "1K" V 8007 4051 40  0000 C CNN
 F 2 "" V 7930 4050 30  0000 C CNN
@@
 	1    0    0    -1
 $EndComp
-$Comp
-L +3.3V #PWR?
-U 1 1 545FDE90
-P 8000 3700
-F 0 "#PWR?" H 8000 3660 30  0001 C CNN
-F 1 "+3.3V" H 8000 3810 30  0000 C CNN
-F 2 "" H 8000 3700 60  0000 C CNN
-F 3 "" H 8000 3700 60  0000 C CNN
-	1    8000 3700
-	1    0    0    -1
-$EndComp
-Wire Wire Line
-	8000 3700 8000 3800
 Wire Wire Line
 	6000 4350 8150 4350
@@
 	6000 4750 6300 4750
 $Comp
-L R R?
+L R R3
 U 1 1 545FDE91
 P 6450 5050
-F 0 "R?" V 6530 5050 40  0000 C CNN
+F 0 "R3" V 6530 5050 40  0000 C CNN
 F 1 "1K" V 6457 5051 40  0000 C CNN
 F 2 "" V 6380 5050 30  0000 C CNN
@@
 $EndComp
 $Comp
-L R R?
+L R R4
 U 1 1 545FDE92
 P 6450 5350
-F 0 "R?" V 6530 5350 40  0000 C CNN
+F 0 "R4" V 6530 5350 40  0000 C CNN
 F 1 "100K" V 6457 5351 40  0000 C CNN
 F 2 "" V 6380 5350 30  0000 C CNN
@@
 	0    1    1    0
 $EndComp
-$Comp
-L +5V #PWR?
-U 1 1 545FDE93
-P 6950 4900
-F 0 "#PWR?" H 6950 4990 20  0001 C CNN
-F 1 "+5V" H 6950 4990 30  0000 C CNN
-F 2 "" H 6950 4900 60  0000 C CNN
-F 3 "" H 6950 4900 60  0000 C CNN
-	1    6950 4900
-	1    0    0    -1
-$EndComp
 Wire Wire Line
 	6100 4750 6100 5350
@@
 Connection ~ 6100 5050
 Wire Wire Line
-	6700 5350 6950 5350
-Wire Wire Line
-	6950 5350 6950 5250
+	6700 5350 7150 5350
 Text Notes 8300 4950 2    60   ~ 0
 TODO: CREATE 5V_SW POWER
@@
 Wire Wire Line
 	6000 4150 6300 4150
-$Comp
-L +3.3V #PWR?
-U 1 1 545FDE94
-P 6950 5250
-F 0 "#PWR?" H 6950 5210 30  0001 C CNN
-F 1 "+3.3V" H 6950 5360 30  0000 C CNN
-F 2 "" H 6950 5250 60  0000 C CNN
-F 3 "" H 6950 5250 60  0000 C CNN
-	1    6950 5250
-	1    0    0    -1
-$EndComp
-Wire Wire Line
-	6950 4900 6950 5050
 Wire Wire Line
 	6950 5050 6700 5050
@@
 Text HLabel 6300 2550 2    60   Output ~ 0
 ~ISO_L_TX
+Text HLabel 7150 5250 1    60   BiDi Italic 12
+3.3V
+Wire Wire Line
+	7150 5350 7150 5250
+Text HLabel 6950 5000 1    60   BiDi Italic 12
+5V_SW
+Wire Wire Line
+	6950 5050 6950 5000
+Text HLabel 2900 5350 3    60   BiDi Italic 12
+GND
+Text HLabel 2450 4250 3    60   BiDi Italic 12
+GND
+Text HLabel 2900 4750 1    60   BiDi Italic 12
+3.3V
+Text HLabel 2250 3600 1    60   BiDi Italic 12
+3.3V
+Text HLabel 8700 3600 3    60   BiDi Italic 12
+GND
+Text HLabel 8000 3750 1    60   BiDi Italic 12
+3.3V
+Wire Wire Line
+	8000 3800 8000 3750
+Text HLabel 7850 2850 1    60   BiDi Italic 12
+3.3V
+Text HLabel 6950 1300 1    60   BiDi Italic 12
+3.3V
+Text HLabel 4000 1550 1    60   BiDi Italic 12
+3.3V
 $EndSCHEMATC

Commit message: Added transceivers for J1850 and ISO
Parts:
- renumbered 10u/ESR<5 to 10u/ESR<1
Changed lines of the file:
@@
 $Descr A4 11693 8268
 encoding utf-8
-Sheet 2 4
-Title ""
-Date ""
-Rev ""
+Sheet 2 5
+Title "GEM"
+Date "Saturday, November 15, 2014"
+Rev "1"
 Comp ""
 Comment1 ""
@@
 Jumper reset non-volatile memory
 $Comp
-L CP1 10u/ESR<5
+L CP1 10u/ESR<1
 U 1 1 545FDE8D
 P 7500 3950
-F 0 "10u/ESR<5" H 7550 4050 50  0000 L CNN
+F 0 "10u/ESR<1" H 7550 4050 50  0000 L CNN
 F 1 "CP1" H 7550 3850 50  0000 L CNN
 F 2 "" H 7500 3950 60  0000 C CNN

Commit message: Added transceivers, power and voltage sense. Updated connections between complete sub groups with busses.
Changed lines of the file:
@@
 $Descr A4 11693 8268
 encoding utf-8
-Sheet 2 5
+Sheet 2 7
 Title "GEM"
 Date "Saturday, November 15, 2014"
@@
 $EndComp
 $Comp
-L GND #PWR1
-U 1 1 545FDE87
-P 6950 2500
-F 0 "#PWR1" H 6950 2500 30  0001 C CNN
-F 1 "GND" H 6950 2430 30  0001 C CNN
-F 2 "" H 6950 2500 60  0000 C CNN
-F 3 "" H 6950 2500 60  0000 C CNN
-	1    6950 2500
-	1    0    0    -1
-$EndComp
-$Comp
 L R R6
 U 1 1 545FDE89
@@
 $EndComp
 $Comp
-L GND #PWR2
+L GND #PWR01
 U 1 1 545FDE8E
 P 7500 4250
-F 0 "#PWR2" H 7500 4250 30  0001 C CNN
+F 0 "#PWR01" H 7500 4250 30  0001 C CNN
 F 1 "GND" H 7500 4180 30  0001 C CNN
 F 2 "" H 7500 4250 60  0000 C CNN
@@
 Text HLabel 4000 1550 1    60   BiDi Italic 12
 3.3V
+Text HLabel 6950 2500 3    60   Input ~ 0
+GND
 $EndSCHEMATC
