File: STN1110.sch (KiCad schematic (older format))
At the start: 15 parts, among them U1 STN1110, X1 16Mhz

Commit message: Linked components to footprints, may have to switch to smaller components. Started board layout.
Parts:
- C1, C2, C3, C4: footprint (none) -> SMD_Packages:SMD-1206
- R1, R2, R3, R4, R5, R6, R7: footprint (none) -> Resistors_SMD:R_1206_HandSoldering
- U1: footprint (none) -> SMD_Packages:SOIC-28
- U2: renamed from 10u/ESR<1; value CP1 -> 10U ESR<5; footprint (none) -> Capacitors_Tantalum_SMD:TantalC_SizeD_EIA-7343_Wave
- X1: footprint (none) -> Crystals:Crystal_HC49-SD_SMD
Other:
- note removed: "TODO: CREATE 5V_SW POWER"
Changed lines of the file:
@@
 F 0 "R2" V 4080 1900 40  0000 C CNN
 F 1 "10K" V 4007 1901 40  0000 C CNN
-F 2 "" V 3930 1900 30  0000 C CNN
+F 2 "Resistors_SMD:R_1206_HandSoldering" V 3930 1900 30  0001 C CNN
 F 3 "" H 4000 1900 30  0000 C CNN
 	1    4000 1900
@@
 F 0 "U1" H 5100 2100 60  0000 C CNN
 F 1 "STN1110" H 5100 5150 60  0000 C CNN
-F 2 "" H 4900 3600 60  0000 C CNN
+F 2 "SMD_Packages:SOIC-28" H 4900 3600 60  0001 C CNN
 F 3 "" H 4900 3600 60  0000 C CNN
 	1    5100 3550
@@
 F 0 "C1" H 2700 3650 40  0000 L CNN
 F 1 "30p" H 2706 3465 40  0000 L CNN
-F 2 "" H 2738 3400 30  0000 C CNN
+F 2 "SMD_Packages:SMD-1206" H 2738 3400 30  0001 C CNN
 F 3 "" H 2700 3550 60  0000 C CNN
 	1    2700 3550
@@
 F 0 "C2" H 2700 4250 40  0000 L CNN
 F 1 "30p" H 2706 4065 40  0000 L CNN
-F 2 "" H 2738 4000 30  0000 C CNN
+F 2 "SMD_Packages:SMD-1206" H 2738 4000 30  0001 C CNN
 F 3 "" H 2700 4150 60  0000 C CNN
 	1    2700 4150
@@
 F 0 "X1" H 3000 4000 60  0000 C CNN
 F 1 "16Mhz" H 3000 3700 60  0000 C CNN
-F 2 "" H 3000 3850 60  0000 C CNN
+F 2 "Crystals:Crystal_HC49-SD_SMD" H 3000 3850 60  0001 C CNN
 F 3 "" H 3000 3850 60  0000 C CNN
 	1    3000 3850
@@
 F 0 "R1" V 2330 3950 40  0000 C CNN
 F 1 "100K" V 2257 3951 40  0000 C CNN
-F 2 "" V 2180 3950 30  0000 C CNN
+F 2 "Resistors_SMD:R_1206_HandSoldering" V 2180 3950 30  0001 C CNN
 F 3 "" H 2250 3950 30  0000 C CNN
 	1    2250 3950
@@
 F 0 "C3" H 2900 5150 40  0000 L CNN
 F 1 "1u" H 2906 4965 40  0000 L CNN
-F 2 "" H 2938 4900 30  0000 C CNN
+F 2 "SMD_Packages:SMD-1206" H 2938 4900 30  0001 C CNN
 F 3 "" H 2900 5050 60  0000 C CNN
 	1    2900 5050
@@
 F 0 "C4" H 6950 2300 40  0000 L CNN
 F 1 "1u" H 6956 2115 40  0000 L CNN
-F 2 "" H 6988 2050 30  0000 C CNN
+F 2 "SMD_Packages:SMD-1206" H 6988 2050 30  0001 C CNN
 F 3 "" H 6950 2200 60  0000 C CNN
 	1    6950 2200
@@
 F 0 "R5" V 7030 1650 40  0000 C CNN
 F 1 "10" V 6957 1651 40  0000 C CNN
-F 2 "" V 6880 1650 30  0000 C CNN
+F 2 "Resistors_SMD:R_1206_HandSoldering" V 6880 1650 30  0001 C CNN
 F 3 "" H 6950 1650 30  0000 C CNN
 	1    6950 1650
@@
 F 0 "R6" V 7930 3200 40  0000 C CNN
 F 1 "100K" V 7857 3201 40  0000 C CNN
-F 2 "" V 7780 3200 30  0000 C CNN
+F 2 "Resistors_SMD:R_1206_HandSoldering" V 7780 3200 30  0001 C CNN
 F 3 "" H 7850 3200 30  0000 C CNN
 	1    7850 3200
@@
 F 0 "JP1" H 8400 3600 60  0000 C CNN
 F 1 "JUMPER" H 8400 3370 40  0000 C CNN
-F 2 "" H 8400 3450 60  0000 C CNN
+F 2 "" H 8400 3450 60  0001 C CNN
 F 3 "" H 8400 3450 60  0000 C CNN
 	1    8400 3450
@@
 Jumper reset non-volatile memory
 $Comp
-L CP1 10u/ESR<1
+L CP1 U2
 U 1 1 545FDE8D
 P 7500 3950
-F 0 "10u/ESR<1" H 7550 4050 50  0000 L CNN
-F 1 "CP1" H 7550 3850 50  0000 L CNN
-F 2 "" H 7500 3950 60  0000 C CNN
+F 0 "U2" H 7550 4050 50  0000 L CNN
+F 1 "10U ESR<5" H 7550 3850 50  0000 L CNN
+F 2 "Capacitors_Tantalum_SMD:TantalC_SizeD_EIA-7343_Wave" H 7500 3950 60  0001 C CNN
 F 3 "" H 7500 3950 60  0000 C CNN
 	1    7500 3950
-	1    0    0    -1
-$EndComp
-$Comp
-L GND #PWR01
-U 1 1 545FDE8E
-P 7500 4250
-F 0 "#PWR01" H 7500 4250 30  0001 C CNN
-F 1 "GND" H 7500 4180 30  0001 C CNN
-F 2 "" H 7500 4250 60  0000 C CNN
-F 3 "" H 7500 4250 60  0000 C CNN
-	1    7500 4250
 	1    0    0    -1
 $EndComp
@@
 F 0 "R7" V 8080 4050 40  0000 C CNN
 F 1 "1K" V 8007 4051 40  0000 C CNN
-F 2 "" V 7930 4050 30  0000 C CNN
+F 2 "Resistors_SMD:R_1206_HandSoldering" V 7930 4050 30  0001 C CNN
 F 3 "" H 8000 4050 30  0000 C CNN
 	1    8000 4050
@@
 F 0 "R3" V 6530 5050 40  0000 C CNN
 F 1 "1K" V 6457 5051 40  0000 C CNN
-F 2 "" V 6380 5050 30  0000 C CNN
+F 2 "Resistors_SMD:R_1206_HandSoldering" V 6380 5050 30  0001 C CNN
 F 3 "" H 6450 5050 30  0000 C CNN
 	1    6450 5050
@@
 F 0 "R4" V 6530 5350 40  0000 C CNN
 F 1 "100K" V 6457 5351 40  0000 C CNN
-F 2 "" V 6380 5350 30  0000 C CNN
+F 2 "Resistors_SMD:R_1206_HandSoldering" V 6380 5350 30  0001 C CNN
 F 3 "" H 6450 5350 30  0000 C CNN
 	1    6450 5350
@@
 Wire Wire Line
 	6700 5350 7150 5350
-Text Notes 8300 4950 2    60   ~ 0
-TODO: CREATE 5V_SW POWER
 Wire Wire Line
 	6000 2950 6300 2950
@@
 Text HLabel 6950 2500 3    60   Input ~ 0
 GND
+Text HLabel 7500 4250 0    60   Input ~ 0
+GND
 $EndSCHEMATC

Commit message: General fine tuning of schematics. Need to review JTAG and update. Added resistors to power stage. Getting prepped for BOM, need to go through item by item. Added current incomplete BOM
Parts:
- removed R4: 100K, Resistors_SMD:R_1206_HandSoldering, symbol R
- C1, C2, C3, C4: footprint SMD_Packages:SMD-1206 -> SMD_Packages:SMD-0805
Connections:
- net 3.3V: no longer U1.14 (CAN_RX)
- new net CAN_RX: U1.14 (CAN_RX)
Changed lines of the file:
@@
 F 0 "C1" H 2700 3650 40  0000 L CNN
 F 1 "30p" H 2706 3465 40  0000 L CNN
-F 2 "SMD_Packages:SMD-1206" H 2738 3400 30  0001 C CNN
+F 2 "SMD_Packages:SMD-0805" H 2738 3400 30  0001 C CNN
 F 3 "" H 2700 3550 60  0000 C CNN
 	1    2700 3550
@@
 F 0 "C2" H 2700 4250 40  0000 L CNN
 F 1 "30p" H 2706 4065 40  0000 L CNN
-F 2 "SMD_Packages:SMD-1206" H 2738 4000 30  0001 C CNN
+F 2 "SMD_Packages:SMD-0805" H 2738 4000 30  0001 C CNN
 F 3 "" H 2700 4150 60  0000 C CNN
 	1    2700 4150
@@
 F 0 "C3" H 2900 5150 40  0000 L CNN
 F 1 "1u" H 2906 4965 40  0000 L CNN
-F 2 "SMD_Packages:SMD-1206" H 2938 4900 30  0001 C CNN
+F 2 "SMD_Packages:SMD-0805" H 2938 4900 30  0001 C CNN
 F 3 "" H 2900 5050 60  0000 C CNN
 	1    2900 5050
@@
 F 0 "C4" H 6950 2300 40  0000 L CNN
 F 1 "1u" H 6956 2115 40  0000 L CNN
-F 2 "SMD_Packages:SMD-1206" H 6988 2050 30  0001 C CNN
+F 2 "SMD_Packages:SMD-0805" H 6988 2050 30  0001 C CNN
 F 3 "" H 6950 2200 60  0000 C CNN
 	1    6950 2200
@@
 	4250 4550 3250 4550
 Wire Wire Line
-	3250 4550 3250 5100
-Wire Wire Line
-	3250 5100 4100 5100
-Wire Wire Line
-	4100 5100 4100 4750
-Connection ~ 4100 4750
-Wire Wire Line
 	2900 4750 2900 4850
 Wire Wire Line
@@
 	3250 4800 2900 4800
 Connection ~ 2900 4800
-Connection ~ 3250 4800
 Wire Wire Line
 	6950 1300 6950 1400
@@
 	0    1    1    0
 $EndComp
-$Comp
-L R R4
-U 1 1 545FDE92
-P 6450 5350
-F 0 "R4" V 6530 5350 40  0000 C CNN
-F 1 "100K" V 6457 5351 40  0000 C CNN
-F 2 "Resistors_SMD:R_1206_HandSoldering" V 6380 5350 30  0001 C CNN
-F 3 "" H 6450 5350 30  0000 C CNN
-	1    6450 5350
-	0    1    1    0
-$EndComp
-Wire Wire Line
-	6100 4750 6100 5350
 Wire Wire Line
 	6100 5050 6200 5050
-Connection ~ 6100 4750
-Wire Wire Line
-	6100 5350 6200 5350
-Connection ~ 6100 5050
-Wire Wire Line
-	6700 5350 7150 5350
 Wire Wire Line
 	6000 2950 6300 2950
@@
 Text HLabel 6300 2550 2    60   Output ~ 0
 ~ISO_L_TX
-Text HLabel 7150 5250 1    60   BiDi Italic 12
-3.3V
-Wire Wire Line
-	7150 5350 7150 5250
 Text HLabel 6950 5000 1    60   BiDi Italic 12
 5V_SW
@@
 Text HLabel 7500 4250 0    60   Input ~ 0
 GND
+Wire Wire Line
+	3250 4550 3250 4800
+Wire Wire Line
+	6100 5050 6100 4750
+Connection ~ 6100 4750
 $EndSCHEMATC

Commit message: Updated parts and data sheets
Parts:
- C1, C2: value 30p -> 30P; footprint SMD_Packages:SMD-0805 -> Capacitors_SMD:C_0805_HandSoldering; Part Number (none) -> GRM1885C1H300JA01D
- C3, C4: footprint SMD_Packages:SMD-0805 -> Capacitors_SMD:C_0805_HandSoldering
- JP1: footprint (none) -> Connect:TESTPOINT
- R1, R2, R3, R5, R6, R7: footprint Resistors_SMD:R_1206_HandSoldering -> Resistors_SMD:R_0805_HandSoldering
- U2: footprint Capacitors_Tantalum_SMD:TantalC_SizeD_EIA-7343_Wave -> (none); Part Number (none) -> TPSR106K006R1500
- X1: footprint Crystals:Crystal_HC49-SD_SMD -> (none); Part Number (none) -> 403C11E16M00000
Changed lines of the file:
@@
 F 0 "R2" V 4080 1900 40  0000 C CNN
 F 1 "10K" V 4007 1901 40  0000 C CNN
-F 2 "Resistors_SMD:R_1206_HandSoldering" V 3930 1900 30  0001 C CNN
+F 2 "Resistors_SMD:R_0805_HandSoldering" V 3930 1900 30  0001 C CNN
 F 3 "" H 4000 1900 30  0000 C CNN
 	1    4000 1900
@@
 P 2700 3550
 F 0 "C1" H 2700 3650 40  0000 L CNN
-F 1 "30p" H 2706 3465 40  0000 L CNN
-F 2 "SMD_Packages:SMD-0805" H 2738 3400 30  0001 C CNN
+F 1 "30P" H 2706 3465 40  0000 L CNN
+F 2 "Capacitors_SMD:C_0805_HandSoldering" H 2738 3400 30  0001 C CNN
 F 3 "" H 2700 3550 60  0000 C CNN
+F 4 "GRM1885C1H300JA01D" H 2700 3550 60  0001 C CNN "Part Number"
 	1    2700 3550
 	0    1    1    0
@@
 P 2700 4150
 F 0 "C2" H 2700 4250 40  0000 L CNN
-F 1 "30p" H 2706 4065 40  0000 L CNN
-F 2 "SMD_Packages:SMD-0805" H 2738 4000 30  0001 C CNN
+F 1 "30P" H 2706 4065 40  0000 L CNN
+F 2 "Capacitors_SMD:C_0805_HandSoldering" H 2738 4000 30  0001 C CNN
 F 3 "" H 2700 4150 60  0000 C CNN
+F 4 "GRM1885C1H300JA01D" H 2700 4150 60  0001 C CNN "Part Number"
 	1    2700 4150
 	0    1    1    0
@@
 F 0 "X1" H 3000 4000 60  0000 C CNN
 F 1 "16Mhz" H 3000 3700 60  0000 C CNN
-F 2 "Crystals:Crystal_HC49-SD_SMD" H 3000 3850 60  0001 C CNN
+F 2 "" H 3000 3850 60  0001 C CNN
 F 3 "" H 3000 3850 60  0000 C CNN
+F 4 "403C11E16M00000" H 3000 3850 60  0001 C CNN "Part Number"
 	1    3000 3850
 	0    1    1    0
@@
 F 0 "R1" V 2330 3950 40  0000 C CNN
 F 1 "100K" V 2257 3951 40  0000 C CNN
-F 2 "Resistors_SMD:R_1206_HandSoldering" V 2180 3950 30  0001 C CNN
+F 2 "Resistors_SMD:R_0805_HandSoldering" V 2180 3950 30  0001 C CNN
 F 3 "" H 2250 3950 30  0000 C CNN
 	1    2250 3950
@@
 F 0 "C3" H 2900 5150 40  0000 L CNN
 F 1 "1u" H 2906 4965 40  0000 L CNN
-F 2 "SMD_Packages:SMD-0805" H 2938 4900 30  0001 C CNN
+F 2 "Capacitors_SMD:C_0805_HandSoldering" H 2938 4900 30  0001 C CNN
 F 3 "" H 2900 5050 60  0000 C CNN
 	1    2900 5050
@@
 F 0 "C4" H 6950 2300 40  0000 L CNN
 F 1 "1u" H 6956 2115 40  0000 L CNN
-F 2 "SMD_Packages:SMD-0805" H 6988 2050 30  0001 C CNN
+F 2 "Capacitors_SMD:C_0805_HandSoldering" H 6988 2050 30  0001 C CNN
 F 3 "" H 6950 2200 60  0000 C CNN
 	1    6950 2200
@@
 F 0 "R5" V 7030 1650 40  0000 C CNN
 F 1 "10" V 6957 1651 40  0000 C CNN
-F 2 "Resistors_SMD:R_1206_HandSoldering" V 6880 1650 30  0001 C CNN
+F 2 "Resistors_SMD:R_0805_HandSoldering" V 6880 1650 30  0001 C CNN
 F 3 "" H 6950 1650 30  0000 C CNN
 	1    6950 1650
@@
 F 0 "R6" V 7930 3200 40  0000 C CNN
 F 1 "100K" V 7857 3201 40  0000 C CNN
-F 2 "Resistors_SMD:R_1206_HandSoldering" V 7780 3200 30  0001 C CNN
+F 2 "Resistors_SMD:R_0805_HandSoldering" V 7780 3200 30  0001 C CNN
 F 3 "" H 7850 3200 30  0000 C CNN
 	1    7850 3200
@@
 F 0 "JP1" H 8400 3600 60  0000 C CNN
 F 1 "JUMPER" H 8400 3370 40  0000 C CNN
-F 2 "" H 8400 3450 60  0001 C CNN
+F 2 "Connect:TESTPOINT" H 8400 3450 60  0001 C CNN
 F 3 "" H 8400 3450 60  0000 C CNN
 	1    8400 3450
@@
 F 0 "U2" H 7550 4050 50  0000 L CNN
 F 1 "10U ESR<5" H 7550 3850 50  0000 L CNN
-F 2 "Capacitors_Tantalum_SMD:TantalC_SizeD_EIA-7343_Wave" H 7500 3950 60  0001 C CNN
+F 2 "" H 7500 3950 60  0001 C CNN
 F 3 "" H 7500 3950 60  0000 C CNN
+F 4 "TPSR106K006R1500" H 7500 3950 60  0001 C CNN "Part Number"
 	1    7500 3950
 	1    0    0    -1
@@
 F 0 "R7" V 8080 4050 40  0000 C CNN
 F 1 "1K" V 8007 4051 40  0000 C CNN
-F 2 "Resistors_SMD:R_1206_HandSoldering" V 7930 4050 30  0001 C CNN
+F 2 "Resistors_SMD:R_0805_HandSoldering" V 7930 4050 30  0001 C CNN
 F 3 "" H 8000 4050 30  0000 C CNN
 	1    8000 4050
@@
 F 0 "R3" V 6530 5050 40  0000 C CNN
 F 1 "1K" V 6457 5051 40  0000 C CNN
-F 2 "Resistors_SMD:R_1206_HandSoldering" V 6380 5050 30  0001 C CNN
+F 2 "Resistors_SMD:R_0805_HandSoldering" V 6380 5050 30  0001 C CNN
 F 3 "" H 6450 5050 30  0000 C CNN
 	1    6450 5050
