File: transceivers.sch (KiCad schematic (older format))
At the start: 36 parts, among them Q1 BC817-40, Q2 BC817-40, Q3 BSS138, Q4 MMBT3646, Q5 MMBT3646, Q6 MMBT3640, U3 LM339, U4 LM317AEMP

Commit message: Linked components to footprints, may have to switch to smaller components. Started board layout.
Parts:
- C8: footprint (none) -> SMD_Packages:SMD-1206
- D7: renamed from D5; footprint (none) -> Diodes_ThroughHole:Diode_DO-35_SOD27_Horizontal_RM10
- D8: renamed from D6; footprint (none) -> Diodes_ThroughHole:Diode_DO-35_SOD27_Horizontal_RM10
- D9: renamed from D7; footprint (none) -> Diodes_ThroughHole:Diode_DO-35_SOD27_Horizontal_RM10
- Q1, Q2, Q3: footprint SOT-23 -> SMD_Packages:SOT-23
- Q4, Q5, Q6: footprint (none) -> SMD_Packages:SOT-23
- R17: renamed from R15; footprint (none) -> Resistors_SMD:R_1206_HandSoldering
- R18: renamed from R16; footprint (none) -> Resistors_SMD:R_1206_HandSoldering
- R19: renamed from R17; footprint (none) -> Resistors_SMD:R_1206_HandSoldering
- R20: renamed from R18; footprint (none) -> Resistors_SMD:R_1206_HandSoldering
- R21: renamed from R19; footprint (none) -> Resistors_SMD:R_1206_HandSoldering
- R22: renamed from R20; footprint (none) -> Resistors_SMD:R_1206_HandSoldering
- R23: renamed from R21; footprint (none) -> Resistors_SMD:R_1206_HandSoldering
- R24: renamed from R22; footprint (none) -> Resistors_SMD:R_1206_HandSoldering
- R25: renamed from R23; footprint (none) -> Resistors_SMD:R_1206_HandSoldering
- R26: renamed from R24; footprint (none) -> Resistors_SMD:R_1206_HandSoldering
- R27: renamed from R25; footprint (none) -> Resistors_SMD:R_1206_HandSoldering
- R28: renamed from R26; footprint (none) -> Resistors_SMD:R_1206_HandSoldering
- R29: renamed from R27; footprint (none) -> Resistors_SMD:R_1206_HandSoldering
- R30: renamed from R28; footprint (none) -> Resistors_SMD:R_1206_HandSoldering
- R31: renamed from R29; footprint (none) -> Resistors_SMD:R_1206_HandSoldering
- R32: renamed from R30; footprint (none) -> Resistors_SMD:R_1206_HandSoldering
- R33: renamed from R31; footprint (none) -> Resistors_SMD:R_1206_HandSoldering
- R34: renamed from R32; footprint (none) -> Resistors_SMD:R_1206_HandSoldering
- R35: renamed from R33; footprint (none) -> Resistors_SMD:R_1206_HandSoldering
- R36: renamed from R34; value R -> 10K; footprint (none) -> Resistors_SMD:R_1206_HandSoldering
- R37: renamed from R35; value R -> 10K; footprint (none) -> Resistors_SMD:R_1206_HandSoldering
- R38: renamed from R36; footprint (none) -> Resistors_SMD:R_1206_HandSoldering
- R39: renamed from R37; footprint (none) -> Resistors_SMD:R_1206_HandSoldering
- R40: renamed from R38; value R -> 10K; footprint (none) -> Resistors_SMD:R_1206_HandSoldering
- U4: renamed from U3; footprint (none) -> SMD_Packages:SOIC-14_N
- U5: renamed from U4; footprint SOT-223 -> SMD_Packages:SOT-223

Commit message: General fine tuning of schematics. Need to review JTAG and update. Added resistors to power stage. Getting prepped for BOM, need to go through item by item. Added current incomplete BOM
Parts:
- C8: footprint SMD_Packages:SMD-1206 -> SMD_Packages:SMD-0805
Connections:
- net at R31.1, R32.1, U5.2 (OUT): now also Q6.1 (E); no longer Q6.3 (C)
- net at D8.1 (A): now also Q6.3 (C); no longer Q6.1 (E)
Changed lines of the file:
@@
 F 0 "C8" H 6000 1900 40  0000 L CNN
 F 1 "0.1U" H 6006 1715 40  0000 L CNN
-F 2 "SMD_Packages:SMD-1206" H 6038 1650 30  0001 C CNN
+F 2 "SMD_Packages:SMD-0805" H 6038 1650 30  0001 C CNN
 F 3 "" H 6000 1800 60  0000 C CNN
 	1    6000 1800
@@
 F 3 "" H 7350 3500 60  0000 C CNN
 	1    7350 3500
-	1    0    0    -1
+	1    0    0    1
 $EndComp
 $Comp

Commit message: Updated parts and data sheets
Parts:
- removed Q4, Q5: MMBT3646, SMD_Packages:SOT-23, symbol NPN
- removed Q6: MMBT3640, SMD_Packages:SOT-23, symbol PNP
- added Q4: MMBT3646, Transistors_SMD:sot23, symbol MMBT3646
- added Q5: MMBT2222, Transistors_SMD:sot23, symbol BC817-40
- added Q6: MMBT3640, Transistors_SMD:sot23, symbol MMBT3640
- C8: footprint SMD_Packages:SMD-0805 -> Capacitors_SMD:C_0805_HandSoldering
- D7, D8, D9: footprint Diodes_ThroughHole:Diode_DO-35_SOD27_Horizontal_RM10 -> (none)
- Q1, Q2: value BC817-40 -> MMBT2222; footprint SMD_Packages:SOT-23 -> Transistors_SMD:sot23
- Q3: footprint SMD_Packages:SOT-23 -> (none)
- R17, R18, R19, R20, R21, R22, R23, R24, R25, R26, R27, R28, R29, R30, R31, R32, R33, R34, R35, R36, R37, R38, R39, R40: footprint Resistors_SMD:R_1206_HandSoldering -> Resistors_SMD:R_0805_HandSoldering
Connections:
- net GND: now also Q4.2 (E), Q5.2 (E)
- net J1850_BUS-: now also Q5.3 (C)
- net at R31.1, R32.1, U5.2 (OUT): now also Q6.3 (C)
- net at R29.1, R31.2: now also Q6.1 (B)
- net at D8.1 (A): now also Q6.2 (E)
- net at R29.2: now also Q4.3 (C)
- net at R25.1: now also Q4.1 (B)
- net at R27.1: now also Q5.1 (B)
