File: MSP430F247.sch (KiCad schematic (older format))
At the start: 3 parts, among them U7 MSP430F247

Commit message: Footprints
Take 2 on setting up the folder structure to work on footprints.
Parts:
- U7: footprint (none) -> GEM_PCB:LQFP-64_10x10mm_Pitch0.5mm
Changed lines of the file:
@@
 F 0 "U7" H 5400 3980 30  0000 C CNN
 F 1 "MSP430F247" H 5400 3920 30  0000 C CNN
-F 2 "" H 5400 3950 60  0000 C CNN
+F 2 "GEM_PCB:LQFP-64_10x10mm_Pitch0.5mm" H 5400 6150 60  0000 C CNN
 F 3 "" H 5400 3950 60  0000 C CNN
 	1    5400 3950
