File: MSP430F247.sch (KiCad schematic (older format))
At the start: 1 part

Commit message: Added JTAG interface
Spy Bi-Wire JTAG interface. Fixed some unused pins.
Parts:
- added 0.1: C, symbol C
- added 10: CP1, symbol CP1
- gave numbers to parts that had none: 1
Connections:
- net 3.3V: now also U7.58 (RST/NMI), 0.1.1, 10.1
- net GND: now also 0.1.2, 10.2
- net ~CS: now reaches U7.44 (P5.0/UCB1STE/UCA1CLK)
- net TDO/TDI: now reaches U7.54 (TDO/TDI)
- net FUSE: now reaches U7.55 (TDI/TCLK)
- net TCK: now reaches U7.57 (TCK)
- no-connect marks 49 -> 44
Changed lines of the file:
@@
 $Descr A4 11693 8268
 encoding utf-8
-Sheet 8 10
+Sheet 8 11
 Title ""
 Date ""
@@
 $EndDescr
 $Comp
-L MSP430F247 U?
+L MSP430F247 U7
 U 1 1 547269CD
 P 5400 3950
-F 0 "U?" H 5400 3980 30  0000 C CNN
+F 0 "U7" H 5400 3980 30  0000 C CNN
 F 1 "MSP430F247" H 5400 3920 30  0000 C CNN
 F 2 "" H 5400 3950 60  0000 C CNN
@@
 	1    0    0    -1
 $EndComp
-Text HLabel 3500 3200 0    60   Input ~ 0
+Text HLabel 2000 3200 0    60   Input ~ 0
 3.3V
 Text HLabel 4750 2400 1    60   Input ~ 0
@@
 Text HLabel 7350 3300 2    60   3State ~ 0
 SPI_CLK
-Wire Wire Line
-	4150 3200 3500 3200
-Wire Wire Line
-	4650 2700 4650 2500
-Wire Wire Line
-	4650 2500 3600 2500
-Wire Wire Line
-	3600 2500 3600 3200
-Connection ~ 3600 3200
-Wire Wire Line
-	4750 2400 4750 2700
-Wire Wire Line
-	4850 2700 4850 2500
-Wire Wire Line
-	4850 2500 4750 2500
-Connection ~ 4750 2500
-Wire Wire Line
-	6150 5800 6150 5200
-Wire Wire Line
-	7350 4700 6650 4700
-Wire Wire Line
-	6650 4600 7350 4600
-Wire Wire Line
-	7350 4500 6650 4500
-Wire Wire Line
-	5050 2700 5050 2500
-Wire Wire Line
-	4950 2700 4950 2500
-Wire Wire Line
-	4150 3300 3600 3300
-Wire Wire Line
-	4150 3400 3600 3400
-Wire Wire Line
-	7350 3500 6650 3500
-Wire Wire Line
-	7350 3400 6650 3400
-Wire Wire Line
-	7350 3300 6650 3300
 NoConn ~ 4150 3500
 NoConn ~ 4150 3600
@@
 NoConn ~ 6650 3800
 NoConn ~ 6650 3700
-NoConn ~ 6650 3600
 NoConn ~ 6650 3200
 NoConn ~ 6150 2700
@@
 NoConn ~ 4150 4000
 NoConn ~ 4150 3900
-NoConn ~ 5350 2700
 NoConn ~ 5450 2700
-NoConn ~ 5550 2700
-NoConn ~ 5650 2700
 NoConn ~ 5750 2700
 NoConn ~ 5850 2700
-NoConn ~ 5250 2700
 NoConn ~ 4150 3800
 NoConn ~ 4150 4100
 NoConn ~ 4150 4200
+Text HLabel 7350 3600 2    60   Output ~ 0
+~CS
+$Comp
+L CP1 10
+U 1 1 5473ADF7
+P 2200 3400
+F 0 "10" H 2250 3500 50  0000 L CNN
+F 1 "CP1" H 2250 3300 50  0000 L CNN
+F 2 "" H 2200 3400 60  0000 C CNN
+F 3 "" H 2200 3400 60  0000 C CNN
+	1    2200 3400
+	1    0    0    -1
+$EndComp
+$Comp
+L C 0.1
+U 1 1 5473B485
+P 2550 3400
+F 0 "0.1" H 2550 3500 40  0000 L CNN
+F 1 "C" H 2556 3315 40  0000 L CNN
+F 2 "" H 2588 3250 30  0000 C CNN
+F 3 "" H 2550 3400 60  0000 C CNN
+	1    2550 3400
+	1    0    0    -1
+$EndComp
+Text HLabel 2200 3900 3    60   Input ~ 0
+GND
+Text HLabel 2550 3900 3    60   Input ~ 0
+GND
+Wire Wire Line
+	4650 2700 4650 2500
+Wire Wire Line
+	4750 2400 4750 2700
+Wire Wire Line
+	4850 2700 4850 2500
+Wire Wire Line
+	4850 2500 4750 2500
+Connection ~ 4750 2500
+Wire Wire Line
+	6150 5800 6150 5200
+Wire Wire Line
+	7350 4700 6650 4700
+Wire Wire Line
+	6650 4600 7350 4600
+Wire Wire Line
+	7350 4500 6650 4500
+Wire Wire Line
+	5050 2700 5050 2500
+Wire Wire Line
+	4950 2700 4950 2500
+Wire Wire Line
+	4150 3300 3600 3300
+Wire Wire Line
+	4150 3400 3600 3400
+Wire Wire Line
+	7350 3500 6650 3500
+Wire Wire Line
+	7350 3400 6650 3400
+Wire Wire Line
+	7350 3300 6650 3300
+Wire Wire Line
+	6650 3600 7350 3600
+Wire Wire Line
+	2000 3200 4150 3200
+Connection ~ 2200 3200
+Connection ~ 2550 3200
+Wire Wire Line
+	3600 3200 3600 2500
+Wire Wire Line
+	3600 2500 4650 2500
+Connection ~ 3600 3200
+Wire Wire Line
+	2200 3600 2200 3900
+Wire Wire Line
+	2550 3600 2550 3900
+Wire Wire Line
+	5250 2700 5250 2500
+Text HLabel 5250 2500 1    60   Input ~ 0
+3.3V
+Text HLabel 5350 2500 1    60   Input ~ 0
+TCK
+Wire Wire Line
+	5350 2500 5350 2700
+Text HLabel 5550 2500 1    60   Input ~ 0
+FUSE
+Wire Wire Line
+	5550 2500 5550 2700
+Text HLabel 5650 2500 1    60   BiDi ~ 0
+TDO/TDI
+Wire Wire Line
+	5650 2500 5650 2700
 $EndSCHEMATC

Commit message: Linked components to footprints, may have to switch to smaller components. Started board layout.
Parts:
- U10: renamed from 0.1; footprint (none) -> Capacitors_SMD:C_1206_HandSoldering
- U11: renamed from U7; footprint (none) -> SMD_Packages:TQFP-64
- U9: renamed from 10; footprint (none) -> Capacitors_SMD:C_1206_HandSoldering
Connections:
- net UART_RX: now also U11.32 (P3.4/UCA0TXD/UCA0SIMO); no longer U11.33 (P3.5/UCA0RXD/UCA0SOMI)
- net UART_RX_BT: now also U11.34 (P3.6/UCA1TXD/UCA1SIMO_); no longer U11.35 (P3.7/UCA1RXD/UCA1SOMI)
- net UART_TX: now also U11.33 (P3.5/UCA0RXD/UCA0SOMI); no longer U11.32 (P3.4/UCA0TXD/UCA0SIMO)
- net UART_TX_BT: now also U11.35 (P3.7/UCA1RXD/UCA1SOMI); no longer U11.34 (P3.6/UCA1TXD/UCA1SIMO_)
Changed lines of the file:
@@
 $EndDescr
 $Comp
-L MSP430F247 U7
+L MSP430F247 U11
 U 1 1 547269CD
 P 5400 3950
-F 0 "U7" H 5400 3980 30  0000 C CNN
+F 0 "U11" H 5400 3980 30  0000 C CNN
 F 1 "MSP430F247" H 5400 3920 30  0000 C CNN
-F 2 "" H 5400 3950 60  0000 C CNN
+F 2 "SMD_Packages:TQFP-64" H 5400 3950 60  0001 C CNN
 F 3 "" H 5400 3950 60  0000 C CNN
 	1    5400 3950
@@
 Text HLabel 4750 2400 1    60   Input ~ 0
 GND
-Text HLabel 6150 5800 3    60   BiDi ~ 0
+Text HLabel 6150 5800 3    60   Output ~ 0
+UART_RX
+Text HLabel 7350 4700 2    60   Input ~ 0
 UART_TX
-Text HLabel 7350 4700 2    60   BiDi ~ 0
-UART_RX
-Text HLabel 7350 4600 2    60   BiDi ~ 0
+Text HLabel 7350 4600 2    60   Input ~ 0
+UART_RX_BT
+Text HLabel 7350 4500 2    60   Output ~ 0
 UART_TX_BT
-Text HLabel 7350 4500 2    60   BiDi ~ 0
-UART_RX_BT
 Text HLabel 5050 2500 1    60   Output ~ 0
 WAKE_SW
@@
 ~CS
 $Comp
-L CP1 10
+L CP1 U9
 U 1 1 5473ADF7
 P 2200 3400
-F 0 "10" H 2250 3500 50  0000 L CNN
+F 0 "U9" H 2250 3500 50  0000 L CNN
 F 1 "CP1" H 2250 3300 50  0000 L CNN
-F 2 "" H 2200 3400 60  0000 C CNN
+F 2 "Capacitors_SMD:C_1206_HandSoldering" H 2200 3400 60  0001 C CNN
 F 3 "" H 2200 3400 60  0000 C CNN
 	1    2200 3400
@@
 $EndComp
 $Comp
-L C 0.1
+L C U10
 U 1 1 5473B485
 P 2550 3400
-F 0 "0.1" H 2550 3500 40  0000 L CNN
+F 0 "U10" H 2550 3500 40  0000 L CNN
 F 1 "C" H 2556 3315 40  0000 L CNN
-F 2 "" H 2588 3250 30  0000 C CNN
+F 2 "Capacitors_SMD:C_1206_HandSoldering" H 2588 3250 30  0001 C CNN
 F 3 "" H 2550 3400 60  0000 C CNN
 	1    2550 3400
@@
 Wire Wire Line
 	6650 4600 7350 4600
-Wire Wire Line
-	7350 4500 6650 4500
 Wire Wire Line
 	5050 2700 5050 2500
@@
 Wire Wire Line
 	5650 2500 5650 2700
+Wire Wire Line
+	6650 4500 7350 4500
 $EndSCHEMATC

Commit message: General fine tuning of schematics. Need to review JTAG and update. Added resistors to power stage. Getting prepped for BOM, need to go through item by item. Added current incomplete BOM
Parts:
- U10: value C -> 0.1u
- U9: value CP1 -> 10u
Connections:
- net FUSE: no longer names the net of U11.55 (TDI/TCLK)
- no-connect marks 44 -> 45
Changed lines of the file:
@@
 Comment4 ""
 $EndDescr
-$Comp
-L MSP430F247 U11
-U 1 1 547269CD
-P 5400 3950
-F 0 "U11" H 5400 3980 30  0000 C CNN
-F 1 "MSP430F247" H 5400 3920 30  0000 C CNN
-F 2 "SMD_Packages:TQFP-64" H 5400 3950 60  0001 C CNN
-F 3 "" H 5400 3950 60  0000 C CNN
-	1    5400 3950
-	1    0    0    -1
-$EndComp
 Text HLabel 2000 3200 0    60   Input ~ 0
 3.3V
@@
 P 2200 3400
 F 0 "U9" H 2250 3500 50  0000 L CNN
-F 1 "CP1" H 2250 3300 50  0000 L CNN
+F 1 "10u" H 2250 3300 50  0000 L CNN
 F 2 "Capacitors_SMD:C_1206_HandSoldering" H 2200 3400 60  0001 C CNN
 F 3 "" H 2200 3400 60  0000 C CNN
@@
 P 2550 3400
 F 0 "U10" H 2550 3500 40  0000 L CNN
-F 1 "C" H 2556 3315 40  0000 L CNN
+F 1 "0.1u" H 2556 3315 40  0000 L CNN
 F 2 "Capacitors_SMD:C_1206_HandSoldering" H 2588 3250 30  0001 C CNN
 F 3 "" H 2550 3400 60  0000 C CNN
@@
 Wire Wire Line
 	5350 2500 5350 2700
-Text HLabel 5550 2500 1    60   Input ~ 0
-FUSE
-Wire Wire Line
-	5550 2500 5550 2700
 Text HLabel 5650 2500 1    60   BiDi ~ 0
 TDO/TDI
@@
 Wire Wire Line
 	6650 4500 7350 4500
+$Comp
+L MSP430F247 U11
+U 1 1 547269CD
+P 5400 3950
+F 0 "U11" H 5400 3980 30  0000 C CNN
+F 1 "MSP430F247" H 5400 3920 30  0000 C CNN
+F 2 "SMD_Packages:TQFP-64" H 5400 3950 60  0001 C CNN
+F 3 "" H 5400 3950 60  0000 C CNN
+	1    5400 3950
+	1    0    0    -1
+$EndComp
+NoConn ~ 5550 2700
 $EndSCHEMATC

Commit message: Updated parts and data sheets
Parts:
- removed U10: 0.1u, Capacitors_SMD:C_1206_HandSoldering, symbol C
- removed U9: 10u, Capacitors_SMD:C_1206_HandSoldering, symbol CP1
- added C18: 2.2n, Capacitors_SMD:C_0805_HandSoldering, symbol C
- added C19: 10U, symbol CP1
- added C20: 0.1U, symbol C
- added R4: 47k, Resistors_SMD:R_0805_HandSoldering, symbol R
Connections:
- net 3.3V: now also C19.1, C20.1, R4.1; no longer U11.58 (RST/NMI)
- net GND: now also C18.1, C19.2, C20.2
- net TDI/VPP: now reaches U11.55 (TDI/TCLK)
- net TMS: now reaches U11.56 (TMS)
- new net ~RST: C18.2, R4.2, U11.58 (RST/NMI)
- no-connect marks 45 -> 43
Changed lines of the file:
@@
 NoConn ~ 4150 4000
 NoConn ~ 4150 3900
-NoConn ~ 5450 2700
 NoConn ~ 5750 2700
 NoConn ~ 5850 2700
@@
 Text HLabel 7350 3600 2    60   Output ~ 0
 ~CS
-$Comp
-L CP1 U9
-U 1 1 5473ADF7
-P 2200 3400
-F 0 "U9" H 2250 3500 50  0000 L CNN
-F 1 "10u" H 2250 3300 50  0000 L CNN
-F 2 "Capacitors_SMD:C_1206_HandSoldering" H 2200 3400 60  0001 C CNN
-F 3 "" H 2200 3400 60  0000 C CNN
-	1    2200 3400
-	1    0    0    -1
-$EndComp
-$Comp
-L C U10
-U 1 1 5473B485
-P 2550 3400
-F 0 "U10" H 2550 3500 40  0000 L CNN
-F 1 "0.1u" H 2556 3315 40  0000 L CNN
-F 2 "Capacitors_SMD:C_1206_HandSoldering" H 2588 3250 30  0001 C CNN
-F 3 "" H 2550 3400 60  0000 C CNN
-	1    2550 3400
-	1    0    0    -1
-$EndComp
 Text HLabel 2200 3900 3    60   Input ~ 0
 GND
@@
 	2550 3600 2550 3900
 Wire Wire Line
-	5250 2700 5250 2500
-Text HLabel 5250 2500 1    60   Input ~ 0
+	5250 1600 5250 2700
+Text HLabel 5250 1050 1    60   Input ~ 0
 3.3V
 Text HLabel 5350 2500 1    60   Input ~ 0
@@
 	1    0    0    -1
 $EndComp
-NoConn ~ 5550 2700
+Text HLabel 5450 2500 1    60   Input ~ 0
+TMS
+Wire Wire Line
+	5450 2700 5450 2500
+Text HLabel 5550 2500 1    60   Input ~ 0
+TDI/VPP
+Wire Wire Line
+	5550 2500 5550 2700
+$Comp
+L R R4
+U 1 1 54763D43
+P 5250 1350
+F 0 "R4" V 5330 1350 40  0000 C CNN
+F 1 "47k" V 5257 1351 40  0000 C CNN
+F 2 "Resistors_SMD:R_0805_HandSoldering" V 5180 1350 30  0001 C CNN
+F 3 "" H 5250 1350 30  0000 C CNN
+	1    5250 1350
+	1    0    0    -1
+$EndComp
+Wire Wire Line
+	5250 1100 5250 1050
+Text HLabel 5450 1600 2    60   Input ~ 0
+~RST
+Wire Wire Line
+	5450 1600 5250 1600
+$Comp
+L C C18
+U 1 1 547688E6
+P 5550 1800
+F 0 "C18" H 5550 1900 40  0000 L CNN
+F 1 "2.2n" H 5556 1715 40  0000 L CNN
+F 2 "Capacitors_SMD:C_0805_HandSoldering" H 5588 1650 30  0001 C CNN
+F 3 "" H 5550 1800 60  0000 C CNN
+	1    5550 1800
+	0    1    1    0
+$EndComp
+Wire Wire Line
+	5250 1800 5350 1800
+Connection ~ 5250 1800
+Text HLabel 5850 1800 2    60   Input ~ 0
+GND
+Wire Wire Line
+	5850 1800 5750 1800
+$Comp
+L C C20
+U 1 1 547811D1
+P 2550 3400
+F 0 "C20" H 2550 3500 40  0000 L CNN
+F 1 "0.1U" H 2556 3315 40  0000 L CNN
+F 2 "" H 2588 3250 30  0001 C CNN
+F 3 "" H 2550 3400 60  0000 C CNN
+	1    2550 3400
+	1    0    0    -1
+$EndComp
+$Comp
+L CP1 C19
+U 1 1 54781237
+P 2200 3400
+F 0 "C19" H 2250 3500 50  0000 L CNN
+F 1 "10U" H 2250 3300 50  0000 L CNN
+F 2 "" H 2200 3400 60  0001 C CNN
+F 3 "" H 2200 3400 60  0000 C CNN
+	1    2200 3400
+	1    0    0    -1
+$EndComp
 $EndSCHEMATC

Commit message: 1st Revision
Complete Board layout, 1st Draft
Parts:
- C19, C20: footprint (none) -> Capacitors_SMD:C_0805_HandSoldering
- U11: footprint SMD_Packages:TQFP-64 -> GEM:LQFP_64PIN_MSP430
Connections:
- net 3.3V renamed VCC/TOOL
Changed lines of the file:
@@
 $Descr A4 11693 8268
 encoding utf-8
-Sheet 8 11
+Sheet 8 12
 Title ""
 Date ""
@@
 $EndDescr
 Text HLabel 2000 3200 0    60   Input ~ 0
-3.3V
+VCC/TOOL
 Text HLabel 4750 2400 1    60   Input ~ 0
 GND
@@
 Text HLabel 2550 3900 3    60   Input ~ 0
 GND
-Wire Wire Line
-	4650 2700 4650 2500
-Wire Wire Line
-	4750 2400 4750 2700
-Wire Wire Line
-	4850 2700 4850 2500
-Wire Wire Line
-	4850 2500 4750 2500
-Connection ~ 4750 2500
-Wire Wire Line
-	6150 5800 6150 5200
-Wire Wire Line
-	7350 4700 6650 4700
-Wire Wire Line
-	6650 4600 7350 4600
-Wire Wire Line
-	5050 2700 5050 2500
-Wire Wire Line
-	4950 2700 4950 2500
-Wire Wire Line
-	4150 3300 3600 3300
-Wire Wire Line
-	4150 3400 3600 3400
-Wire Wire Line
-	7350 3500 6650 3500
-Wire Wire Line
-	7350 3400 6650 3400
-Wire Wire Line
-	7350 3300 6650 3300
-Wire Wire Line
-	6650 3600 7350 3600
-Wire Wire Line
-	2000 3200 4150 3200
-Connection ~ 2200 3200
-Connection ~ 2550 3200
-Wire Wire Line
-	3600 3200 3600 2500
-Wire Wire Line
-	3600 2500 4650 2500
-Connection ~ 3600 3200
-Wire Wire Line
-	2200 3600 2200 3900
-Wire Wire Line
-	2550 3600 2550 3900
-Wire Wire Line
-	5250 1600 5250 2700
 Text HLabel 5250 1050 1    60   Input ~ 0
-3.3V
+VCC/TOOL
 Text HLabel 5350 2500 1    60   Input ~ 0
 TCK
-Wire Wire Line
-	5350 2500 5350 2700
 Text HLabel 5650 2500 1    60   BiDi ~ 0
 TDO/TDI
-Wire Wire Line
-	5650 2500 5650 2700
-Wire Wire Line
-	6650 4500 7350 4500
 $Comp
 L MSP430F247 U11
@@
 F 0 "U11" H 5400 3980 30  0000 C CNN
 F 1 "MSP430F247" H 5400 3920 30  0000 C CNN
-F 2 "SMD_Packages:TQFP-64" H 5400 3950 60  0001 C CNN
+F 2 "GEM:LQFP_64PIN_MSP430" H 5400 3950 60  0001 C CNN
 F 3 "" H 5400 3950 60  0000 C CNN
 	1    5400 3950
@@
 Text HLabel 5450 2500 1    60   Input ~ 0
 TMS
-Wire Wire Line
-	5450 2700 5450 2500
 Text HLabel 5550 2500 1    60   Input ~ 0
 TDI/VPP
-Wire Wire Line
-	5550 2500 5550 2700
 $Comp
 L R R4
@@
 	1    0    0    -1
 $EndComp
-Wire Wire Line
-	5250 1100 5250 1050
-Text HLabel 5450 1600 2    60   Input ~ 0
+Text HLabel 5450 1650 2    60   Input ~ 0
 ~RST
-Wire Wire Line
-	5450 1600 5250 1600
 $Comp
 L C C18
@@
 	0    1    1    0
 $EndComp
-Wire Wire Line
-	5250 1800 5350 1800
-Connection ~ 5250 1800
 Text HLabel 5850 1800 2    60   Input ~ 0
 GND
-Wire Wire Line
-	5850 1800 5750 1800
 $Comp
 L C C20
@@
 F 0 "C20" H 2550 3500 40  0000 L CNN
 F 1 "0.1U" H 2556 3315 40  0000 L CNN
-F 2 "" H 2588 3250 30  0001 C CNN
+F 2 "Capacitors_SMD:C_0805_HandSoldering" H 2588 3250 30  0001 C CNN
 F 3 "" H 2550 3400 60  0000 C CNN
 	1    2550 3400
@@
 F 0 "C19" H 2250 3500 50  0000 L CNN
 F 1 "10U" H 2250 3300 50  0000 L CNN
-F 2 "" H 2200 3400 60  0001 C CNN
+F 2 "Capacitors_SMD:C_0805_HandSoldering" H 2200 3400 60  0001 C CNN
 F 3 "" H 2200 3400 60  0000 C CNN
 	1    2200 3400
 	1    0    0    -1
 $EndComp
+Connection ~ 5250 1650
+Wire Wire Line
+	5450 1650 5250 1650
+Wire Wire Line
+	5850 1800 5750 1800
+Connection ~ 5250 1800
+Wire Wire Line
+	5250 1800 5350 1800
+Wire Wire Line
+	5250 1100 5250 1050
+Wire Wire Line
+	5550 2500 5550 2700
+Wire Wire Line
+	5450 2700 5450 2500
+Wire Wire Line
+	6650 4500 7350 4500
+Wire Wire Line
+	5650 2500 5650 2700
+Wire Wire Line
+	5350 2500 5350 2700
+Wire Wire Line
+	5250 1600 5250 2700
+Wire Wire Line
+	2550 3600 2550 3900
+Wire Wire Line
+	2200 3600 2200 3900
+Connection ~ 3600 3200
+Wire Wire Line
+	3600 2500 4650 2500
+Wire Wire Line
+	3600 3200 3600 2500
+Connection ~ 2550 3200
+Connection ~ 2200 3200
+Wire Wire Line
+	2000 3200 4150 3200
+Wire Wire Line
+	6650 3600 7350 3600
+Wire Wire Line
+	7350 3300 6650 3300
+Wire Wire Line
+	7350 3400 6650 3400
+Wire Wire Line
+	7350 3500 6650 3500
+Wire Wire Line
+	4150 3400 3600 3400
+Wire Wire Line
+	4150 3300 3600 3300
+Wire Wire Line
+	4950 2700 4950 2500
+Wire Wire Line
+	5050 2700 5050 2500
+Wire Wire Line
+	6650 4600 7350 4600
+Wire Wire Line
+	7350 4700 6650 4700
+Wire Wire Line
+	6150 5800 6150 5200
+Connection ~ 4750 2500
+Wire Wire Line
+	4850 2500 4750 2500
+Wire Wire Line
+	4850 2700 4850 2500
+Wire Wire Line
+	4750 2400 4750 2700
+Wire Wire Line
+	4650 2500 4650 2700
 $EndSCHEMATC
