File: STATUS_LIGHTS.sch (KiCad schematic (older format))
At the start: 12 parts

Commit message: Linked components to footprints, may have to switch to smaller components. Started board layout.
Parts:
- D1, D2, D3, D4: footprint (none) -> LEDs:LED-1206
- D5: renamed from D14; footprint (none) -> LEDs:LED-1206
- D6: renamed from D15; footprint (none) -> LEDs:LED-1206
- R11, R12, R13, R14: value R -> 330; footprint (none) -> Resistors_SMD:R_1206_HandSoldering
- R15: renamed from R47; value R -> 330; footprint (none) -> Resistors_SMD:R_1206_HandSoldering
- R16: renamed from R48; value R -> 330; footprint (none) -> Resistors_SMD:R_1206_HandSoldering
Changed lines of the file:
@@
 F 0 "D1" H 2000 3050 50  0000 C CNN
 F 1 "LED" H 2000 2850 50  0000 C CNN
-F 2 "" H 2000 2950 60  0000 C CNN
+F 2 "LEDs:LED-1206" H 2000 2950 60  0001 C CNN
 F 3 "" H 2000 2950 60  0000 C CNN
 	1    2000 2950
@@
 F 0 "D2" H 2550 3050 50  0000 C CNN
 F 1 "LED" H 2550 2850 50  0000 C CNN
-F 2 "" H 2550 2950 60  0000 C CNN
+F 2 "LEDs:LED-1206" H 2550 2950 60  0001 C CNN
 F 3 "" H 2550 2950 60  0000 C CNN
 	1    2550 2950
@@
 F 0 "D3" H 3100 3050 50  0000 C CNN
 F 1 "LED" H 3100 2850 50  0000 C CNN
-F 2 "" H 3100 2950 60  0000 C CNN
+F 2 "LEDs:LED-1206" H 3100 2950 60  0001 C CNN
 F 3 "" H 3100 2950 60  0000 C CNN
 	1    3100 2950
@@
 F 0 "D4" H 3550 3050 50  0000 C CNN
 F 1 "LED" H 3550 2850 50  0000 C CNN
-F 2 "" H 3550 2950 60  0000 C CNN
+F 2 "LEDs:LED-1206" H 3550 2950 60  0001 C CNN
 F 3 "" H 3550 2950 60  0000 C CNN
 	1    3550 2950
@@
 P 2000 3550
 F 0 "R11" V 2080 3550 40  0000 C CNN
-F 1 "R" V 2007 3551 40  0000 C CNN
-F 2 "" V 1930 3550 30  0000 C CNN
+F 1 "330" V 2007 3551 40  0000 C CNN
+F 2 "Resistors_SMD:R_1206_HandSoldering" V 1930 3550 30  0001 C CNN
 F 3 "" H 2000 3550 30  0000 C CNN
 	1    2000 3550
@@
 P 2550 3550
 F 0 "R12" V 2630 3550 40  0000 C CNN
-F 1 "R" V 2557 3551 40  0000 C CNN
-F 2 "" V 2480 3550 30  0000 C CNN
+F 1 "330" V 2557 3551 40  0000 C CNN
+F 2 "Resistors_SMD:R_1206_HandSoldering" V 2480 3550 30  0001 C CNN
 F 3 "" H 2550 3550 30  0000 C CNN
 	1    2550 3550
@@
 P 3100 3550
 F 0 "R13" V 3180 3550 40  0000 C CNN
-F 1 "R" V 3107 3551 40  0000 C CNN
-F 2 "" V 3030 3550 30  0000 C CNN
+F 1 "330" V 3107 3551 40  0000 C CNN
+F 2 "Resistors_SMD:R_1206_HandSoldering" V 3030 3550 30  0001 C CNN
 F 3 "" H 3100 3550 30  0000 C CNN
 	1    3100 3550
@@
 P 3550 3550
 F 0 "R14" V 3630 3550 40  0000 C CNN
-F 1 "R" V 3557 3551 40  0000 C CNN
-F 2 "" V 3480 3550 30  0000 C CNN
+F 1 "330" V 3557 3551 40  0000 C CNN
+F 2 "Resistors_SMD:R_1206_HandSoldering" V 3480 3550 30  0001 C CNN
 F 3 "" H 3550 3550 30  0000 C CNN
 	1    3550 3550
@@
 	3550 4550 2000 4550
 $Comp
-L LED D14
+L LED D5
 U 1 1 54798AE5
 P 4050 2950
-F 0 "D14" H 4050 3050 50  0000 C CNN
+F 0 "D5" H 4050 3050 50  0000 C CNN
 F 1 "LED" H 4050 2850 50  0000 C CNN
-F 2 "" H 4050 2950 60  0000 C CNN
+F 2 "LEDs:LED-1206" H 4050 2950 60  0001 C CNN
 F 3 "" H 4050 2950 60  0000 C CNN
 	1    4050 2950
@@
 3.3V
 $Comp
-L R R47
+L R R15
 U 1 1 54798AEC
 P 4050 3550
-F 0 "R47" V 4130 3550 40  0000 C CNN
-F 1 "R" V 4057 3551 40  0000 C CNN
-F 2 "" V 3980 3550 30  0000 C CNN
+F 0 "R15" V 4130 3550 40  0000 C CNN
+F 1 "330" V 4057 3551 40  0000 C CNN
+F 2 "Resistors_SMD:R_1206_HandSoldering" V 3980 3550 30  0001 C CNN
 F 3 "" H 4050 3550 30  0000 C CNN
 	1    4050 3550
@@
 ~BT_CNT_LED
 $Comp
-L LED D15
+L LED D6
 U 1 1 54799D0D
 P 4650 2950
-F 0 "D15" H 4650 3050 50  0000 C CNN
+F 0 "D6" H 4650 3050 50  0000 C CNN
 F 1 "LED" H 4650 2850 50  0000 C CNN
-F 2 "" H 4650 2950 60  0000 C CNN
+F 2 "LEDs:LED-1206" H 4650 2950 60  0001 C CNN
 F 3 "" H 4650 2950 60  0000 C CNN
 	1    4650 2950
@@
 3.3V
 $Comp
-L R R48
+L R R16
 U 1 1 54799D14
 P 4650 3550
-F 0 "R48" V 4730 3550 40  0000 C CNN
-F 1 "R" V 4657 3551 40  0000 C CNN
-F 2 "" V 4580 3550 30  0000 C CNN
+F 0 "R16" V 4730 3550 40  0000 C CNN
+F 1 "330" V 4657 3551 40  0000 C CNN
+F 2 "Resistors_SMD:R_1206_HandSoldering" V 4580 3550 30  0001 C CNN
 F 3 "" H 4650 3550 30  0000 C CNN
 	1    4650 3550
@@
 Wire Wire Line
 	4650 3150 4650 3300
-Text HLabel 1950 5000 0    60   Input ~ 0
+Text HLabel 1900 5000 0    60   Input ~ 0
 ~BT_ACT_LED
 Wire Wire Line

Commit message: General fine tuning of schematics. Need to review JTAG and update. Added resistors to power stage. Getting prepped for BOM, need to go through item by item. Added current incomplete BOM
Parts:
- D1, D2, D3, D4, D5, D6: footprint LEDs:LED-1206 -> LEDs:LED-0805
Changed lines of the file:
@@
 F 0 "D1" H 2000 3050 50  0000 C CNN
 F 1 "LED" H 2000 2850 50  0000 C CNN
-F 2 "LEDs:LED-1206" H 2000 2950 60  0001 C CNN
+F 2 "LEDs:LED-0805" H 2000 2950 60  0001 C CNN
 F 3 "" H 2000 2950 60  0000 C CNN
 	1    2000 2950
@@
 F 0 "D2" H 2550 3050 50  0000 C CNN
 F 1 "LED" H 2550 2850 50  0000 C CNN
-F 2 "LEDs:LED-1206" H 2550 2950 60  0001 C CNN
+F 2 "LEDs:LED-0805" H 2550 2950 60  0001 C CNN
 F 3 "" H 2550 2950 60  0000 C CNN
 	1    2550 2950
@@
 F 0 "D3" H 3100 3050 50  0000 C CNN
 F 1 "LED" H 3100 2850 50  0000 C CNN
-F 2 "LEDs:LED-1206" H 3100 2950 60  0001 C CNN
+F 2 "LEDs:LED-0805" H 3100 2950 60  0001 C CNN
 F 3 "" H 3100 2950 60  0000 C CNN
 	1    3100 2950
@@
 F 0 "D4" H 3550 3050 50  0000 C CNN
 F 1 "LED" H 3550 2850 50  0000 C CNN
-F 2 "LEDs:LED-1206" H 3550 2950 60  0001 C CNN
+F 2 "LEDs:LED-0805" H 3550 2950 60  0001 C CNN
 F 3 "" H 3550 2950 60  0000 C CNN
 	1    3550 2950
@@
 F 0 "D5" H 4050 3050 50  0000 C CNN
 F 1 "LED" H 4050 2850 50  0000 C CNN
-F 2 "LEDs:LED-1206" H 4050 2950 60  0001 C CNN
+F 2 "LEDs:LED-0805" H 4050 2950 60  0001 C CNN
 F 3 "" H 4050 2950 60  0000 C CNN
 	1    4050 2950
@@
 F 0 "D6" H 4650 3050 50  0000 C CNN
 F 1 "LED" H 4650 2850 50  0000 C CNN
-F 2 "LEDs:LED-1206" H 4650 2950 60  0001 C CNN
+F 2 "LEDs:LED-0805" H 4650 2950 60  0001 C CNN
 F 3 "" H 4650 2950 60  0000 C CNN
 	1    4650 2950

Commit message: Updated parts and data sheets
Parts:
- D1, D2, D3, D4, D5, D6: Part Number (none) -> APT2012ZGC
- R11, R12, R13, R14, R15, R16: footprint Resistors_SMD:R_1206_HandSoldering -> Resistors_SMD:R_0805_HandSoldering
Changed lines of the file:
@@
 F 2 "LEDs:LED-0805" H 2000 2950 60  0001 C CNN
 F 3 "" H 2000 2950 60  0000 C CNN
+F 4 "APT2012ZGC" H 2000 2950 60  0001 C CNN "Part Number"
 	1    2000 2950
 	0    1    1    0
@@
 F 2 "LEDs:LED-0805" H 2550 2950 60  0001 C CNN
 F 3 "" H 2550 2950 60  0000 C CNN
+F 4 "APT2012ZGC" H 2550 2950 60  0001 C CNN "Part Number"
 	1    2550 2950
 	0    1    1    0
@@
 F 2 "LEDs:LED-0805" H 3100 2950 60  0001 C CNN
 F 3 "" H 3100 2950 60  0000 C CNN
+F 4 "APT2012ZGC" H 3100 2950 60  0001 C CNN "Part Number"
 	1    3100 2950
 	0    1    1    0
@@
 F 2 "LEDs:LED-0805" H 3550 2950 60  0001 C CNN
 F 3 "" H 3550 2950 60  0000 C CNN
+F 4 "APT2012ZGC" H 3550 2950 60  0001 C CNN "Part Number"
 	1    3550 2950
 	0    1    1    0
@@
 F 0 "R11" V 2080 3550 40  0000 C CNN
 F 1 "330" V 2007 3551 40  0000 C CNN
-F 2 "Resistors_SMD:R_1206_HandSoldering" V 1930 3550 30  0001 C CNN
+F 2 "Resistors_SMD:R_0805_HandSoldering" V 1930 3550 30  0001 C CNN
 F 3 "" H 2000 3550 30  0000 C CNN
 	1    2000 3550
@@
 F 0 "R12" V 2630 3550 40  0000 C CNN
 F 1 "330" V 2557 3551 40  0000 C CNN
-F 2 "Resistors_SMD:R_1206_HandSoldering" V 2480 3550 30  0001 C CNN
+F 2 "Resistors_SMD:R_0805_HandSoldering" V 2480 3550 30  0001 C CNN
 F 3 "" H 2550 3550 30  0000 C CNN
 	1    2550 3550
@@
 F 0 "R13" V 3180 3550 40  0000 C CNN
 F 1 "330" V 3107 3551 40  0000 C CNN
-F 2 "Resistors_SMD:R_1206_HandSoldering" V 3030 3550 30  0001 C CNN
+F 2 "Resistors_SMD:R_0805_HandSoldering" V 3030 3550 30  0001 C CNN
 F 3 "" H 3100 3550 30  0000 C CNN
 	1    3100 3550
@@
 F 0 "R14" V 3630 3550 40  0000 C CNN
 F 1 "330" V 3557 3551 40  0000 C CNN
-F 2 "Resistors_SMD:R_1206_HandSoldering" V 3480 3550 30  0001 C CNN
+F 2 "Resistors_SMD:R_0805_HandSoldering" V 3480 3550 30  0001 C CNN
 F 3 "" H 3550 3550 30  0000 C CNN
 	1    3550 3550
@@
 F 2 "LEDs:LED-0805" H 4050 2950 60  0001 C CNN
 F 3 "" H 4050 2950 60  0000 C CNN
+F 4 "APT2012ZGC" H 4050 2950 60  0001 C CNN "Part Number"
 	1    4050 2950
 	0    1    1    0
@@
 F 0 "R15" V 4130 3550 40  0000 C CNN
 F 1 "330" V 4057 3551 40  0000 C CNN
-F 2 "Resistors_SMD:R_1206_HandSoldering" V 3980 3550 30  0001 C CNN
+F 2 "Resistors_SMD:R_0805_HandSoldering" V 3980 3550 30  0001 C CNN
 F 3 "" H 4050 3550 30  0000 C CNN
 	1    4050 3550
@@
 F 2 "LEDs:LED-0805" H 4650 2950 60  0001 C CNN
 F 3 "" H 4650 2950 60  0000 C CNN
+F 4 "APT2012ZGC" H 4650 2950 60  0001 C CNN "Part Number"
 	1    4650 2950
 	0    1    1    0
@@
 F 0 "R16" V 4730 3550 40  0000 C CNN
 F 1 "330" V 4657 3551 40  0000 C CNN
-F 2 "Resistors_SMD:R_1206_HandSoldering" V 4580 3550 30  0001 C CNN
+F 2 "Resistors_SMD:R_0805_HandSoldering" V 4580 3550 30  0001 C CNN
 F 3 "" H 4650 3550 30  0000 C CNN
 	1    4650 3550
