File: STATUS_LIGHTS.sch (KiCad schematic (older format))
At the start: 8 parts

Commit message: Added Bluetooth module and SD card
Added RN4020 and a microSD card to libraries, connected most pins. Also
added datasheets.
Parts:
- added D5, D6: LED, symbol LED
- added R15, R16: R, symbol R
Connections:
- net 3.3V: now also D5.1 (A), D6.1 (A)
- new net: D5.2 (K), R15.1
- new net: D6.2 (K), R16.1
- new net ~BT_ACT_LED: R16.2
- new net ~BT_CNT_LED: R15.2
Changed lines of the file:
@@
 $Descr A4 11693 8268
 encoding utf-8
-Sheet 4 8
+Sheet 4 10
 Title "GEM"
 Date "Saturday, November 15, 2014"
@@
 Wire Wire Line
 	3550 4550 2000 4550
+$Comp
+L LED D5
+U 1 1 54798AE5
+P 4050 2950
+F 0 "D5" H 4050 3050 50  0000 C CNN
+F 1 "LED" H 4050 2850 50  0000 C CNN
+F 2 "" H 4050 2950 60  0000 C CNN
+F 3 "" H 4050 2950 60  0000 C CNN
+	1    4050 2950
+	0    1    1    0
+$EndComp
+Text HLabel 4050 2550 1    60   Input ~ 0
+3.3V
+$Comp
+L R R15
+U 1 1 54798AEC
+P 4050 3550
+F 0 "R15" V 4130 3550 40  0000 C CNN
+F 1 "R" V 4057 3551 40  0000 C CNN
+F 2 "" V 3980 3550 30  0000 C CNN
+F 3 "" H 4050 3550 30  0000 C CNN
+	1    4050 3550
+	1    0    0    -1
+$EndComp
+Wire Wire Line
+	4050 3150 4050 3300
+Wire Wire Line
+	4050 2550 4050 2750
+Text HLabel 1950 4750 0    60   Input ~ 0
+~BT_CNT_LED
+Wire Wire Line
+	1950 4750 4050 4750
+Wire Wire Line
+	4050 4750 4050 3800
+$Comp
+L LED D6
+U 1 1 54799D0D
+P 4650 2950
+F 0 "D6" H 4650 3050 50  0000 C CNN
+F 1 "LED" H 4650 2850 50  0000 C CNN
+F 2 "" H 4650 2950 60  0000 C CNN
+F 3 "" H 4650 2950 60  0000 C CNN
+	1    4650 2950
+	0    1    1    0
+$EndComp
+Text HLabel 4650 2550 1    60   Input ~ 0
+3.3V
+$Comp
+L R R16
+U 1 1 54799D14
+P 4650 3550
+F 0 "R16" V 4730 3550 40  0000 C CNN
+F 1 "R" V 4657 3551 40  0000 C CNN
+F 2 "" V 4580 3550 30  0000 C CNN
+F 3 "" H 4650 3550 30  0000 C CNN
+	1    4650 3550
+	1    0    0    -1
+$EndComp
+Wire Wire Line
+	4650 2550 4650 2750
+Wire Wire Line
+	4650 3150 4650 3300
+Text HLabel 1950 5000 0    60   Input ~ 0
+~BT_ACT_LED
+Wire Wire Line
+	4650 3800 4650 5000
+Wire Wire Line
+	4650 5000 1950 5000
 $EndSCHEMATC

Commit message: Added JTAG interface
Spy Bi-Wire JTAG interface. Fixed some unused pins.
Parts:
- renumbered D5 to D14, D6 to D15, R15 to R47, R16 to R48
Changed lines of the file:
@@
 $Descr A4 11693 8268
 encoding utf-8
-Sheet 4 10
+Sheet 4 11
 Title "GEM"
 Date "Saturday, November 15, 2014"
@@
 	3550 4550 2000 4550
 $Comp
-L LED D5
+L LED D14
 U 1 1 54798AE5
 P 4050 2950
-F 0 "D5" H 4050 3050 50  0000 C CNN
+F 0 "D14" H 4050 3050 50  0000 C CNN
 F 1 "LED" H 4050 2850 50  0000 C CNN
 F 2 "" H 4050 2950 60  0000 C CNN
@@
 3.3V
 $Comp
-L R R15
+L R R47
 U 1 1 54798AEC
 P 4050 3550
-F 0 "R15" V 4130 3550 40  0000 C CNN
+F 0 "R47" V 4130 3550 40  0000 C CNN
 F 1 "R" V 4057 3551 40  0000 C CNN
 F 2 "" V 3980 3550 30  0000 C CNN
@@
 Text HLabel 1950 4750 0    60   Input ~ 0
 ~BT_CNT_LED
-Wire Wire Line
-	1950 4750 4050 4750
-Wire Wire Line
-	4050 4750 4050 3800
-$Comp
-L LED D6
+$Comp
+L LED D15
 U 1 1 54799D0D
 P 4650 2950
-F 0 "D6" H 4650 3050 50  0000 C CNN
+F 0 "D15" H 4650 3050 50  0000 C CNN
 F 1 "LED" H 4650 2850 50  0000 C CNN
 F 2 "" H 4650 2950 60  0000 C CNN
@@
 3.3V
 $Comp
-L R R16
+L R R48
 U 1 1 54799D14
 P 4650 3550
-F 0 "R16" V 4730 3550 40  0000 C CNN
+F 0 "R48" V 4730 3550 40  0000 C CNN
 F 1 "R" V 4657 3551 40  0000 C CNN
 F 2 "" V 4580 3550 30  0000 C CNN
@@
 ~BT_ACT_LED
 Wire Wire Line
-	4650 3800 4650 5000
-Wire Wire Line
-	4650 5000 1950 5000
+	1950 4750 4050 4750
+Wire Wire Line
+	4050 4750 4050 3800
+Wire Wire Line
+	1900 5000 4650 5000
+Wire Wire Line
+	4650 5000 4650 3800
 $EndSCHEMATC

Commit message: Updated power supply removing a short. Updated resistor values for LED's after finding what LED's are available in 0805 size.
Parts:
- R11, R12, R13, R14, R47, R48: value R -> 100
Changed lines of the file:
@@
 P 2000 3550
 F 0 "R11" V 2080 3550 40  0000 C CNN
-F 1 "R" V 2007 3551 40  0000 C CNN
+F 1 "100" V 2007 3551 40  0000 C CNN
 F 2 "" V 1930 3550 30  0000 C CNN
 F 3 "" H 2000 3550 30  0000 C CNN
@@
 P 2550 3550
 F 0 "R12" V 2630 3550 40  0000 C CNN
-F 1 "R" V 2557 3551 40  0000 C CNN
+F 1 "100" V 2557 3551 40  0000 C CNN
 F 2 "" V 2480 3550 30  0000 C CNN
 F 3 "" H 2550 3550 30  0000 C CNN
@@
 P 3100 3550
 F 0 "R13" V 3180 3550 40  0000 C CNN
-F 1 "R" V 3107 3551 40  0000 C CNN
+F 1 "100" V 3107 3551 40  0000 C CNN
 F 2 "" V 3030 3550 30  0000 C CNN
 F 3 "" H 3100 3550 30  0000 C CNN
@@
 P 3550 3550
 F 0 "R14" V 3630 3550 40  0000 C CNN
-F 1 "R" V 3557 3551 40  0000 C CNN
+F 1 "100" V 3557 3551 40  0000 C CNN
 F 2 "" V 3480 3550 30  0000 C CNN
 F 3 "" H 3550 3550 30  0000 C CNN
@@
 P 4050 3550
 F 0 "R47" V 4130 3550 40  0000 C CNN
-F 1 "R" V 4057 3551 40  0000 C CNN
+F 1 "100" V 4057 3551 40  0000 C CNN
 F 2 "" V 3980 3550 30  0000 C CNN
 F 3 "" H 4050 3550 30  0000 C CNN
@@
 P 4650 3550
 F 0 "R48" V 4730 3550 40  0000 C CNN
-F 1 "R" V 4657 3551 40  0000 C CNN
+F 1 "100" V 4657 3551 40  0000 C CNN
 F 2 "" V 4580 3550 30  0000 C CNN
 F 3 "" H 4650 3550 30  0000 C CNN
