File: POWER.sch (KiCad schematic (older format))
At the start: 26 parts, among them Q7 MMBF170, Q8 MOSFET_P, Q9 MOSFET_P, U5 LMR16006XDDC, U6 LMR16006XDDC

Commit message: Updated power supply removing a short. Updated resistor values for LED's after finding what LED's are available in 0805 size.
Connections:
- net GND: no longer R41.2, R42.1, R43.2, R44.1, U5.3 (FB), U6.3 (FB)
- new net: R41.2, R42.1, U5.3 (FB)
- new net: R43.2, R44.1, U6.3 (FB)
Changed lines of the file:
@@
 	9950 1650 9950 1900
 Connection ~ 9950 1750
-Connection ~ 8850 1750
 Wire Wire Line
 	9550 1150 10500 1150
@@
 	9950 4300 9950 4550
 Connection ~ 9950 4400
-Connection ~ 8850 4400
 Wire Wire Line
 	9550 3800 10550 3800
