File: POWER.sch (KiCad schematic (older format))
At the start: 26 parts, among them Q7 MMBF170, Q8 MOSFET_P, Q9 MOSFET_P, U5 LMR16006XDDC, U6 LMR16006XDDC

Commit message: Linked components to footprints, may have to switch to smaller components. Started board layout.
Parts:
- C10, C11, C12, C13, C14, C15, C16, C9: footprint (none) -> SMD_Packages:SMD-1206
- D10: renamed from D8; footprint (none) -> Diodes_SMD:Diode-SMB_Standard
- D11: renamed from D9; footprint (none) -> Diodes_SMD:Diode-SMB_Standard
- L1: value 47U -> 47u; footprint (none) -> Inductors:SELF-WE-TPC_M
- Q7: footprint SOT-23 -> SMD_Packages:SOT-23
- Q8, Q9: footprint (none) -> Transistors_TO-220:TO-220_FET-GDS_Horizontal_LargePads
- R41: renamed from R39; footprint (none) -> Resistors_SMD:R_1206_HandSoldering
- R42: renamed from R40; footprint (none) -> Resistors_SMD:R_1206_HandSoldering
- R43: renamed from R41; footprint (none) -> Resistors_SMD:R_1206_HandSoldering
- R44: renamed from R42; footprint (none) -> Resistors_SMD:R_1206_HandSoldering
- R45: renamed from R43; footprint (none) -> Resistors_SMD:R_1206_HandSoldering
- R46: renamed from R44; footprint (none) -> Resistors_SMD:R_1206_HandSoldering
- U6: renamed from U5; footprint (none) -> SMD_Packages:SOT-23-6
- U7: renamed from U6; footprint (none) -> SMD_Packages:SOT-23-6
- U8: renamed from 33u1; value INDUCTOR -> 33U; footprint (none) -> Inductors_NEOSID:Neosid_Inductor_SMS-ME3015
- renumbered D10 to D12, D11 to D13
Changed lines of the file:
@@
 $EndDescr
 $Comp
-L LMR16006XDDC U5
+L LMR16006XDDC U6
 U 1 1 5468AF74
 P 7400 1150
-F 0 "U5" H 7500 750 60  0000 C CNN
+F 0 "U6" H 7500 750 60  0000 C CNN
 F 1 "LMR16006XDDC" H 7450 1550 60  0000 C CNN
-F 2 "" H 7450 1550 60  0000 C CNN
+F 2 "SMD_Packages:SOT-23-6" H 7450 1550 60  0001 C CNN
 F 3 "" H 7450 1550 60  0000 C CNN
 	1    7400 1150
@@
 F 0 "C9" H 2550 1300 40  0000 L CNN
 F 1 "C" H 2556 1115 40  0000 L CNN
-F 2 "" H 2588 1050 30  0000 C CNN
+F 2 "SMD_Packages:SMD-1206" H 2588 1050 30  0001 C CNN
 F 3 "" H 2550 1200 60  0000 C CNN
 	1    2550 1200
@@
 $EndComp
 $Comp
-L TVS D8
+L TVS D10
 U 1 1 5468B1EB
 P 3300 1300
-F 0 "D8" H 3300 1450 60  0000 C CNN
+F 0 "D10" H 3300 1450 60  0000 C CNN
 F 1 "TVS" H 3300 1150 60  0000 C CNN
-F 2 "" H 3300 1300 60  0000 C CNN
+F 2 "Diodes_SMD:Diode-SMB_Standard" H 3300 1300 60  0001 C CNN
 F 3 "" H 3300 1300 60  0000 C CNN
 	1    3300 1300
@@
 F 0 "C10" H 4050 1300 40  0000 L CNN
 F 1 "C" H 4056 1115 40  0000 L CNN
-F 2 "" H 4088 1050 30  0000 C CNN
+F 2 "SMD_Packages:SMD-1206" H 4088 1050 30  0001 C CNN
 F 3 "" H 4050 1200 60  0000 C CNN
 	1    4050 1200
@@
 F 0 "F1" H 3050 950 40  0000 C CNN
 F 1 "PTC_FUSE" H 2850 850 40  0000 C CNN
-F 2 "" H 2950 900 60  0000 C CNN
+F 2 "" H 2950 900 60  0001 C CNN
 F 3 "" H 2950 900 60  0000 C CNN
 	1    2950 900
@@
 $EndComp
 $Comp
-L DIODE D9
+L DIODE D11
 U 1 1 5468B5EE
 P 3700 900
-F 0 "D9" H 3700 1000 40  0000 C CNN
+F 0 "D11" H 3700 1000 40  0000 C CNN
 F 1 "S2A" H 3700 800 40  0000 C CNN
-F 2 "" H 3700 900 60  0000 C CNN
+F 2 "Diodes_SMD:Diode-SMB_Standard" H 3700 900 60  0001 C CNN
 F 3 "" H 3700 900 60  0000 C CNN
 	1    3700 900
@@
 F 0 "C11" H 6400 1300 40  0000 L CNN
 F 1 "4.7U" H 6406 1115 40  0000 L CNN
-F 2 "" H 6438 1050 30  0000 C CNN
+F 2 "SMD_Packages:SMD-1206" H 6438 1050 30  0001 C CNN
 F 3 "" H 6400 1200 60  0000 C CNN
 F 4 "3.0m" H 6400 1200 60  0001 C CNN "ESR"
@@
 F 0 "C13" H 8350 1000 40  0000 L CNN
 F 1 "100n" H 8356 815 40  0000 L CNN
-F 2 "" H 8388 750 30  0000 C CNN
+F 2 "SMD_Packages:SMD-1206" H 8388 750 30  0001 C CNN
 F 3 "" H 8350 900 60  0000 C CNN
 F 4 "64m" H 8350 900 60  0001 C CNN "ESR"
@@
 P 9250 1150
 F 0 "L1" V 9200 1150 40  0000 C CNN
-F 1 "47U" V 9350 1150 40  0000 C CNN
-F 2 "" H 9250 1150 60  0000 C CNN
+F 1 "47u" V 9350 1150 40  0000 C CNN
+F 2 "Inductors:SELF-WE-TPC_M" H 9250 1150 60  0001 C CNN
 F 3 "" H 9250 1150 60  0000 C CNN
 	1    9250 1150
@@
 $EndComp
 $Comp
-L DIODESCH D10
+L DIODESCH D12
 U 1 1 5468BDE4
 P 8850 1450
-F 0 "D10" H 8850 1550 40  0000 C CNN
+F 0 "D12" H 8850 1550 40  0000 C CNN
 F 1 "MBR0530T1G" H 8850 1350 40  0000 C CNN
-F 2 "" H 8850 1450 60  0000 C CNN
+F 2 "" H 8850 1450 60  0001 C CNN
 F 3 "" H 8850 1450 60  0000 C CNN
 	1    8850 1450
@@
 $EndComp
 $Comp
-L R R41
+L R R43
 U 1 1 5468BE35
 P 9950 1400
-F 0 "R41" V 10030 1400 40  0000 C CNN
+F 0 "R43" V 10030 1400 40  0000 C CNN
 F 1 "28K" V 9957 1401 40  0000 C CNN
-F 2 "" V 9880 1400 30  0000 C CNN
+F 2 "Resistors_SMD:R_1206_HandSoldering" V 9880 1400 30  0001 C CNN
 F 3 "" H 9950 1400 30  0000 C CNN
 	1    9950 1400
@@
 $EndComp
 $Comp
-L R R42
+L R R44
 U 1 1 5468BEB5
 P 9950 2150
-F 0 "R42" V 10030 2150 40  0000 C CNN
+F 0 "R44" V 10030 2150 40  0000 C CNN
 F 1 "8.45K" V 9957 2151 40  0000 C CNN
-F 2 "" V 9880 2150 30  0000 C CNN
+F 2 "Resistors_SMD:R_1206_HandSoldering" V 9880 2150 30  0001 C CNN
 F 3 "" H 9950 2150 30  0000 C CNN
 	1    9950 2150
@@
 F 0 "C15" H 10400 1900 40  0000 L CNN
 F 1 "22U" H 10406 1715 40  0000 L CNN
-F 2 "" H 10438 1650 30  0000 C CNN
+F 2 "SMD_Packages:SMD-1206" H 10438 1650 30  0001 C CNN
 F 3 "" H 10400 1800 60  0000 C CNN
 	1    10400 1800
@@
 3.3V REGULATOR
 $Comp
-L LMR16006XDDC U6
+L LMR16006XDDC U7
 U 1 1 5468D235
 P 7400 3800
-F 0 "U6" H 7500 3400 60  0000 C CNN
+F 0 "U7" H 7500 3400 60  0000 C CNN
 F 1 "LMR16006XDDC" H 7450 4200 60  0000 C CNN
-F 2 "" H 7450 4200 60  0000 C CNN
+F 2 "SMD_Packages:SOT-23-6" H 7450 4200 60  0001 C CNN
 F 3 "" H 7450 4200 60  0000 C CNN
 	1    7400 3800
@@
 F 0 "C12" H 6400 3950 40  0000 L CNN
 F 1 "4.7U" H 6406 3765 40  0000 L CNN
-F 2 "" H 6438 3700 30  0000 C CNN
+F 2 "SMD_Packages:SMD-1206" H 6438 3700 30  0001 C CNN
 F 3 "" H 6400 3850 60  0000 C CNN
 F 4 "3m" H 6400 3850 60  0001 C CNN "ESR"
@@
 F 0 "C14" H 8350 3650 40  0000 L CNN
 F 1 "100n" H 8356 3465 40  0000 L CNN
-F 2 "" H 8388 3400 30  0000 C CNN
+F 2 "SMD_Packages:SMD-1206" H 8388 3400 30  0001 C CNN
 F 3 "" H 8350 3550 60  0000 C CNN
 F 4 "64m" H 8350 3550 60  0001 C CNN "ESR"
@@
 $EndComp
 $Comp
-L INDUCTOR 33u1
+L INDUCTOR U8
 U 1 1 5468D250
 P 9250 3800
-F 0 "33u1" V 9200 3800 40  0000 C CNN
-F 1 "INDUCTOR" V 9350 3800 40  0000 C CNN
-F 2 "" H 9250 3800 60  0000 C CNN
+F 0 "U8" V 9200 3800 40  0000 C CNN
+F 1 "33U" V 9350 3800 40  0000 C CNN
+F 2 "Inductors_NEOSID:Neosid_Inductor_SMS-ME3015" H 9250 3800 60  0001 C CNN
 F 3 "" H 9250 3800 60  0000 C CNN
 	1    9250 3800
@@
 $EndComp
 $Comp
-L DIODESCH D11
+L DIODESCH D13
 U 1 1 5468D256
 P 8850 4100
-F 0 "D11" H 8850 4200 40  0000 C CNN
+F 0 "D13" H 8850 4200 40  0000 C CNN
 F 1 "MBR0530T1G" H 8850 4000 40  0000 C CNN
-F 2 "" H 8850 4100 60  0000 C CNN
+F 2 "" H 8850 4100 60  0001 C CNN
 F 3 "" H 8850 4100 60  0000 C CNN
 	1    8850 4100
@@
 $EndComp
 $Comp
-L R R43
+L R R45
 U 1 1 5468D25C
 P 9950 4050
-F 0 "R43" V 10030 4050 40  0000 C CNN
+F 0 "R45" V 10030 4050 40  0000 C CNN
 F 1 "36K" V 9957 4051 40  0000 C CNN
-F 2 "" V 9880 4050 30  0000 C CNN
+F 2 "Resistors_SMD:R_1206_HandSoldering" V 9880 4050 30  0001 C CNN
 F 3 "" H 9950 4050 30  0000 C CNN
 	1    9950 4050
@@
 $EndComp
 $Comp
-L R R44
+L R R46
 U 1 1 5468D262
 P 9950 4800
-F 0 "R44" V 10030 4800 40  0000 C CNN
+F 0 "R46" V 10030 4800 40  0000 C CNN
 F 1 "6.49K" V 9957 4801 40  0000 C CNN
-F 2 "" V 9880 4800 30  0000 C CNN
+F 2 "Resistors_SMD:R_1206_HandSoldering" V 9880 4800 30  0001 C CNN
 F 3 "" H 9950 4800 30  0000 C CNN
 	1    9950 4800
@@
 F 0 "C16" H 10400 4550 40  0000 L CNN
 F 1 "4.7u" H 10406 4365 40  0000 L CNN
-F 2 "" H 10438 4300 30  0000 C CNN
+F 2 "SMD_Packages:SMD-1206" H 10438 4300 30  0001 C CNN
 F 3 "" H 10400 4450 60  0000 C CNN
 F 4 "4m" H 10400 4450 60  0001 C CNN "ESR"
@@
 ~PWR_SAVE
 $Comp
-L R R39
+L R R41
 U 1 1 54691105
 P 1350 5200
-F 0 "R39" V 1430 5200 40  0000 C CNN
+F 0 "R41" V 1430 5200 40  0000 C CNN
 F 1 "100K" V 1357 5201 40  0000 C CNN
-F 2 "" V 1280 5200 30  0000 C CNN
+F 2 "Resistors_SMD:R_1206_HandSoldering" V 1280 5200 30  0001 C CNN
 F 3 "" H 1350 5200 30  0000 C CNN
 	1    1350 5200
@@
 F 0 "Q7" H 1750 5401 40  0000 R CNN
 F 1 "MMBF170" H 1750 5700 40  0000 R CNN
-F 2 "SOT-23" H 1620 5652 29  0000 C CNN
+F 2 "SMD_Packages:SOT-23" H 1620 5652 29  0000 C CNN
 F 3 "" H 1750 5550 60  0000 C CNN
 	1    1750 5550
@@
 $EndComp
 $Comp
-L R R40
+L R R42
 U 1 1 5469125B
 P 1850 4950
-F 0 "R40" V 1930 4950 40  0000 C CNN
+F 0 "R42" V 1930 4950 40  0000 C CNN
 F 1 "100K" V 1857 4951 40  0000 C CNN
-F 2 "" V 1780 4950 30  0000 C CNN
+F 2 "Resistors_SMD:R_1206_HandSoldering" V 1780 4950 30  0001 C CNN
 F 3 "" H 1850 4950 30  0000 C CNN
 	1    1850 4950
@@
 F 0 "Q8" H 2750 6340 60  0000 R CNN
 F 1 "MOSFET_P" H 2750 5970 60  0000 R CNN
-F 2 "" H 2750 6150 60  0000 C CNN
+F 2 "Transistors_TO-220:TO-220_FET-GDS_Horizontal_LargePads" H 2750 6150 60  0001 C CNN
 F 3 "" H 2750 6150 60  0000 C CNN
 	1    2750 6150
@@
 F 0 "Q9" H 3750 6340 60  0000 R CNN
 F 1 "MOSFET_P" H 3750 5970 60  0000 R CNN
-F 2 "" H 3750 6150 60  0000 C CNN
+F 2 "Transistors_TO-220:TO-220_FET-GDS_Horizontal_LargePads" H 3750 6150 60  0001 C CNN
 F 3 "" H 3750 6150 60  0000 C CNN
 	1    3750 6150

Commit message: General fine tuning of schematics. Need to review JTAG and update. Added resistors to power stage. Getting prepped for BOM, need to go through item by item. Added current incomplete BOM
Parts:
- added R49, R50: 100K, symbol R
- C10: value C -> 47u; footprint SMD_Packages:SMD-1206 -> SMD_Packages:SMD-0805
- C11, C12, C13, C14, C15, C16: footprint SMD_Packages:SMD-1206 -> SMD_Packages:SMD-0805
- C9: value C -> 10n; footprint SMD_Packages:SMD-1206 -> SMD_Packages:SMD-0805
Connections:
- net BAT: now also R49.1, R50.1
- net at U6.4 (~SHDN): now also R49.2
- net at U7.4 (~SHDN): now also R50.2
- no-connect marks 2 -> 0
Changed lines of the file:
@@
 P 2550 1200
 F 0 "C9" H 2550 1300 40  0000 L CNN
-F 1 "C" H 2556 1115 40  0000 L CNN
-F 2 "SMD_Packages:SMD-1206" H 2588 1050 30  0001 C CNN
+F 1 "10n" H 2556 1115 40  0000 L CNN
+F 2 "SMD_Packages:SMD-0805" H 2588 1050 30  0001 C CNN
 F 3 "" H 2550 1200 60  0000 C CNN
 	1    2550 1200
@@
 P 4050 1200
 F 0 "C10" H 4050 1300 40  0000 L CNN
-F 1 "C" H 4056 1115 40  0000 L CNN
-F 2 "SMD_Packages:SMD-1206" H 4088 1050 30  0001 C CNN
+F 1 "47u" H 4056 1115 40  0000 L CNN
+F 2 "SMD_Packages:SMD-0805" H 4088 1050 30  0001 C CNN
 F 3 "" H 4050 1200 60  0000 C CNN
 	1    4050 1200
@@
 F 0 "C11" H 6400 1300 40  0000 L CNN
 F 1 "4.7U" H 6406 1115 40  0000 L CNN
-F 2 "SMD_Packages:SMD-1206" H 6438 1050 30  0001 C CNN
+F 2 "SMD_Packages:SMD-0805" H 6438 1050 30  0001 C CNN
 F 3 "" H 6400 1200 60  0000 C CNN
 F 4 "3.0m" H 6400 1200 60  0001 C CNN "ESR"
@@
 F 0 "C13" H 8350 1000 40  0000 L CNN
 F 1 "100n" H 8356 815 40  0000 L CNN
-F 2 "SMD_Packages:SMD-1206" H 8388 750 30  0001 C CNN
+F 2 "SMD_Packages:SMD-0805" H 8388 750 30  0001 C CNN
 F 3 "" H 8350 900 60  0000 C CNN
 F 4 "64m" H 8350 900 60  0001 C CNN "ESR"
@@
 F 0 "C15" H 10400 1900 40  0000 L CNN
 F 1 "22U" H 10406 1715 40  0000 L CNN
-F 2 "SMD_Packages:SMD-1206" H 10438 1650 30  0001 C CNN
+F 2 "SMD_Packages:SMD-0805" H 10438 1650 30  0001 C CNN
 F 3 "" H 10400 1800 60  0000 C CNN
 	1    10400 1800
@@
 Text HLabel 10400 2500 3    60   Input ~ 0
 GND
-NoConn ~ 6950 1150
 Text Notes 6000 2850 0    60   ~ 0
 3.3V REGULATOR
@@
 F 0 "C12" H 6400 3950 40  0000 L CNN
 F 1 "4.7U" H 6406 3765 40  0000 L CNN
-F 2 "SMD_Packages:SMD-1206" H 6438 3700 30  0001 C CNN
+F 2 "SMD_Packages:SMD-0805" H 6438 3700 30  0001 C CNN
 F 3 "" H 6400 3850 60  0000 C CNN
 F 4 "3m" H 6400 3850 60  0001 C CNN "ESR"
@@
 F 0 "C14" H 8350 3650 40  0000 L CNN
 F 1 "100n" H 8356 3465 40  0000 L CNN
-F 2 "SMD_Packages:SMD-1206" H 8388 3400 30  0001 C CNN
+F 2 "SMD_Packages:SMD-0805" H 8388 3400 30  0001 C CNN
 F 3 "" H 8350 3550 60  0000 C CNN
 F 4 "64m" H 8350 3550 60  0001 C CNN "ESR"
@@
 F 0 "C16" H 10400 4550 40  0000 L CNN
 F 1 "4.7u" H 10406 4365 40  0000 L CNN
-F 2 "SMD_Packages:SMD-1206" H 10438 4300 30  0001 C CNN
+F 2 "SMD_Packages:SMD-0805" H 10438 4300 30  0001 C CNN
 F 3 "" H 10400 4450 60  0000 C CNN
 F 4 "4m" H 10400 4450 60  0001 C CNN "ESR"
@@
 Text HLabel 10400 5150 3    60   Input ~ 0
 GND
-NoConn ~ 6950 3800
 Text Notes 6000 5500 0    60   ~ 0
 5V REGULATOR
@@
 Wire Wire Line
 	4050 6250 4050 5900
+$Comp
+L R R50
+U 1 1 5474860C
+P 6650 3850
+F 0 "R50" V 6730 3850 40  0000 C CNN
+F 1 "100K" V 6657 3851 40  0000 C CNN
+F 2 "" V 6580 3850 30  0001 C CNN
+F 3 "" H 6650 3850 30  0000 C CNN
+	1    6650 3850
+	1    0    0    -1
+$EndComp
+Wire Wire Line
+	6950 3800 6800 3800
+Wire Wire Line
+	6800 3800 6800 4100
+Wire Wire Line
+	6800 4100 6650 4100
+Wire Wire Line
+	6650 3600 6650 3550
+Connection ~ 6650 3550
+$Comp
+L R R49
+U 1 1 54748CEF
+P 6650 1200
+F 0 "R49" V 6730 1200 40  0000 C CNN
+F 1 "100K" V 6657 1201 40  0000 C CNN
+F 2 "" V 6580 1200 30  0001 C CNN
+F 3 "" H 6650 1200 30  0000 C CNN
+	1    6650 1200
+	1    0    0    -1
+$EndComp
+Wire Wire Line
+	6950 1150 6800 1150
+Wire Wire Line
+	6800 1150 6800 1450
+Wire Wire Line
+	6800 1450 6650 1450
+Wire Wire Line
+	6650 950  6650 900
+Connection ~ 6650 900
 $EndSCHEMATC
