File: POWER.sch (KiCad schematic (older format))
At the start: 28 parts, among them Q7 MMBF170, Q8 MOSFET_P, Q9 MOSFET_P, U6 LMR16006XDDC, U7 LMR16006XDDC, U8 33U

Commit message: Updated parts and data sheets
Parts:
- removed Q7: MMBF170, SMD_Packages:SOT-23, symbol MMBF170
- removed Q8, Q9: MOSFET_P, Transistors_TO-220:TO-220_FET-GDS_Horizontal_LargePads, symbol MOSFET_P
- added Q7: DMN3730U, Transistors_SMD:sot23, symbol MOSFET_N
- added Q8, Q9: ZXMP6A13F, Transistors_SMD:sot23, symbol ZXMP6A13F
- C10, C9: footprint SMD_Packages:SMD-0805 -> Capacitors_SMD:C_0805_HandSoldering
- C11, C12: footprint SMD_Packages:SMD-0805 -> Capacitors_SMD:C_1206_HandSoldering; Part Number (none) -> GRM31CR71H475KA12L
- C13, C14: footprint SMD_Packages:SMD-0805 -> Capacitors_SMD:C_0805_HandSoldering; Part Number (none) -> C0805C104K5RACTU
- C15: footprint SMD_Packages:SMD-0805 -> Capacitors_SMD:C_0805_HandSoldering; ESR (none) -> 9m; Part Number (none) -> GRM21BR60J226ME39L
- C16: footprint SMD_Packages:SMD-0805 -> Capacitors_SMD:C_0805_HandSoldering; Part Number (none) -> C0805C475K8PACTU
- D10: value TVS -> SMAJ12CA; footprint Diodes_SMD:Diode-SMB_Standard -> (none)
- D11: footprint Diodes_SMD:Diode-SMB_Standard -> (none)
- D12: NOTE: (none) -> Create SOD-123 Footprint
- F1: value PTC_FUSE -> 1206L075/13.2; footprint (none) -> SMD_Packages:SMD-1206
- L1: footprint Inductors:SELF-WE-TPC_M -> (none); NOTE: (none) -> Create SDR0604 Footprint; Part Number (none) -> SDR0604-470KL
- L2: renamed from U8; footprint Inductors_NEOSID:Neosid_Inductor_SMS-ME3015 -> (none); Part Number (none) -> SRN3015-330M
- R41, R42, R43, R44, R45, R46: footprint Resistors_SMD:R_1206_HandSoldering -> Resistors_SMD:R_0805_HandSoldering
- R49, R50: footprint (none) -> Resistors_SMD:R_0805_HandSoldering
- U6: value LMR16006XDDC -> LMR16006XDDCT
- U7: value LMR16006XDDC -> LMR16006YDDC
Connections:
- net 5V: now also Q9.2 (S)
- net 5V_SW: now also Q9.3 (D)
- net BAT: now also Q8.2 (S)
- net BAT_SW: now also Q8.3 (D)
- net GND: now also Q7.S
- net ~PWR_SAVE: now also Q7.G
- net at R42.2: now also Q7.D, Q8.1 (G), Q9.1 (G)
Other:
- moved on the sheet: R41
Changed lines of the file:
@@
 P 7400 1150
 F 0 "U6" H 7500 750 60  0000 C CNN
-F 1 "LMR16006XDDC" H 7450 1550 60  0000 C CNN
+F 1 "LMR16006XDDCT" H 7450 1550 60  0000 C CNN
 F 2 "SMD_Packages:SOT-23-6" H 7450 1550 60  0001 C CNN
 F 3 "" H 7450 1550 60  0000 C CNN
@@
 F 0 "C9" H 2550 1300 40  0000 L CNN
 F 1 "10n" H 2556 1115 40  0000 L CNN
-F 2 "SMD_Packages:SMD-0805" H 2588 1050 30  0001 C CNN
+F 2 "Capacitors_SMD:C_0805_HandSoldering" H 2588 1050 30  0001 C CNN
 F 3 "" H 2550 1200 60  0000 C CNN
 	1    2550 1200
@@
 P 3300 1300
 F 0 "D10" H 3300 1450 60  0000 C CNN
-F 1 "TVS" H 3300 1150 60  0000 C CNN
-F 2 "Diodes_SMD:Diode-SMB_Standard" H 3300 1300 60  0001 C CNN
+F 1 "SMAJ12CA" H 3300 1150 60  0000 C CNN
+F 2 "" H 3300 1300 60  0001 C CNN
 F 3 "" H 3300 1300 60  0000 C CNN
 	1    3300 1300
@@
 F 0 "C10" H 4050 1300 40  0000 L CNN
 F 1 "47u" H 4056 1115 40  0000 L CNN
-F 2 "SMD_Packages:SMD-0805" H 4088 1050 30  0001 C CNN
+F 2 "Capacitors_SMD:C_0805_HandSoldering" H 4088 1050 30  0001 C CNN
 F 3 "" H 4050 1200 60  0000 C CNN
 	1    4050 1200
@@
 P 2950 900
 F 0 "F1" H 3050 950 40  0000 C CNN
-F 1 "PTC_FUSE" H 2850 850 40  0000 C CNN
-F 2 "" H 2950 900 60  0001 C CNN
+F 1 "1206L075/13.2" H 2850 850 40  0000 C CNN
+F 2 "SMD_Packages:SMD-1206" H 2950 900 60  0001 C CNN
 F 3 "" H 2950 900 60  0000 C CNN
 	1    2950 900
@@
 F 0 "D11" H 3700 1000 40  0000 C CNN
 F 1 "S2A" H 3700 800 40  0000 C CNN
-F 2 "Diodes_SMD:Diode-SMB_Standard" H 3700 900 60  0001 C CNN
+F 2 "" H 3700 900 60  0001 C CNN
 F 3 "" H 3700 900 60  0000 C CNN
 	1    3700 900
@@
 F 0 "C11" H 6400 1300 40  0000 L CNN
 F 1 "4.7U" H 6406 1115 40  0000 L CNN
-F 2 "SMD_Packages:SMD-0805" H 6438 1050 30  0001 C CNN
+F 2 "Capacitors_SMD:C_1206_HandSoldering" H 6438 1050 30  0001 C CNN
 F 3 "" H 6400 1200 60  0000 C CNN
 F 4 "3.0m" H 6400 1200 60  0001 C CNN "ESR"
+F 5 "GRM31CR71H475KA12L" H 6400 1200 60  0001 C CNN "Part Number"
 	1    6400 1200
 	1    0    0    -1
@@
 F 0 "C13" H 8350 1000 40  0000 L CNN
 F 1 "100n" H 8356 815 40  0000 L CNN
-F 2 "SMD_Packages:SMD-0805" H 8388 750 30  0001 C CNN
+F 2 "Capacitors_SMD:C_0805_HandSoldering" H 8388 750 30  0001 C CNN
 F 3 "" H 8350 900 60  0000 C CNN
 F 4 "64m" H 8350 900 60  0001 C CNN "ESR"
+F 5 "C0805C104K5RACTU" H 8350 900 60  0001 C CNN "Part Number"
 	1    8350 900
 	0    1    1    0
@@
 F 0 "L1" V 9200 1150 40  0000 C CNN
 F 1 "47u" V 9350 1150 40  0000 C CNN
-F 2 "Inductors:SELF-WE-TPC_M" H 9250 1150 60  0001 C CNN
+F 2 "" H 9250 1150 60  0001 C CNN
 F 3 "" H 9250 1150 60  0000 C CNN
+F 4 "SDR0604-470KL" V 9250 1150 60  0001 C CNN "Part Number"
+F 5 "Create SDR0604 Footprint" V 9250 1150 60  0001 C CNN "NOTE:"
 	1    9250 1150
 	0    -1   -1   0
@@
 F 2 "" H 8850 1450 60  0001 C CNN
 F 3 "" H 8850 1450 60  0000 C CNN
+F 4 "Create SOD-123 Footprint" H 8850 1450 60  0001 C CNN "NOTE:"
 	1    8850 1450
 	0    -1   -1   0
@@
 F 0 "R43" V 10030 1400 40  0000 C CNN
 F 1 "28K" V 9957 1401 40  0000 C CNN
-F 2 "Resistors_SMD:R_1206_HandSoldering" V 9880 1400 30  0001 C CNN
+F 2 "Resistors_SMD:R_0805_HandSoldering" V 9880 1400 30  0001 C CNN
 F 3 "" H 9950 1400 30  0000 C CNN
 	1    9950 1400
@@
 F 0 "R44" V 10030 2150 40  0000 C CNN
 F 1 "8.45K" V 9957 2151 40  0000 C CNN
-F 2 "Resistors_SMD:R_1206_HandSoldering" V 9880 2150 30  0001 C CNN
+F 2 "Resistors_SMD:R_0805_HandSoldering" V 9880 2150 30  0001 C CNN
 F 3 "" H 9950 2150 30  0000 C CNN
 	1    9950 2150
@@
 F 0 "C15" H 10400 1900 40  0000 L CNN
 F 1 "22U" H 10406 1715 40  0000 L CNN
-F 2 "SMD_Packages:SMD-0805" H 10438 1650 30  0001 C CNN
+F 2 "Capacitors_SMD:C_0805_HandSoldering" H 10438 1650 30  0001 C CNN
 F 3 "" H 10400 1800 60  0000 C CNN
+F 4 "9m" H 10400 1800 60  0001 C CNN "ESR"
+F 5 "GRM21BR60J226ME39L" H 10400 1800 60  0001 C CNN "Part Number"
 	1    10400 1800
 	1    0    0    -1
@@
 P 7400 3800
 F 0 "U7" H 7500 3400 60  0000 C CNN
-F 1 "LMR16006XDDC" H 7450 4200 60  0000 C CNN
+F 1 "LMR16006YDDC" H 7450 4200 60  0000 C CNN
 F 2 "SMD_Packages:SOT-23-6" H 7450 4200 60  0001 C CNN
 F 3 "" H 7450 4200 60  0000 C CNN
@@
 F 0 "C12" H 6400 3950 40  0000 L CNN
 F 1 "4.7U" H 6406 3765 40  0000 L CNN
-F 2 "SMD_Packages:SMD-0805" H 6438 3700 30  0001 C CNN
+F 2 "Capacitors_SMD:C_1206_HandSoldering" H 6438 3700 30  0001 C CNN
 F 3 "" H 6400 3850 60  0000 C CNN
 F 4 "3m" H 6400 3850 60  0001 C CNN "ESR"
+F 5 "GRM31CR71H475KA12L" H 6400 3850 60  0001 C CNN "Part Number"
 	1    6400 3850
 	1    0    0    -1
@@
 F 0 "C14" H 8350 3650 40  0000 L CNN
 F 1 "100n" H 8356 3465 40  0000 L CNN
-F 2 "SMD_Packages:SMD-0805" H 8388 3400 30  0001 C CNN
+F 2 "Capacitors_SMD:C_0805_HandSoldering" H 8388 3400 30  0001 C CNN
 F 3 "" H 8350 3550 60  0000 C CNN
 F 4 "64m" H 8350 3550 60  0001 C CNN "ESR"
+F 5 "C0805C104K5RACTU" H 8350 3550 60  0001 C CNN "Part Number"
 	1    8350 3550
 	0    1    1    0
 $EndComp
 $Comp
-L INDUCTOR U8
+L INDUCTOR L2
 U 1 1 5468D250
 P 9250 3800
-F 0 "U8" V 9200 3800 40  0000 C CNN
+F 0 "L2" V 9200 3800 40  0000 C CNN
 F 1 "33U" V 9350 3800 40  0000 C CNN
-F 2 "Inductors_NEOSID:Neosid_Inductor_SMS-ME3015" H 9250 3800 60  0001 C CNN
+F 2 "" H 9250 3800 60  0001 C CNN
 F 3 "" H 9250 3800 60  0000 C CNN
+F 4 "SRN3015-330M" V 9250 3800 60  0001 C CNN "Part Number"
 	1    9250 3800
 	0    -1   -1   0
@@
 F 0 "R45" V 10030 4050 40  0000 C CNN
 F 1 "36K" V 9957 4051 40  0000 C CNN
-F 2 "Resistors_SMD:R_1206_HandSoldering" V 9880 4050 30  0001 C CNN
+F 2 "Resistors_SMD:R_0805_HandSoldering" V 9880 4050 30  0001 C CNN
 F 3 "" H 9950 4050 30  0000 C CNN
 	1    9950 4050
@@
 F 0 "R46" V 10030 4800 40  0000 C CNN
 F 1 "6.49K" V 9957 4801 40  0000 C CNN
-F 2 "Resistors_SMD:R_1206_HandSoldering" V 9880 4800 30  0001 C CNN
+F 2 "Resistors_SMD:R_0805_HandSoldering" V 9880 4800 30  0001 C CNN
 F 3 "" H 9950 4800 30  0000 C CNN
 	1    9950 4800
@@
 F 0 "C16" H 10400 4550 40  0000 L CNN
 F 1 "4.7u" H 10406 4365 40  0000 L CNN
-F 2 "SMD_Packages:SMD-0805" H 10438 4300 30  0001 C CNN
+F 2 "Capacitors_SMD:C_0805_HandSoldering" H 10438 4300 30  0001 C CNN
 F 3 "" H 10400 4450 60  0000 C CNN
 F 4 "4m" H 10400 4450 60  0001 C CNN "ESR"
+F 5 "C0805C475K8PACTU" H 10400 4450 60  0001 C CNN "Part Number"
 	1    10400 4450
 	1    0    0    -1
@@
 Text HLabel 10550 3800 2    60   Output ~ 0
 5V
-Text HLabel 1100 5600 0    60   Input ~ 0
+Text HLabel 1100 5550 0    60   Input ~ 0
 ~PWR_SAVE
 $Comp
 L R R41
 U 1 1 54691105
-P 1350 5200
-F 0 "R41" V 1430 5200 40  0000 C CNN
-F 1 "100K" V 1357 5201 40  0000 C CNN
-F 2 "Resistors_SMD:R_1206_HandSoldering" V 1280 5200 30  0001 C CNN
-F 3 "" H 1350 5200 30  0000 C CNN
-	1    1350 5200
-	1    0    0    -1
-$EndComp
-$Comp
-L MMBF170 Q7
-U 1 1 54691154
-P 1750 5550
-F 0 "Q7" H 1750 5401 40  0000 R CNN
-F 1 "MMBF170" H 1750 5700 40  0000 R CNN
-F 2 "SMD_Packages:SOT-23" H 1620 5652 29  0000 C CNN
-F 3 "" H 1750 5550 60  0000 C CNN
-	1    1750 5550
+P 1350 5150
+F 0 "R41" V 1430 5150 40  0000 C CNN
+F 1 "100K" V 1357 5151 40  0000 C CNN
+F 2 "Resistors_SMD:R_0805_HandSoldering" V 1280 5150 30  0001 C CNN
+F 3 "" H 1350 5150 30  0000 C CNN
+	1    1350 5150
 	1    0    0    -1
 $EndComp
@@
 F 0 "R42" V 1930 4950 40  0000 C CNN
 F 1 "100K" V 1857 4951 40  0000 C CNN
-F 2 "Resistors_SMD:R_1206_HandSoldering" V 1780 4950 30  0001 C CNN
+F 2 "Resistors_SMD:R_0805_HandSoldering" V 1780 4950 30  0001 C CNN
 F 3 "" H 1850 4950 30  0000 C CNN
 	1    1850 4950
@@
 Text HLabel 1850 4550 1    60   Input ~ 0
 BAT
-Text HLabel 1350 4800 1    60   Input ~ 0
+Text HLabel 1350 4750 1    60   Input ~ 0
 3.3V
 Text HLabel 2450 5900 1    60   Input ~ 0
@@
 Text HLabel 4050 5900 1    60   Output ~ 0
 5V_SW
-$Comp
-L MOSFET_P Q8
-U 1 1 54693107
-P 2750 6150
-F 0 "Q8" H 2750 6340 60  0000 R CNN
-F 1 "MOSFET_P" H 2750 5970 60  0000 R CNN
-F 2 "Transistors_TO-220:TO-220_FET-GDS_Horizontal_LargePads" H 2750 6150 60  0001 C CNN
-F 3 "" H 2750 6150 60  0000 C CNN
-	1    2750 6150
-	0    1    1    0
-$EndComp
-$Comp
-L MOSFET_P Q9
-U 1 1 54693157
-P 3750 6150
-F 0 "Q9" H 3750 6340 60  0000 R CNN
-F 1 "MOSFET_P" H 3750 5970 60  0000 R CNN
-F 2 "Transistors_TO-220:TO-220_FET-GDS_Horizontal_LargePads" H 3750 6150 60  0001 C CNN
-F 3 "" H 3750 6150 60  0000 C CNN
-	1    3750 6150
-	0    1    1    0
-$EndComp
 Wire Wire Line
 	6850 1500 6850 1400
@@
 Connection ~ 10400 3800
 Wire Wire Line
-	1100 5600 1550 5600
-Wire Wire Line
-	1350 5450 1350 5600
-Connection ~ 1350 5600
-Wire Wire Line
-	1350 4950 1350 4800
+	1100 5550 1550 5550
+Wire Wire Line
+	1350 5400 1350 5550
+Connection ~ 1350 5550
+Wire Wire Line
+	1350 4900 1350 4750
 Wire Wire Line
 	1850 4550 1850 4700
@@
 F 0 "R50" V 6730 3850 40  0000 C CNN
 F 1 "100K" V 6657 3851 40  0000 C CNN
-F 2 "" V 6580 3850 30  0001 C CNN
+F 2 "Resistors_SMD:R_0805_HandSoldering" V 6580 3850 30  0001 C CNN
 F 3 "" H 6650 3850 30  0000 C CNN
 	1    6650 3850
@@
 F 0 "R49" V 6730 1200 40  0000 C CNN
 F 1 "100K" V 6657 1201 40  0000 C CNN
-F 2 "" V 6580 1200 30  0001 C CNN
+F 2 "Resistors_SMD:R_0805_HandSoldering" V 6580 1200 30  0001 C CNN
 F 3 "" H 6650 1200 30  0000 C CNN
 	1    6650 1200
@@
 	6650 950  6650 900
 Connection ~ 6650 900
+$Comp
+L MOSFET_N Q7
+U 1 1 5476B2EB
+P 1750 5550
+F 0 "Q7" H 1760 5720 60  0000 R CNN
+F 1 "DMN3730U" H 1760 5400 60  0000 R CNN
+F 2 "Transistors_SMD:sot23" H 1750 5300 60  0001 C CNN
+F 3 "" H 1750 5550 60  0000 C CNN
+	1    1750 5550
+	1    0    0    -1
+$EndComp
+$Comp
+L ZXMP6A13F Q8
+U 1 1 54780A52
+P 2750 6150
+F 0 "Q8" H 2750 6340 60  0000 R CNN
+F 1 "ZXMP6A13F" H 2750 5970 60  0000 R CNN
+F 2 "Transistors_SMD:sot23" H 2750 6150 60  0001 C CNN
+F 3 "" H 2750 6150 60  0000 C CNN
+	1    2750 6150
+	0    1    1    0
+$EndComp
+$Comp
+L ZXMP6A13F Q9
+U 1 1 54780A91
+P 3750 6150
+F 0 "Q9" H 3750 6340 60  0000 R CNN
+F 1 "ZXMP6A13F" H 3750 5970 60  0000 R CNN
+F 2 "Transistors_SMD:sot23" H 3750 6150 60  0001 C CNN
+F 3 "" H 3750 6150 60  0000 C CNN
+	1    3750 6150
+	0    1    1    0
+$EndComp
 $EndSCHEMATC
