File: GEM.kicad_pcb (KiCad board)
At the start: 2 copper layers, 0 parts

Commit message: Linked components to footprints, may have to switch to smaller components. Started board layout.
Parts:
- added C1: 30p, SMD_Packages:SMD-1206, F.Cu at (121.5, 18.4)
- added C10: C, SMD_Packages:SMD-1206, F.Cu at (64.2, 65.3)
- added C11: 4.7U, SMD_Packages:SMD-1206, F.Cu at (63.2, 72.5)
- added C12: 4.7U, SMD_Packages:SMD-1206, F.Cu at (56.7, 76.5)
- added C13: 100n, SMD_Packages:SMD-1206, F.Cu at (64.2, 68.2)
- added C14: 100n, SMD_Packages:SMD-1206, F.Cu at (55.2, 80.0)
- added C15: 22U, SMD_Packages:SMD-1206, F.Cu at (62.5, 76.5)
- added C16: 4.7u, SMD_Packages:SMD-1206, F.Cu at (55.2, 83.0)
- added C17: 0.1U, SMD_Packages:SMD-1206, F.Cu at (76.3, 83.0)
- added C2: 30p, SMD_Packages:SMD-1206, F.Cu at (81.8, 40.5)
- added C3: 1u, SMD_Packages:SMD-1206, F.Cu at (87.5, 40.5)
- added C4: 1u, SMD_Packages:SMD-1206, F.Cu at (121.5, 21.3)
- added C5: 1U, SMD_Packages:SMD-1206, F.Cu at (125.6, 47.2)
- added C6: 560P, SMD_Packages:SMD-1206, F.Cu at (127.2, 53.8)
- added C7: 560P, SMD_Packages:SMD-1206, F.Cu at (125.6, 50.1)
- added C8: 0.1U, SMD_Packages:SMD-1206, F.Cu at (39.9, 34.4)
- added C9: C, SMD_Packages:SMD-1206, F.Cu at (62.4, 62.4)
- added D1: LED, LEDs:LED-1206, F.Cu at (97.4, 56.5)
- added D10: TVS, Diodes_SMD:Diode-SMB_Standard, F.Cu at (43.2, 59.7)
- added D11: S2A, Diodes_SMD:Diode-SMB_Standard, F.Cu at (50.5, 59.7)
- added D2: LED, LEDs:LED-1206, F.Cu at (102.3, 56.5)
- added D3: LED, LEDs:LED-1206, F.Cu at (97.4, 61.3)
- added D4: LED, LEDs:LED-1206, F.Cu at (102.3, 61.3)
- added D5: LED, LEDs:LED-1206, F.Cu at (97.4, 66.1)
- added D6: LED, LEDs:LED-1206, F.Cu at (102.3, 66.1)
- added D7: BAT46, Diodes_ThroughHole:Diode_DO-35_SOD27_Horizontal_RM10, F.Cu at (181.8, 73.7)
- added D8: BAT46, Diodes_ThroughHole:Diode_DO-35_SOD27_Horizontal_RM10, F.Cu at (181.6, 78.1)
- added D9: BAT46, Diodes_ThroughHole:Diode_DO-35_SOD27_Horizontal_RM10, F.Cu at (182.0, 69.0)
- added L1: 47u, Inductors:SELF-WE-TPC_M, F.Cu at (49.2, 81.5)
- added Q1: BC817-40, SMD_Packages:SOT-23, F.Cu at (60.9, 45.9)
- added Q2: BC817-40, SMD_Packages:SOT-23, F.Cu at (71.3, 18.7)
- added Q3: BSS138, SMD_Packages:SOT-23, F.Cu at (70.5, 42.8)
- added Q4: MMBT3646, SMD_Packages:SOT-23, F.Cu at (68.0, 39.1)
- added Q5: MMBT3646, SMD_Packages:SOT-23, F.Cu at (65.9, 45.9)
- added Q6: MMBT3640, SMD_Packages:SOT-23, F.Cu at (73.1, 39.1)
- added Q7: MMBF170, SMD_Packages:SOT-23, F.Cu at (60.0, 79.8)
- added Q8: MOSFET_P, Transistors_TO-220:TO-220_FET-GDS_Horizontal_LargePads, F.Cu at (183.4, 60.6)
- added Q9: MOSFET_P, Transistors_TO-220:TO-220_FET-GDS_Horizontal_LargePads, F.Cu at (156.8, 60.5)
- added R1: 100K, Resistors_SMD:R_1206_HandSoldering, F.Cu at (98.3, 30.5)
- added R10: 100, Resistors_SMD:R_1206_HandSoldering, F.Cu at (119.1, 56.0)
- added R11: 330, Resistors_SMD:R_1206_HandSoldering, F.Cu at (77.0, 57.6)
- added R12: 330, Resistors_SMD:R_1206_HandSoldering, F.Cu at (91.3, 64.4)
- added R13: 330, Resistors_SMD:R_1206_HandSoldering, F.Cu at (77.0, 64.4)
- added R14: 330, Resistors_SMD:R_1206_HandSoldering, F.Cu at (84.2, 57.6)
- added R15: 330, Resistors_SMD:R_1206_HandSoldering, F.Cu at (84.2, 64.4)
- added R16: 330, Resistors_SMD:R_1206_HandSoldering, F.Cu at (91.3, 57.6)
- added R17: 10K, Resistors_SMD:R_1206_HandSoldering, F.Cu at (65.5, 20.4)
- added R18: 10K, Resistors_SMD:R_1206_HandSoldering, F.Cu at (40.8, 46.2)
- added R19: 1K, Resistors_SMD:R_1206_HandSoldering, F.Cu at (54.9, 34.0)
- added R2: 10K, Resistors_SMD:R_1206_HandSoldering, F.Cu at (115.1, 20.4)
- added R20: 1K, Resistors_SMD:R_1206_HandSoldering, F.Cu at (62.1, 27.2)
- added R21: 10K, Resistors_SMD:R_1206_HandSoldering, F.Cu at (47.9, 40.8)
- added R22: 510 0.5W, Resistors_SMD:R_1206_HandSoldering, F.Cu at (19.0, 46.9)
- added R23: 510 0.5W, Resistors_SMD:R_1206_HandSoldering, F.Cu at (43.7, 20.4)
- added R24: 10K, Resistors_SMD:R_1206_HandSoldering, F.Cu at (62.1, 34.0)
- added R25: 10K, Resistors_SMD:R_1206_HandSoldering, F.Cu at (55.1, 40.8)
- added R26: 374, Resistors_SMD:R_1206_HandSoldering, F.Cu at (69.2, 27.2)
- added R27: 1K, Resistors_SMD:R_1206_HandSoldering, F.Cu at (55.1, 47.6)
- added R28: 866, Resistors_SMD:R_1206_HandSoldering, F.Cu at (69.2, 34.0)
- added R29: 2.2K, Resistors_SMD:R_1206_HandSoldering, F.Cu at (54.9, 27.2)
- added R3: 1K, Resistors_SMD:R_1206_HandSoldering, F.Cu at (98.3, 37.3)
- added R30: 10K, Resistors_SMD:R_1206_HandSoldering, F.Cu at (62.2, 40.8)
- added R31: 10K, Resistors_SMD:R_1206_HandSoldering, F.Cu at (33.6, 46.2)
- added R32: 240, Resistors_SMD:R_1206_HandSoldering, F.Cu at (58.4, 20.4)
- added R33: 10K, Resistors_SMD:R_1206_HandSoldering, F.Cu at (29.5, 39.4)
- added R34: 2K, Resistors_SMD:R_1206_HandSoldering, F.Cu at (47.8, 27.2)
- added R35: 8K, Resistors_SMD:R_1206_HandSoldering, F.Cu at (47.8, 34.0)
- added R36: 10K, Resistors_SMD:R_1206_HandSoldering, F.Cu at (26.5, 46.9)
- added R37: 10K, Resistors_SMD:R_1206_HandSoldering, F.Cu at (40.6, 29.6)
- added R38: 10K, Resistors_SMD:R_1206_HandSoldering, F.Cu at (51.2, 20.4)
- added R39: 10K, Resistors_SMD:R_1206_HandSoldering, F.Cu at (47.9, 47.6)
- added R4: 100K, Resistors_SMD:R_1206_HandSoldering, F.Cu at (105.5, 30.5)
- added R40: 10K, Resistors_SMD:R_1206_HandSoldering, F.Cu at (36.7, 39.4)
- added R41: 100K, Resistors_SMD:R_1206_HandSoldering, F.Cu at (43.2, 68.4)
- added R42: 100K, Resistors_SMD:R_1206_HandSoldering, F.Cu at (50.3, 68.4)
- added R43: 28K, Resistors_SMD:R_1206_HandSoldering, F.Cu at (50.3, 75.2)
- added R44: 8.45K, Resistors_SMD:R_1206_HandSoldering, F.Cu at (63.1, 57.6)
- added R45: 36K, Resistors_SMD:R_1206_HandSoldering, F.Cu at (57.8, 67.7)
- added R46: 6.49K, Resistors_SMD:R_1206_HandSoldering, F.Cu at (43.2, 75.2)
- added R47: 62K, Resistors_SMD:R_1206_HandSoldering, F.Cu at (84.2, 78.2)
- added R48: 10K, Resistors_SMD:R_1206_HandSoldering, F.Cu at (77.0, 78.2)
- added R5: 10, Resistors_SMD:R_1206_HandSoldering, F.Cu at (115.1, 27.2)
- added R6: 100K, Resistors_SMD:R_1206_HandSoldering, F.Cu at (105.5, 37.3)
- added R7: 1K, Resistors_SMD:R_1206_HandSoldering, F.Cu at (112.6, 34.0)
- added R8: 4.7K, Resistors_SMD:R_1206_HandSoldering, F.Cu at (119.1, 49.2)
- added R9: 100, Resistors_SMD:R_1206_HandSoldering, F.Cu at (111.4, 57.2)
- added U1: STN1110, SMD_Packages:SOIC-28, F.Cu at (160.5, 98.3)
- added U10: C, Capacitors_SMD:C_1206_HandSoldering, F.Cu at (105.8, 95.2)
- added U11: MSP430F247, SMD_Packages:TQFP-64, F.Cu at (181.3, 107.8)
- added U2: 10U ESR<5, Capacitors_Tantalum_SMD:TantalC_SizeD_EIA-7343_Wave, F.Cu at (104.5, 22.0)
- added U3: MCP2551, SMD_Packages:SOIC-8-N, F.Cu at (111.7, 49.7)
- added U4: LM339, SMD_Packages:SOIC-14_N, F.Cu at (182.6, 92.9)
- added U5: LM317AEMP, SMD_Packages:SOT-223, F.Cu at (157.4, 74.6)
- added U6: LMR16006XDDC, SMD_Packages:SOT-23-6, F.Cu at (42.7, 80.6)
- added U7: LMR16006XDDC, SMD_Packages:SOT-23-6, F.Cu at (57.0, 73.0)
- added U8: 33U, Inductors_NEOSID:Neosid_Inductor_SMS-ME3015, F.Cu at (57.2, 59.1)
- added U9: CP1, Capacitors_SMD:C_1206_HandSoldering, F.Cu at (125.4, 67.2)
- added X1: 16Mhz, Crystals:Crystal_HC49-SD_SMD, F.Cu at (169.7, 95.6)
Other:
- board outline added: 38.1 x 76.2 mm
- copper layers 2 -> 4

Commit message: General fine tuning of schematics. Need to review JTAG and update. Added resistors to power stage. Getting prepped for BOM, need to go through item by item. Added current incomplete BOM
Parts:
- removed C1, C2: 30p, SMD_Packages:SMD-1206
- removed C10, C9: C, SMD_Packages:SMD-1206
- removed C11, C12: 4.7U, SMD_Packages:SMD-1206
- removed C13, C14: 100n, SMD_Packages:SMD-1206
- removed C15: 22U, SMD_Packages:SMD-1206
- removed C16: 4.7u, SMD_Packages:SMD-1206
- removed C17, C8: 0.1U, SMD_Packages:SMD-1206
- removed C3, C4: 1u, SMD_Packages:SMD-1206
- removed C5: 1U, SMD_Packages:SMD-1206
- removed C6, C7: 560P, SMD_Packages:SMD-1206
- removed D1, D2, D3, D4, D5, D6: LED, LEDs:LED-1206
- removed D10: TVS, Diodes_SMD:Diode-SMB_Standard
- removed D11: S2A, Diodes_SMD:Diode-SMB_Standard
- removed D7, D8, D9: BAT46, Diodes_ThroughHole:Diode_DO-35_SOD27_Horizontal_RM10
- removed L1: 47u, Inductors:SELF-WE-TPC_M
- removed Q1, Q2: BC817-40, SMD_Packages:SOT-23
- removed Q3: BSS138, SMD_Packages:SOT-23
- removed Q4, Q5: MMBT3646, SMD_Packages:SOT-23
- removed Q6: MMBT3640, SMD_Packages:SOT-23
- removed Q7: MMBF170, SMD_Packages:SOT-23
- removed Q8, Q9: MOSFET_P, Transistors_TO-220:TO-220_FET-GDS_Horizontal_LargePads
- removed R1, R4, R41, R42, R6: 100K, Resistors_SMD:R_1206_HandSoldering
- removed R10, R9: 100, Resistors_SMD:R_1206_HandSoldering
- removed R11, R12, R13, R14, R15, R16: 330, Resistors_SMD:R_1206_HandSoldering
- removed R17, R18, R2, R21, R24, R25, R30, R31, R33, R36, R37, R38, R39, R40, R48: 10K, Resistors_SMD:R_1206_HandSoldering
- removed R19, R20, R27, R3, R7: 1K, Resistors_SMD:R_1206_HandSoldering
- removed R22, R23: 510 0.5W, Resistors_SMD:R_1206_HandSoldering
- removed R26: 374, Resistors_SMD:R_1206_HandSoldering
- removed R28: 866, Resistors_SMD:R_1206_HandSoldering
- removed R29: 2.2K, Resistors_SMD:R_1206_HandSoldering
- removed R32: 240, Resistors_SMD:R_1206_HandSoldering
- removed R34: 2K, Resistors_SMD:R_1206_HandSoldering
- removed R35: 8K, Resistors_SMD:R_1206_HandSoldering
- removed R43: 28K, Resistors_SMD:R_1206_HandSoldering
- removed R44: 8.45K, Resistors_SMD:R_1206_HandSoldering
- removed R45: 36K, Resistors_SMD:R_1206_HandSoldering
- removed R46: 6.49K, Resistors_SMD:R_1206_HandSoldering
- removed R47: 62K, Resistors_SMD:R_1206_HandSoldering
- removed R5: 10, Resistors_SMD:R_1206_HandSoldering
- removed R8: 4.7K, Resistors_SMD:R_1206_HandSoldering
- removed U1: STN1110, SMD_Packages:SOIC-28
- removed U10: C, Capacitors_SMD:C_1206_HandSoldering
- removed U11: MSP430F247, SMD_Packages:TQFP-64
- removed U2: 10U ESR<5, Capacitors_Tantalum_SMD:TantalC_SizeD_EIA-7343_Wave
- removed U3: MCP2551, SMD_Packages:SOIC-8-N
- removed U4: LM339, SMD_Packages:SOIC-14_N
- removed U5: LM317AEMP, SMD_Packages:SOT-223
- removed U6, U7: LMR16006XDDC, SMD_Packages:SOT-23-6
- removed U8: 33U, Inductors_NEOSID:Neosid_Inductor_SMS-ME3015
- removed U9: CP1, Capacitors_SMD:C_1206_HandSoldering
- removed X1: 16Mhz, Crystals:Crystal_HC49-SD_SMD
Other:
- board outline removed

Commit message: 1st Revision
Complete Board layout, 1st Draft
Parts:
- added C18: 2.2n, Capacitors_SMD:C_0805_HandSoldering, F.Cu at (142.8, 76.3)
- added C19: 10U, Capacitors_SMD:C_0805_HandSoldering, F.Cu at (143.0, 83.4)
- added C20: 0.1U, Capacitors_SMD:C_0805_HandSoldering, F.Cu at (143.0, 81.2)
- added D5: LED, LEDs:LED-0805, F.Cu at (182.9, 94.3)
- added D6: LED, LEDs:LED-0805, F.Cu at (186.5, 94.3)
- added JP2: JUMPER3, GEM:TESTPOINT3, F.Cu at (168.4, 94.4)
- added P1: CONN_01X04, GEM:P4, F.Cu at (173.6, 91.6)
- added R15: 330, Resistors_SMD:R_0805_HandSoldering, F.Cu at (182.9, 89.7)
- added R16: 330, Resistors_SMD:R_0805_HandSoldering, F.Cu at (186.5, 89.7)
- added R4: 47k, Resistors_SMD:R_0805_HandSoldering, F.Cu at (142.9, 78.5)
- added U11: MSP430F247, GEM:LQFP_64PIN_MSP430, F.Cu at (153.2, 80.8)
- added U12: RN4020, GEM:RN4020_BT, F.Cu at (188.0, 75.7)
- added U13: microSD, GEM:MicroSD_Slot, F.Cu at (170.1, 80.8)
- added U14: JTAG_HEADER, GEM:JTAG2X7, F.Cu at (151.9, 93.7)
Routing:
- net /MSP430F247/WAKE_HW: track 0.00 -> 80.9 mm, vias 0 -> 2
- net /MSP430F247/SPI/PIO: track 0.00 -> 69.5 mm, vias 0 -> 3
- net /JTAG/VCC/TOOL: track 0.00 -> 57.9 mm, vias 0 -> 2
- net /BreakoutPin4/GND: track 0.00 -> 53.6 mm, vias 0 -> 13
- net /JTAG/~RST: track 0.00 -> 45.9 mm, vias 0 -> 2
- net /MSP430F247/CMD: track 0.00 -> 44.8 mm, vias 0 -> 2
- net /MSP430F247/WAKE_SW: track 0.00 -> 40.8 mm
- net /BreakoutPin4/3.3V: track 0.00 -> 26.3 mm, vias 0 -> 2
- net /MSP430F247/UART_TX_BT: track 0.00 -> 25.5 mm, vias 0 -> 2
- net /MSP430F247/UART_RX_BT: track 0.00 -> 25.2 mm, vias 0 -> 2
- net /BreakoutPin4/UART_TX: track 0.00 -> 20.3 mm
- net /JTAG/TDO/TDI: track 0.00 -> 19.2 mm, vias 0 -> 2
- net /BreakoutPin4/UART_RX: track 0.00 -> 18.4 mm
- net /JTAG/TDI/VPP: track 0.00 -> 18.3 mm, vias 0 -> 2
- net /JTAG/TCK: track 0.00 -> 17.6 mm, vias 0 -> 2
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- added copper zone on F.Cu, net /BreakoutPin4/3.3V
- added copper zone on B.Cu, net /BreakoutPin4/GND
Other:
- board outline added: 63.5 x 35.6 mm
- net class Default: clearance 0.254 -> 0.2032
- rule trace_clearance: 0.254 -> 0.2032
- board text added: "GEM GROUP 8"
