File: JTAG.sch (KiCad schematic (older format))
At the start: 2 parts, among them U10 JTAG_HEADER

Commit message: Linked components to footprints, may have to switch to smaller components. Started board layout.
Parts:
- renumbered U10 to U14
Connections:
- no-connect marks 1 -> 0
Changed lines of the file:
@@
 $EndDescr
 $Comp
-L JTAG_HEADER U10
+L JTAG_HEADER U14
 U 1 1 5474BF80
 P 5900 3400
-F 0 "U10" H 5900 3400 60  0000 C TNN
+F 0 "U14" H 5900 3400 60  0000 C TNN
 F 1 "JTAG_HEADER" H 5900 3400 60  0000 C BNN
-F 2 "" H 5900 3400 60  0000 C CNN
+F 2 "" H 5900 3400 60  0001 C CNN
 F 3 "" H 5900 3400 60  0000 C CNN
 	1    5900 3400
@@
 F 0 "JP2" H 2550 2900 60  0000 C CNN
 F 1 "JUMPER" H 2550 2670 40  0000 C CNN
-F 2 "" H 2550 2750 60  0000 C CNN
+F 2 "" H 2550 2750 60  0001 C CNN
 F 3 "" H 2550 2750 60  0000 C CNN
 	1    2550 2750
@@
 Wire Wire Line
 	2950 3050 2550 3050
-Wire Wire Line
-	2550 3050 2550 3300
-NoConn ~ 2550 3300
 Text HLabel 7950 3300 2    60   Output ~ 0
 TCK

Commit message: General fine tuning of schematics. Need to review JTAG and update. Added resistors to power stage. Getting prepped for BOM, need to go through item by item. Added current incomplete BOM
Connections:
- net TDI/VPP: now reaches U14.3 (TDI/VPP)
- net TMS: now reaches U14.5 (TMS)
- net FUSE renamed TEST/VPP
Changed lines of the file:
@@
 $EndDescr
-$Comp
-L JTAG_HEADER U14
-U 1 1 5474BF80
-P 5900 3400
-F 0 "U14" H 5900 3400 60  0000 C TNN
-F 1 "JTAG_HEADER" H 5900 3400 60  0000 C BNN
-F 2 "" H 5900 3400 60  0001 C CNN
-F 3 "" H 5900 3400 60  0000 C CNN
-	1    5900 3400
-	1    0    0    -1
-$EndComp
 $Comp
 L JUMPER JP2
@@
 Wire Wire Line
 	6850 3300 7950 3300
-Text HLabel 3850 3300 0    60   Output ~ 0
-FUSE
-Wire Wire Line
-	4850 3300 3850 3300
 Text HLabel 7950 2700 2    60   BiDi ~ 0
 TDO/TDI
@@
 Wire Wire Line
 	7950 3500 6850 3500
+Text HLabel 7150 2900 2    60   Input ~ 0
+TDI/VPP
+$Comp
+L JTAG_HEADER U14
+U 1 1 5474BF80
+P 5900 3400
+F 0 "U14" H 5900 3400 60  0000 C TNN
+F 1 "JTAG_HEADER" H 5900 3400 60  0000 C BNN
+F 2 "" H 5900 3400 60  0001 C CNN
+F 3 "" H 5900 3400 60  0000 C CNN
+	1    5900 3400
+	1    0    0    -1
+$EndComp
+Wire Wire Line
+	7150 2900 6850 2900
+Text HLabel 7150 3100 2    60   Input ~ 0
+TMS
+Wire Wire Line
+	6850 3100 7150 3100
+Text HLabel 4550 3300 0    60   Input ~ 0
+TEST/VPP
+Wire Wire Line
+	4550 3300 4850 3300
 $EndSCHEMATC

Commit message: Updated parts and data sheets
Parts:
- added JP3: JUMPER, Connect:TESTPOINT, symbol JUMPER
- JP2: footprint (none) -> Connect:TESTPOINT
Connections:
- net 3.3V: now also JP2.2, JP3.2; no longer JP2.1, U14.2 (VCC/TOOL)
- net ~RST: now reaches U14.11 (~RST)
- net at U14.4 (VCC_TARG): now also JP3.1; no longer JP2.2
- new net: JP2.1, U14.2 (VCC/TOOL)
Other:
- moved on the sheet: JP2
Changed lines of the file:
@@
 L JUMPER JP2
 U 1 1 5474DC6F
-P 2550 2750
-F 0 "JP2" H 2550 2900 60  0000 C CNN
-F 1 "JUMPER" H 2550 2670 40  0000 C CNN
-F 2 "" H 2550 2750 60  0001 C CNN
-F 3 "" H 2550 2750 60  0000 C CNN
-	1    2550 2750
-	0    1    1    0
+P 3100 2400
+F 0 "JP2" H 3100 2550 60  0000 C CNN
+F 1 "JUMPER" H 3100 2320 40  0000 C CNN
+F 2 "Connect:TESTPOINT" H 3100 2400 60  0001 C CNN
+F 3 "" H 3100 2400 60  0000 C CNN
+	1    3100 2400
+	-1   0    0    1
 $EndComp
 Text HLabel 2550 2100 1    60   Input ~ 0
 3.3V
 Wire Wire Line
-	2550 2100 2550 2450
-Wire Wire Line
-	4850 2700 2950 2700
-Wire Wire Line
-	2950 2700 2950 2450
-Wire Wire Line
-	2950 2450 2550 2450
-Wire Wire Line
-	4850 2900 2950 2900
-Wire Wire Line
-	2950 2900 2950 3050
-Wire Wire Line
-	2950 3050 2550 3050
+	2550 2100 2550 3050
 Text HLabel 7950 3300 2    60   Output ~ 0
 TCK
@@
 Wire Wire Line
 	4550 3300 4850 3300
+Text HLabel 7100 3700 2    60   Input ~ 0
+~RST
+Wire Wire Line
+	6850 3700 7100 3700
+$Comp
+L JUMPER JP3
+U 1 1 54768CBB
+P 3100 3050
+F 0 "JP3" H 3100 3200 60  0000 C CNN
+F 1 "JUMPER" H 3100 2970 40  0000 C CNN
+F 2 "Connect:TESTPOINT" H 3100 3050 60  0001 C CNN
+F 3 "" H 3100 3050 60  0000 C CNN
+	1    3100 3050
+	-1   0    0    1
+$EndComp
+Wire Wire Line
+	4750 3050 4750 2900
+Wire Wire Line
+	4750 2900 4850 2900
+Wire Wire Line
+	2550 3050 2800 3050
+Wire Wire Line
+	2800 2400 2550 2400
+Connection ~ 2550 2400
+Wire Wire Line
+	3400 3050 4750 3050
+Wire Wire Line
+	3400 2400 4750 2400
+Wire Wire Line
+	4750 2400 4750 2700
+Wire Wire Line
+	4750 2700 4850 2700
 $EndSCHEMATC

Commit message: 1st Revision
Complete Board layout, 1st Draft
Parts:
- removed JP2, JP3: JUMPER, Connect:TESTPOINT, symbol JUMPER
- added JP2: JUMPER3, GEM:TESTPOINT3, symbol JUMPER3
- U14: footprint (none) -> GEM:JTAG2X7
Connections:
- net 3.3V: now also U14.4 (VCC_TARG), JP2.1
- net at U14.2 (VCC/TOOL): now also JP2.3
- net TEST/VPP: no longer names the net of U14.8 (TEST/VPP)
- new net VCC/TOOL: JP2.2
- no-connect marks 0 -> 1
Changed lines of the file:
@@
 $Descr A4 11693 8268
 encoding utf-8
-Sheet 11 11
+Sheet 11 12
 Title ""
 Date ""
@@
 Comment4 ""
 $EndDescr
-$Comp
-L JUMPER JP2
-U 1 1 5474DC6F
-P 3100 2400
-F 0 "JP2" H 3100 2550 60  0000 C CNN
-F 1 "JUMPER" H 3100 2320 40  0000 C CNN
-F 2 "Connect:TESTPOINT" H 3100 2400 60  0001 C CNN
-F 3 "" H 3100 2400 60  0000 C CNN
-	1    3100 2400
-	-1   0    0    1
-$EndComp
-Text HLabel 2550 2100 1    60   Input ~ 0
+Text HLabel 3500 3200 0    60   Input ~ 0
 3.3V
-Wire Wire Line
-	2550 2100 2550 3050
 Text HLabel 7950 3300 2    60   Output ~ 0
 TCK
-Wire Wire Line
-	6850 3300 7950 3300
 Text HLabel 7950 2700 2    60   BiDi ~ 0
 TDO/TDI
-Wire Wire Line
-	7950 2700 6850 2700
 Text HLabel 7950 3500 2    60   Input ~ 0
 GND
-Wire Wire Line
-	7950 3500 6850 3500
 Text HLabel 7150 2900 2    60   Input ~ 0
 TDI/VPP
@@
 U 1 1 5474BF80
 P 5900 3400
-F 0 "U14" H 5900 3400 60  0000 C TNN
+F 0 "U14" H 5900 3300 60  0000 C TNN
 F 1 "JTAG_HEADER" H 5900 3400 60  0000 C BNN
-F 2 "" H 5900 3400 60  0001 C CNN
+F 2 "GEM:JTAG2X7" H 5900 3400 60  0001 C CNN
 F 3 "" H 5900 3400 60  0000 C CNN
 	1    5900 3400
 	1    0    0    -1
 $EndComp
+Text HLabel 7150 3100 2    60   Input ~ 0
+TMS
+Text HLabel 7100 3700 2    60   Input ~ 0
+~RST
+Text HLabel 3850 2650 2    60   Output ~ 0
+VCC/TOOL
+$Comp
+L JUMPER3 JP2
+U 1 1 54C7E8FC
+P 3600 2650
+F 0 "JP2" H 3650 2550 40  0000 L CNN
+F 1 "JUMPER3" H 3600 2750 40  0000 C CNN
+F 2 "GEM:TESTPOINT3" H 3650 3250 60  0000 C CNN
+F 3 "" H 3600 2650 60  0000 C CNN
+	1    3600 2650
+	0    -1   -1   0
+$EndComp
+Wire Wire Line
+	6850 3300 7950 3300
+Wire Wire Line
+	7950 2700 6850 2700
+Wire Wire Line
+	7950 3500 6850 3500
 Wire Wire Line
 	7150 2900 6850 2900
-Text HLabel 7150 3100 2    60   Input ~ 0
-TMS
 Wire Wire Line
 	6850 3100 7150 3100
-Text HLabel 4550 3300 0    60   Input ~ 0
-TEST/VPP
 Wire Wire Line
-	4550 3300 4850 3300
-Text HLabel 7100 3700 2    60   Input ~ 0
-~RST
+	4850 2700 4550 2700
 Wire Wire Line
-	6850 3700 7100 3700
-$Comp
-L JUMPER JP3
-U 1 1 54768CBB
-P 3100 3050
-F 0 "JP3" H 3100 3200 60  0000 C CNN
-F 1 "JUMPER" H 3100 2970 40  0000 C CNN
-F 2 "Connect:TESTPOINT" H 3100 3050 60  0001 C CNN
-F 3 "" H 3100 3050 60  0000 C CNN
-	1    3100 3050
-	-1   0    0    1
-$EndComp
+	4550 2700 4550 2400
 Wire Wire Line
-	4750 3050 4750 2900
+	4550 2400 3600 2400
 Wire Wire Line
-	4750 2900 4850 2900
+	3600 2900 4850 2900
 Wire Wire Line
-	2550 3050 2800 3050
+	3500 3200 3800 3200
 Wire Wire Line
-	2800 2400 2550 2400
-Connection ~ 2550 2400
+	3800 3200 3800 2900
+Connection ~ 3800 2900
 Wire Wire Line
-	3400 3050 4750 3050
+	3850 2650 3700 2650
+NoConn ~ 4850 3300
 Wire Wire Line
-	3400 2400 4750 2400
-Wire Wire Line
-	4750 2400 4750 2700
-Wire Wire Line
-	4750 2700 4850 2700
+	7100 3700 6850 3700
 $EndSCHEMATC
