File: MicroSD.sch (KiCad schematic (older format))
At the start: 1 part, among them U4? microSD

Commit message: Added JTAG interface
Spy Bi-Wire JTAG interface. Fixed some unused pins.
Parts:
- gave numbers to parts that had none: 1
Other:
- note added: "Might Need Pull Up Resistors Not Sure"
Changed lines of the file:
@@
 $Descr A4 11693 8268
 encoding utf-8
-Sheet 10 10
+Sheet 10 11
 Title ""
 Date ""
@@
 $EndDescr
 $Comp
-L microSD U4?
+L microSD U9
 U 1 1 547AAAD6
 P 5650 3000
-F 0 "U4?" H 5650 3000 60  0000 C TNN
+F 0 "U9" H 5650 3000 60  0000 C TNN
 F 1 "microSD" H 5650 3000 60  0000 C BNN
 F 2 "" H 5650 3000 60  0000 C CNN
@@
 Wire Wire Line
 	4950 3100 4400 3100
+Text Notes 6550 2300 2    60   ~ 0
+Might Need Pull Up Resistors Not Sure
 $EndSCHEMATC

Commit message: Linked components to footprints, may have to switch to smaller components. Started board layout.
Parts:
- renumbered U9 to U13
Changed lines of the file:
@@
 $EndDescr
 $Comp
-L microSD U9
+L microSD U13
 U 1 1 547AAAD6
 P 5650 3000
-F 0 "U9" H 5650 3000 60  0000 C TNN
+F 0 "U13" H 5650 3000 60  0000 C TNN
 F 1 "microSD" H 5650 3000 60  0000 C BNN
-F 2 "" H 5650 3000 60  0000 C CNN
+F 2 "" H 5650 3000 60  0001 C CNN
 F 3 "" H 5650 3000 60  0000 C CNN
 	1    5650 3000

Commit message: 1st Revision
Complete Board layout, 1st Draft
Parts:
- U13: footprint (none) -> GEM:MicroSD_Slot
Changed lines of the file:
@@
 $Descr A4 11693 8268
 encoding utf-8
-Sheet 10 11
+Sheet 10 12
 Title ""
 Date ""
@@
 F 0 "U13" H 5650 3000 60  0000 C TNN
 F 1 "microSD" H 5650 3000 60  0000 C BNN
-F 2 "" H 5650 3000 60  0001 C CNN
+F 2 "GEM:MicroSD_Slot" H 5650 3000 60  0001 C CNN
 F 3 "" H 5650 3000 60  0000 C CNN
 	1    5650 3000
