File: RN4020.sch (KiCad schematic (older format))
At the start: 1 part, among them U3? RN4020

Commit message: Added JTAG interface
Spy Bi-Wire JTAG interface. Fixed some unused pins.
Parts:
- gave numbers to parts that had none: 1
Changed lines of the file:
@@
 $Descr A4 11693 8268
 encoding utf-8
-Sheet 9 10
+Sheet 9 11
 Title ""
 Date ""
@@
 $EndDescr
 $Comp
-L RN4020 U3?
+L RN4020 U8
 U 1 1 5478E599
 P 5850 3750
-F 0 "U3?" H 5850 3750 60  0000 C BNN
+F 0 "U8" H 5850 3750 60  0000 C BNN
 F 1 "RN4020" H 5850 3750 60  0000 C TNN
 F 2 "" H 5850 3750 60  0000 C CNN
@@
 	6650 3900 6650 3300
 Connection ~ 6650 3300
+Connection ~ 5150 3600
 $EndSCHEMATC

Commit message: Linked components to footprints, may have to switch to smaller components. Started board layout.
Parts:
- renumbered U8 to U12
Changed lines of the file:
@@
 $EndDescr
 $Comp
-L RN4020 U8
+L RN4020 U12
 U 1 1 5478E599
 P 5850 3750
-F 0 "U8" H 5850 3750 60  0000 C BNN
+F 0 "U12" H 5850 3750 60  0000 C BNN
 F 1 "RN4020" H 5850 3750 60  0000 C TNN
-F 2 "" H 5850 3750 60  0000 C CNN
+F 2 "" H 5850 3750 60  0001 C CNN
 F 3 "" H 5850 3750 60  0000 C CNN
 	1    5850 3750

Commit message: 1st Revision
Complete Board layout, 1st Draft
Parts:
- U12: footprint (none) -> GEM:RN4020_BT
Changed lines of the file:
@@
 $Descr A4 11693 8268
 encoding utf-8
-Sheet 9 11
+Sheet 9 12
 Title ""
 Date ""
@@
 F 0 "U12" H 5850 3750 60  0000 C BNN
 F 1 "RN4020" H 5850 3750 60  0000 C TNN
-F 2 "" H 5850 3750 60  0001 C CNN
+F 2 "GEM:RN4020_BT" H 5850 3750 60  0001 C CNN
 F 3 "" H 5850 3750 60  0000 C CNN
 	1    5850 3750
