File: VOLTAGE_SENSE.sch (KiCad schematic (older format))
At the start: 5 parts

Commit message: Linked components to footprints, may have to switch to smaller components. Started board layout.
Parts:
- C17: value C -> 0.1U; footprint (none) -> SMD_Packages:SMD-1206
- R47: renamed from R45; value R -> 62K; footprint (none) -> Resistors_SMD:R_1206_HandSoldering
- R48: renamed from R46; value R -> 10K; footprint (none) -> Resistors_SMD:R_1206_HandSoldering
- renumbered D12 to D14, D13 to D15
Changed lines of the file:
@@
 $EndDescr
 $Comp
-L R R45
+L R R47
 U 1 1 546AC07E
 P 3000 2600
-F 0 "R45" V 3080 2600 40  0000 C CNN
-F 1 "R" V 3007 2601 40  0000 C CNN
-F 2 "" V 2930 2600 30  0000 C CNN
+F 0 "R47" V 3080 2600 40  0000 C CNN
+F 1 "62K" V 3007 2601 40  0000 C CNN
+F 2 "Resistors_SMD:R_1206_HandSoldering" V 2930 2600 30  0001 C CNN
 F 3 "" H 3000 2600 30  0000 C CNN
 	1    3000 2600
@@
 $EndComp
 $Comp
-L R R46
+L R R48
 U 1 1 546AC124
 P 3000 3400
-F 0 "R46" V 3080 3400 40  0000 C CNN
-F 1 "R" V 3007 3401 40  0000 C CNN
-F 2 "" V 2930 3400 30  0000 C CNN
+F 0 "R48" V 3080 3400 40  0000 C CNN
+F 1 "10K" V 3007 3401 40  0000 C CNN
+F 2 "Resistors_SMD:R_1206_HandSoldering" V 2930 3400 30  0001 C CNN
 F 3 "" H 3000 3400 30  0000 C CNN
 	1    3000 3400
@@
 P 2550 3350
 F 0 "C17" H 2550 3450 40  0000 L CNN
-F 1 "C" H 2556 3265 40  0000 L CNN
-F 2 "" H 2588 3200 30  0000 C CNN
+F 1 "0.1U" H 2556 3265 40  0000 L CNN
+F 2 "SMD_Packages:SMD-1206" H 2588 3200 30  0001 C CNN
 F 3 "" H 2550 3350 60  0000 C CNN
 	1    2550 3350
@@
 $EndComp
 $Comp
-L DIODESCH D12
+L DIODESCH D14
 U 1 1 546AC513
 P 3750 2650
-F 0 "D12" H 3750 2750 40  0000 C CNN
+F 0 "D14" H 3750 2750 40  0000 C CNN
 F 1 "DIODESCH" H 3750 2550 40  0000 C CNN
-F 2 "" H 3750 2650 60  0000 C CNN
+F 2 "" H 3750 2650 60  0001 C CNN
 F 3 "" H 3750 2650 60  0000 C CNN
 	1    3750 2650
@@
 $EndComp
 $Comp
-L DIODESCH D13
+L DIODESCH D15
 U 1 1 546AC588
 P 3750 3350
-F 0 "D13" H 3750 3450 40  0000 C CNN
+F 0 "D15" H 3750 3450 40  0000 C CNN
 F 1 "DIODESCH" H 3750 3250 40  0000 C CNN
-F 2 "" H 3750 3350 60  0000 C CNN
+F 2 "" H 3750 3350 60  0001 C CNN
 F 3 "" H 3750 3350 60  0000 C CNN
 	1    3750 3350

Commit message: General fine tuning of schematics. Need to review JTAG and update. Added resistors to power stage. Getting prepped for BOM, need to go through item by item. Added current incomplete BOM
Parts:
- C17: footprint SMD_Packages:SMD-1206 -> SMD_Packages:SMD-0805
Changed lines of the file:
@@
 F 0 "C17" H 2550 3450 40  0000 L CNN
 F 1 "0.1U" H 2556 3265 40  0000 L CNN
-F 2 "SMD_Packages:SMD-1206" H 2588 3200 30  0001 C CNN
+F 2 "SMD_Packages:SMD-0805" H 2588 3200 30  0001 C CNN
 F 3 "" H 2550 3350 60  0000 C CNN
 	1    2550 3350

Commit message: Updated parts and data sheets
Parts:
- C17: footprint SMD_Packages:SMD-0805 -> Capacitors_SMD:C_0805_HandSoldering
- D14, D15: value DIODESCH -> BAT46
- R47, R48: footprint Resistors_SMD:R_1206_HandSoldering -> Resistors_SMD:R_0805_HandSoldering
Changed lines of the file:
@@
 F 0 "R47" V 3080 2600 40  0000 C CNN
 F 1 "62K" V 3007 2601 40  0000 C CNN
-F 2 "Resistors_SMD:R_1206_HandSoldering" V 2930 2600 30  0001 C CNN
+F 2 "Resistors_SMD:R_0805_HandSoldering" V 2930 2600 30  0001 C CNN
 F 3 "" H 3000 2600 30  0000 C CNN
 	1    3000 2600
@@
 F 0 "R48" V 3080 3400 40  0000 C CNN
 F 1 "10K" V 3007 3401 40  0000 C CNN
-F 2 "Resistors_SMD:R_1206_HandSoldering" V 2930 3400 30  0001 C CNN
+F 2 "Resistors_SMD:R_0805_HandSoldering" V 2930 3400 30  0001 C CNN
 F 3 "" H 3000 3400 30  0000 C CNN
 	1    3000 3400
@@
 F 0 "C17" H 2550 3450 40  0000 L CNN
 F 1 "0.1U" H 2556 3265 40  0000 L CNN
-F 2 "SMD_Packages:SMD-0805" H 2588 3200 30  0001 C CNN
+F 2 "Capacitors_SMD:C_0805_HandSoldering" H 2588 3200 30  0001 C CNN
 F 3 "" H 2550 3350 60  0000 C CNN
 	1    2550 3350
@@
 P 3750 2650
 F 0 "D14" H 3750 2750 40  0000 C CNN
-F 1 "DIODESCH" H 3750 2550 40  0000 C CNN
+F 1 "BAT46" H 3750 2550 40  0000 C CNN
 F 2 "" H 3750 2650 60  0001 C CNN
 F 3 "" H 3750 2650 60  0000 C CNN
@@
 P 3750 3350
 F 0 "D15" H 3750 3450 40  0000 C CNN
-F 1 "DIODESCH" H 3750 3250 40  0000 C CNN
+F 1 "BAT46" H 3750 3250 40  0000 C CNN
 F 2 "" H 3750 3350 60  0001 C CNN
 F 3 "" H 3750 3350 60  0000 C CNN
